Commit message: maybe final add all body

File: moi_arm_description/urdf/moi_arm.xacro (robot description, xacro)
@@ -346,7 +346,7 @@
 <link name="Component5_3">
   <inertial>
-    <origin xyz="0.0005767742551691102 2.0749739274017465e-07 2.0905313929953095e-07" rpy="0 0 0"/>
+    <origin xyz="0.0005767742551684579 2.0749790605179008e-07 2.0905367620338566e-07" rpy="0 0 0"/>
     <mass value="0.013145620261468437"/>
-    <inertia ixx="1e-06" iyy="0.0" izz="0.0" ixy="-0.0" iyz="0.0" ixz="-0.0"/>
+    <inertia ixx="1e-06" iyy="0.0" izz="0.0" ixy="-0.0" iyz="-0.0" ixz="0.0"/>
   </inertial>
   <visual>
@@ -506,7 +506,7 @@
 <link name="Component9_2">
   <inertial>
-    <origin xyz="-0.05300000085833196 -0.03104819671407337 8.663853407475663e-07" rpy="0 0 0"/>
+    <origin xyz="-0.053000000837303475 8.647958510688003e-07 0.031048613299398786" rpy="0 0 0"/>
     <mass value="0.7282309507071387"/>
-    <inertia ixx="0.000224" iyy="0.000727" izz="0.000822" ixy="-0.0" iyz="0.0" ixz="-0.0"/>
+    <inertia ixx="0.000224" iyy="0.000822" izz="0.000727" ixy="-0.0" iyz="-0.0" ixz="0.0"/>
   </inertial>
   <visual>
@@ -521,4 +521,244 @@
     <geometry>
       <mesh filename="file://$(find moi_arm_description)/meshes/Component9_2.stl" scale="0.001 0.001 0.001"/>
+    </geometry>
+  </collision>
+</link>
+<link name="Component10_2">
+  <inertial>
+    <origin xyz="-0.012000117657645493 -0.009499269916191766 0.05294225526470597" rpy="0 0 0"/>
+    <mass value="1.0029838563695943"/>
+    <inertia ixx="0.001903" iyy="0.002087" izz="0.000249" ixy="-0.0" iyz="0.0" ixz="-0.0"/>
+  </inertial>
+  <visual>
+    <origin xyz="-0.0105 0.072981 -0.350413" rpy="0 0 0"/>
+    <geometry>
+      <mesh filename="file://$(find moi_arm_description)/meshes/Component10_2.stl" scale="0.001 0.001 0.001"/>
+    </geometry>
+    <material name="silver"/>
+  </visual>
+  <collision>
+    <origin xyz="-0.0105 0.072981 -0.350413" rpy="0 0 0"/>
+    <geometry>
+      <mesh filename="file://$(find moi_arm_description)/meshes/Component10_2.stl" scale="0.001 0.001 0.001"/>
+    </geometry>
+  </collision>
+</link>
+<link name="Component12_1">
+  <inertial>
+    <origin xyz="-0.025500001764371456 3.338235568528525e-08 0.003609738501345827" rpy="0 0 0"/>
+    <mass value="0.35698450055073755"/>
+    <inertia ixx="9.9e-05" iyy="0.000177" izz="0.000181" ixy="0.0" iyz="0.0" ixz="0.0"/>
+  </inertial>
+  <visual>
+    <origin xyz="-0.023 0.082481 -0.474413" rpy="0 0 0"/>
+    <geometry>
+      <mesh filename="file://$(find moi_arm_description)/meshes/Component12_1.stl" scale="0.001 0.001 0.001"/>
+    </geometry>
+    <material name="silver"/>
+  </visual>
+  <collision>
+    <origin xyz="-0.023 0.082481 -0.474413" rpy="0 0 0"/>
+    <geometry>
+      <mesh filename="file://$(find moi_arm_description)/meshes/Component12_1.stl" scale="0.001 0.001 0.001"/>
+    </geometry>
+  </collision>
+</link>
+<link name="Component4_2">
+  <inertial>
+    <origin xyz="-0.008000000670917414 -0.007982460039636222 0.0023970220537695708" rpy="0 0 0"/>
+    <mass value="0.02516998505835531"/>
+    <inertia ixx="2e-06" iyy="4e-06" izz="5e-06" ixy="0.0" iyz="-0.0" ixz="0.0"/>
+  </inertial>
+  <visual>
+    <origin xyz="-0.0055 0.074481 -0.492806" rpy="0 0 0"/>
+    <geometry>
+      <mesh filename="file://$(find moi_arm_description)/meshes/Component4_2.stl" scale="0.001 0.001 0.001"/>
+    </geometry>
+    <material name="silver"/>
+  </visual>
+  <collision>
+    <origin xyz="-0.0055 0.074481 -0.492806" rpy="0 0 0"/>
+    <geometry>
+      <mesh filename="file://$(find moi_arm_description)/meshes/Component4_2.stl" scale="0.001 0.001 0.001"/>
+    </geometry>
+  </collision>
+</link>
+<link name="Component5_5">
+  <inertial>
+    <origin xyz="0.0005767744058065068 -1.4019937155662632e-08 -3.3672760357816856e-07" rpy="0 0 0"/>
+    <mass value="0.013145620261468437"/>
+    <inertia ixx="1e-06" iyy="0.0" izz="0.0" ixy="0.0" iyz="0.0" ixz="-0.0"/>
+  </inertial>
+  <visual>
+    <origin xyz="-0.01545 0.082481 -0.534306" rpy="0 0 0"/>
+    <geometry>
+      <mesh filename="file://$(find moi_arm_description)/meshes/Component5_5.stl" scale="0.001 0.001 0.001"/>
+    </geometry>
+    <material name="silver"/>
+  </visual>
+  <collision>
+    <origin xyz="-0.01545 0.082481 -0.534306" rpy="0 0 0"/>
+    <geometry>
+      <mesh filename="file://$(find moi_arm_description)/meshes/Component5_5.stl" scale="0.001 0.001 0.001"/>
+    </geometry>
+  </collision>
+</link>
+<link name="Component8_5">
+  <inertial>
+    <origin xyz="-0.002777925429963366 0.009249998583650346 -0.0224569712862136" rpy="0 0 0"/>
+    <mass value="0.051461187075064724"/>
+    <inertia ixx="1.4e-05" iyy="1e-05" izz="4e-06" ixy="0.0" iyz="0.0" ixz="-0.0"/>
+  </inertial>
+  <visual>
+    <origin xyz="0.0135 0.091731 -0.543306" rpy="0 0 0"/>
+    <geometry>
+      <mesh filename="file://$(find moi_arm_description)/meshes/Component8_5.stl" scale="0.001 0.001 0.001"/>
+    </geometry>
+    <material name="silver"/>
+  </visual>
+  <collision>
+    <origin xyz="0.0135 0.091731 -0.543306" rpy="0 0 0"/>
+    <geometry>
+      <mesh filename="file://$(find moi_arm_description)/meshes/Component8_5.stl" scale="0.001 0.001 0.001"/>
+    </geometry>
+  </collision>
+</link>
+<link name="Component6_5">
+  <inertial>
+    <origin xyz="-0.011000000652923338 0.009249997718981523 -0.021533847588900423" rpy="0 0 0"/>
+    <mass value="0.20992105246147483"/>
+    <inertia ixx="5e-05" iyy="4.7e-05" izz="2e-05" ixy="-0.0" iyz="0.0" ixz="-0.0"/>
+  </inertial>
+  <visual>
+    <origin xyz="-0.0085 0.091731 -0.543306" rpy="0 0 0"/>
+    <geometry>
+      <mesh filename="file://$(find moi_arm_description)/meshes/Component6_5.stl" scale="0.001 0.001 0.001"/>
+    </geometry>
+    <material name="silver"/>
+  </visual>
+  <collision>
+    <origin xyz="-0.0085 0.091731 -0.543306" rpy="0 0 0"/>
+    <geometry>
+      <mesh filename="file://$(find moi_arm_description)/meshes/Component6_5.stl" scale="0.001 0.001 0.001"/>
+    </geometry>
+  </collision>
+</link>
+<link name="Component7_5">
+  <inertial>
+    <origin xyz="-0.0018119637897111365 -0.008000026888941511 0.021152599170006336" rpy="0 0 0"/>
+    <mass value="0.061219272040330903"/>
+    <inertia ixx="1.4e-05" iyy="1e-05" izz="4e-06" ixy="0.0" iyz="0.0" ixz="0.0"/>
+  </inertial>
+  <visual>
+    <origin xyz="-0.0135 0.074481 -0.498306" rpy="0 0 0"/>
+    <geometry>
+      <mesh filename="file://$(find moi_arm_description)/meshes/Component7_5.stl" scale="0.001 0.001 0.001"/>
+    </geometry>
+    <material name="silver"/>
+  </visual>
+  <collision>
+    <origin xyz="-0.0135 0.074481 -0.498306" rpy="0 0 0"/>
+    <geometry>
+      <mesh filename="file://$(find moi_arm_description)/meshes/Component7_5.stl" scale="0.001 0.001 0.001"/>
+    </geometry>
+  </collision>
+</link>
+<link name="Component13_1">
+  <inertial>
+    <origin xyz="-0.15211825499488402 0.018784043229143926 -0.4776890566257409" rpy="0 0 0"/>
+    <mass value="1.0315085930732382"/>
+    <inertia ixx="0.017798" iyy="0.019327" izz="0.004867" ixy="4.7e-05" iyz="0.000171" ixz="-0.004447"/>
+  </inertial>
+  <visual>
+    <origin xyz="-0.01845 0.082481 -0.534306" rpy="0 0 0"/>
+    <geometry>
+      <mesh filename="file://$(find moi_arm_description)/meshes/Component13_1.stl" scale="0.001 0.001 0.001"/>
+    </geometry>
+    <material name="silver"/>
+  </visual>
+  <collision>
+    <origin xyz="-0.01845 0.082481 -0.534306" rpy="0 0 0"/>
+    <geometry>
+      <mesh filename="file://$(find moi_arm_description)/meshes/Component13_1.stl" scale="0.001 0.001 0.001"/>
+    </geometry>
+  </collision>
+</link>
+<link name="Component5_6">
+  <inertial>
+    <origin xyz="-1.681908239634447e-09 0.0005767607955906827 -2.8295855780680057e-07" rpy="0 0 0"/>
+    <mass value="0.013145620261468437"/>
+    <inertia ixx="0.0" iyy="1e-06" izz="0.0" ixy="-0.0" iyz="0.0" ixz="-0.0"/>
+  </inertial>
+  <visual>
+    <origin xyz="0.00165 0.026031 -0.534556" rpy="0 0 0"/>
+    <geometry>
+      <mesh filename="file://$(find moi_arm_description)/meshes/Component5_6.stl" scale="0.001 0.001 0.001"/>
+    </geometry>
+    <material name="silver"/>
+  </visual>
+  <collision>
+    <origin xyz="0.00165 0.026031 -0.534556" rpy="0 0 0"/>
+    <geometry>
+      <mesh filename="file://$(find moi_arm_description)/meshes/Component5_6.stl" scale="0.001 0.001 0.001"/>
+    </geometry>
+  </collision>
+</link>
+<link name="Component7_6">
+  <inertial>
+    <origin xyz="0.009250025083460886 0.003188036516552001 -0.02384735112771652" rpy="0 0 0"/>
+    <mass value="0.061219272040330903"/>
+    <inertia ixx="1e-05" iyy="1.4e-05" izz="4e-06" ixy="-0.0" iyz="0.0" ixz="-0.0"/>
+  </inertial>
+  <visual>
+    <origin xyz="0.0109 0.032981 -0.543556" rpy="0 0 0"/>
+    <geometry>
+      <mesh filename="file://$(find moi_arm_description)/meshes/Component7_6.stl" scale="0.001 0.001 0.001"/>
+    </geometry>
+    <material name="silver"/>
+  </visual>
+  <collision>
+    <origin xyz="0.0109 0.032981 -0.543556" rpy="0 0 0"/>
+    <geometry>
+      <mesh filename="file://$(find moi_arm_description)/meshes/Component7_6.stl" scale="0.001 0.001 0.001"/>
+    </geometry>
+  </collision>
+</link>
+<link name="Component6_6">
+  <inertial>
+    <origin xyz="0.00924999831012794 0.010999997484802126 -0.021533811185405094" rpy="0 0 0"/>
+    <mass value="0.20992105246147483"/>
+    <inertia ixx="4.7e-05" iyy="5e-05" izz="2e-05" ixy="0.0" iyz="0.0" ixz="-0.0"/>
+  </inertial>
+  <visual>
+    <origin xyz="0.0109 0.054981 -0.543556" rpy="0 0 0"/>
+    <geometry>
+      <mesh filename="file://$(find moi_arm_description)/meshes/Component6_6.stl" scale="0.001 0.001 0.001"/>
+    </geometry>
+    <material name="silver"/>
+  </visual>
+  <collision>
+    <origin xyz="0.0109 0.054981 -0.543556" rpy="0 0 0"/>
+    <geometry>
+      <mesh filename="file://$(find moi_arm_description)/meshes/Component6_6.stl" scale="0.001 0.001 0.001"/>
+    </geometry>
+  </collision>
+</link>
+<link name="Component8_6">
+  <inertial>
+    <origin xyz="0.013499998309469474 0.0022220735730321753 -0.006706947797067597" rpy="0 0 0"/>
+    <mass value="0.051461187075064724"/>
+    <inertia ixx="1e-05" iyy="1.4e-05" izz="4e-06" ixy="-0.0" iyz="-0.0" ixz="-0.0"/>
+  </inertial>
+  <visual>
+    <origin xyz="0.01515 0.059981 -0.527806" rpy="0 0 0"/>
+    <geometry>
+      <mesh filename="file://$(find moi_arm_description)/meshes/Component8_6.stl" scale="0.001 0.001 0.001"/>
+    </geometry>
+    <material name="silver"/>
+  </visual>
+  <collision>
+    <origin xyz="0.01515 0.059981 -0.527806" rpy="0 0 0"/>
+    <geometry>
+      <mesh filename="file://$(find moi_arm_description)/meshes/Component8_6.stl" scale="0.001 0.001 0.001"/>
     </geometry>
   </collision>
@@ -653,3 +893,65 @@
   <child link="Component9_2"/>
 </joint>
+<joint name="Rigid 28" type="fixed">
+  <origin xyz="-0.041 0.0105 0.052971" rpy="0 0 0"/>
+  <parent link="Component9_2"/>
+  <child link="Component10_2"/>
+</joint>
+<joint name="Rigid 29" type="fixed">
+  <origin xyz="0.0125 -0.0095 0.124" rpy="0 0 0"/>
+  <parent link="Component10_2"/>
+  <child link="Component12_1"/>
+</joint>
+<joint name="Rigid 30" type="fixed">
+  <origin xyz="-0.0175 0.008 0.018393" rpy="0 0 0"/>
+  <parent link="Component12_1"/>
+  <child link="Component4_2"/>
+</joint>
+<joint name="Revolute 31" type="continuous">
+  <origin xyz="0.00195 -0.008 0.036" rpy="0 0 0"/>
+  <parent link="Component7_5"/>
+  <child link="Component5_5"/>
+  <axis xyz="1.0 -0.0 -0.0"/>
+</joint>
+<joint name="Rigid 32" type="fixed">
+  <origin xyz="-0.022 0.0 0.0" rpy="0 0 0"/>
+  <parent link="Component6_5"/>
+  <child link="Component8_5"/>
+</joint>
+<joint name="Rigid 33" type="fixed">
+  <origin xyz="-0.005 -0.01725 0.045" rpy="0 0 0"/>
+  <parent link="Component7_5"/>
+  <child link="Component6_5"/>
+</joint>
+<joint name="Rigid 34" type="fixed">
+  <origin xyz="0.008 0.0 0.0055" rpy="0 0 0"/>
+  <parent link="Component4_2"/>
+  <child link="Component7_5"/>
+</joint>
+<joint name="Rigid 35" type="fixed">
+  <origin xyz="0.003 0.0 0.0" rpy="0 0 0"/>
+  <parent link="Component5_5"/>
+  <child link="Component13_1"/>
+</joint>
+<joint name="Revolute 36" type="continuous">
+  <origin xyz="0.00925 0.00695 -0.009" rpy="0 0 0"/>
+  <parent link="Component7_6"/>
+  <child link="Component5_6"/>
+  <axis xyz="0.0 1.0 1e-06"/>
+</joint>
+<joint name="Rigid 37" type="fixed">
+  <origin xyz="0.0 0.022 0.0" rpy="0 0 0"/>
+  <parent link="Component6_6"/>
+  <child link="Component7_6"/>
+</joint>
+<joint name="Rigid 38" type="fixed">
+  <origin xyz="0.00425 0.005 0.01575" rpy="0 0 0"/>
+  <parent link="Component8_6"/>
+  <child link="Component6_6"/>
+</joint>
+<joint name="Rigid 39" type="fixed">
+  <origin xyz="-0.0336 0.0225 -0.0065" rpy="0 0 0"/>
+  <parent link="Component13_1"/>
+  <child link="Component8_6"/>
+</joint>
 </robot>

Commit message: edit

File: moi_arm_description/urdf/moi_arm.xacro (robot description, xacro)
@@ -666,7 +666,7 @@
 <link name="Component13_1">
   <inertial>
-    <origin xyz="-0.15211825499488402 0.018784043229143926 -0.4776890566257409" rpy="0 0 0"/>
-    <mass value="1.0315085930732382"/>
-    <inertia ixx="0.017798" iyy="0.019327" izz="0.004867" ixy="4.7e-05" iyz="0.000171" ixz="-0.004447"/>
+    <origin xyz="-0.020207239586969048 0.013746542101945272 -0.005523783162298623" rpy="0 0 0"/>
+    <mass value="0.06677763124410402"/>
+    <inertia ixx="2.1e-05" iyy="3.7e-05" izz="2.9e-05" ixy="-0.0" iyz="3e-06" ixz="0.0"/>
   </inertial>
   <visual>
