Commit message: i should change file name

File: mycobot320_4_4_description/urdf/mycobot320_4_4.xacro (robot description, xacro)
@@ -284,4 +284,5 @@
   </collision>
 </link>
+<!-- joint -->
 <joint name="joint2_to_joint1" type="continuous">
   <origin xyz="0.0 0.060072 0.114761" rpy="0 0 0"/>
@@ -325,4 +326,5 @@
   <child link="gripper_base_1"/>
 </joint>
+<!-- gripper joints -->
 <joint name="gripper_controller" type="revolute">
   <origin xyz="0.060541 -0.010461 0.018171" rpy="0 0 0"/>
@@ -338,4 +340,5 @@
   <axis xyz="-0.000407 -1.0 0.000299"/>
   <limit upper="0.261799" lower="-0.698132" effort="100" velocity="100"/>
+  <mimic joint="gripper_controller" multiplier="-1" offset="0"/>
 </joint>
 <joint name="gripper_base_to_gripper_right2" type="revolute">
@@ -345,4 +348,5 @@
   <axis xyz="0.000407 1.0 -0.000299"/>
   <limit upper="0.0" lower="-0.698132" effort="100" velocity="100"/>
+  <mimic joint="gripper_controller" multiplier="-1" offset="0"/>
 </joint>
 <joint name="gripper_base_to_gripper_left3" type="revolute">
@@ -352,4 +356,5 @@
   <axis xyz="-0.000407 -1.0 0.000299"/>
   <limit upper="0.0" lower="-0.698132" effort="100" velocity="100"/>
+  <mimic joint="gripper_controller" multiplier="-1" offset="0"/>
 </joint>
 <joint name="gripper_left3_to_gripper_left1" type="revolute">
@@ -359,4 +364,5 @@
   <axis xyz="0.000407 1.0 -0.000299"/>
   <limit upper="0.0" lower="-0.698132" effort="100" velocity="100"/>
+  <mimic joint="gripper_controller" multiplier="-1" offset="0"/>
 </joint>
 <joint name="gripper_base_to_gripper_left2" type="revolute">
@@ -366,4 +372,5 @@
   <axis xyz="-0.000407 -1.0 0.000299"/>
   <limit upper="0.0" lower="-0.698132" effort="100" velocity="100"/>
+  <mimic joint="gripper_controller" multiplier="-1" offset="0"/>
 </joint>
 </robot>
