Commit message: plz_final

File: mycobot320_description/urdf/mycobot320.xacro (robot description, xacro)
@@ -24,14 +24,14 @@
   </collision>
 </link>
-<link name="link1">
-  <inertial>
-    <origin xyz="0.006894482331010262 0.00017712892998957702 0.055490142550686156" rpy="0 0 0"/>
+<link name="link1_1">
+  <inertial>
+    <origin xyz="0.0068967662247303866 -3.47113377312247e-07 0.055490142550686156" rpy="0 0 0"/>
     <mass value="3.4735206294395446"/>
-    <inertia ixx="0.004461" iyy="0.004757" izz="0.002424" ixy="-8e-06" iyz="-2e-05" ixz="-0.000777"/>
+    <inertia ixx="0.004461" iyy="0.004757" izz="0.002424" ixy="0.0" iyz="0.0" ixz="-0.000777"/>
   </inertial>
   <visual>
     <origin xyz="0.0 -0.060072 -0.114761" rpy="0 0 0"/>
     <geometry>
-      <mesh filename="file://$(find mycobot320_description)/meshes/link1.stl" scale="0.001 0.001 0.001"/>
+      <mesh filename="file://$(find mycobot320_description)/meshes/link1_1.stl" scale="0.001 0.001 0.001"/>
     </geometry>
     <material name="silver"/>
@@ -40,337 +40,330 @@
     <origin xyz="0.0 -0.060072 -0.114761" rpy="0 0 0"/>
     <geometry>
-      <mesh filename="file://$(find mycobot320_description)/meshes/link1.stl" scale="0.001 0.001 0.001"/>
-    </geometry>
-  </collision>
-</link>
-<link name="link2">
-  <inertial>
-    <origin xyz="0.036837500623841266 0.00316217625421885 0.06796391862996645" rpy="0 0 0"/>
+      <mesh filename="file://$(find mycobot320_description)/meshes/link1_1.stl" scale="0.001 0.001 0.001"/>
+    </geometry>
+  </collision>
+</link>
+<link name="link2_1">
+  <inertial>
+    <origin xyz="0.036906585755672405 -3.471133772081636e-07 0.06799995568162978" rpy="0 0 0"/>
     <mass value="5.91988968680626"/>
-    <inertia ixx="0.0188" iyy="0.019319" izz="0.004177" ixy="-1.3e-05" iyz="-0.000494" ixz="1.3e-05"/>
-  </inertial>
-  <visual>
-    <origin xyz="-0.044985 -0.06123 -0.199761" rpy="0 0 0"/>
-    <geometry>
-      <mesh filename="file://$(find mycobot320_description)/meshes/link2.stl" scale="0.001 0.001 0.001"/>
-    </geometry>
-    <material name="silver"/>
-  </visual>
-  <collision>
-    <origin xyz="-0.044985 -0.06123 -0.199761" rpy="0 0 0"/>
-    <geometry>
-      <mesh filename="file://$(find mycobot320_description)/meshes/link2.stl" scale="0.001 0.001 0.001"/>
-    </geometry>
-  </collision>
-</link>
-<link name="link3">
-  <inertial>
-    <origin xyz="-0.035053164367318285 0.0007402802945343234 0.04947264616599745" rpy="0 0 0"/>
+    <inertia ixx="0.0188" iyy="0.019335" izz="0.004161" ixy="-0.0" iyz="-0.0" ixz="-0.0"/>
+  </inertial>
+  <visual>
+    <origin xyz="-0.045 -0.060072 -0.199761" rpy="0 0 0"/>
+    <geometry>
+      <mesh filename="file://$(find mycobot320_description)/meshes/link2_1.stl" scale="0.001 0.001 0.001"/>
+    </geometry>
+    <material name="silver"/>
+  </visual>
+  <collision>
+    <origin xyz="-0.045 -0.060072 -0.199761" rpy="0 0 0"/>
+    <geometry>
+      <mesh filename="file://$(find mycobot320_description)/meshes/link2_1.stl" scale="0.001 0.001 0.001"/>
+    </geometry>
+  </collision>
+</link>
+<link name="link3_1">
+  <inertial>
+    <origin xyz="-0.03502268825299221 3.0162871079306153e-05 0.04949994627901183" rpy="0 0 0"/>
     <mass value="4.802107093668197"/>
-    <inertia ixx="0.01014" iyy="0.010576" izz="0.003394" ixy="-1.1e-05" iyz="-0.000239" ixz="6e-06"/>
-  </inertial>
-  <visual>
-    <origin xyz="-0.044871 -0.065655 -0.335689" rpy="0 0 0"/>
-    <geometry>
-      <mesh filename="file://$(find mycobot320_description)/meshes/link3.stl" scale="0.001 0.001 0.001"/>
-    </geometry>
-    <material name="silver"/>
-  </visual>
-  <collision>
-    <origin xyz="-0.044871 -0.065655 -0.335689" rpy="0 0 0"/>
-    <geometry>
-      <mesh filename="file://$(find mycobot320_description)/meshes/link3.stl" scale="0.001 0.001 0.001"/>
-    </geometry>
-  </collision>
-</link>
-<link name="link4">
-  <inertial>
-    <origin xyz="0.03443819780244397 -0.00012625243718576706 0.010527987134175576" rpy="0 0 0"/>
+    <inertia ixx="0.01014" iyy="0.010584" izz="0.003386" ixy="0.0" iyz="-4e-06" ixz="0.0"/>
+  </inertial>
+  <visual>
+    <origin xyz="-0.045 -0.060072 -0.335761" rpy="0 0 0"/>
+    <geometry>
+      <mesh filename="file://$(find mycobot320_description)/meshes/link3_1.stl" scale="0.001 0.001 0.001"/>
+    </geometry>
+    <material name="silver"/>
+  </visual>
+  <collision>
+    <origin xyz="-0.045 -0.060072 -0.335761" rpy="0 0 0"/>
+    <geometry>
+      <mesh filename="file://$(find mycobot320_description)/meshes/link3_1.stl" scale="0.001 0.001 0.001"/>
+    </geometry>
+  </collision>
+</link>
+<link name="link4_1">
+  <inertial>
+    <origin xyz="0.03442387286919221 6.191592391589784e-06 0.010576061998245567" rpy="0 0 0"/>
     <mass value="2.265107015236222"/>
-    <inertia ixx="0.001594" iyy="0.001803" izz="0.001597" ixy="2.6e-05" iyz="1.2e-05" ixz="-0.000322"/>
-  </inertial>
-  <visual>
-    <origin xyz="-0.044787 -0.068938 -0.434634" rpy="0 0 0"/>
-    <geometry>
-      <mesh filename="file://$(find mycobot320_description)/meshes/link4.stl" scale="0.001 0.001 0.001"/>
-    </geometry>
-    <material name="silver"/>
-  </visual>
-  <collision>
-    <origin xyz="-0.044787 -0.068938 -0.434634" rpy="0 0 0"/>
-    <geometry>
-      <mesh filename="file://$(find mycobot320_description)/meshes/link4.stl" scale="0.001 0.001 0.001"/>
-    </geometry>
-  </collision>
-</link>
-<link name="link5">
-  <inertial>
-    <origin xyz="0.00010333354821902285 -0.004029254098592533 0.04192318950838286" rpy="0 0 0"/>
+    <inertia ixx="0.001595" iyy="0.001803" izz="0.001595" ixy="-0.0" iyz="-0.0" ixz="-0.000324"/>
+  </inertial>
+  <visual>
+    <origin xyz="-0.045 -0.060133 -0.434761" rpy="0 0 0"/>
+    <geometry>
+      <mesh filename="file://$(find mycobot320_description)/meshes/link4_1.stl" scale="0.001 0.001 0.001"/>
+    </geometry>
+    <material name="silver"/>
+  </visual>
+  <collision>
+    <origin xyz="-0.045 -0.060133 -0.434761" rpy="0 0 0"/>
+    <geometry>
+      <mesh filename="file://$(find mycobot320_description)/meshes/link4_1.stl" scale="0.001 0.001 0.001"/>
+    </geometry>
+  </collision>
+</link>
+<link name="link5_1">
+  <inertial>
+    <origin xyz="-1.3877787807814457e-16 2.6368392026507315e-05 0.042116616834545706" rpy="0 0 0"/>
     <mass value="3.029827579494103"/>
-    <inertia ixx="0.0025" iyy="0.002971" izz="0.002446" ixy="0.0" iyz="5.1e-05" ixz="-0.0"/>
-  </inertial>
-  <visual>
-    <origin xyz="-0.089883 -0.06579 -0.479428" rpy="0 0 0"/>
-    <geometry>
-      <mesh filename="file://$(find mycobot320_description)/meshes/link5.stl" scale="0.001 0.001 0.001"/>
-    </geometry>
-    <material name="silver"/>
-  </visual>
-  <collision>
-    <origin xyz="-0.089883 -0.06579 -0.479428" rpy="0 0 0"/>
-    <geometry>
-      <mesh filename="file://$(find mycobot320_description)/meshes/link5.stl" scale="0.001 0.001 0.001"/>
-    </geometry>
-  </collision>
-</link>
-<link name="link6">
-  <inertial>
-    <origin xyz="0.00999958715963864 -3.8937722489085225e-06 -2.536791209295508e-05" rpy="0 0 0"/>
+    <inertia ixx="0.0025" iyy="0.002976" izz="0.002441" ixy="0.0" iyz="-0.0" ixz="-0.0"/>
+  </inertial>
+  <visual>
+    <origin xyz="-0.09 -0.06016 -0.479761" rpy="0 0 0"/>
+    <geometry>
+      <mesh filename="file://$(find mycobot320_description)/meshes/link5_1.stl" scale="0.001 0.001 0.001"/>
+    </geometry>
+    <material name="silver"/>
+  </visual>
+  <collision>
+    <origin xyz="-0.09 -0.06016 -0.479761" rpy="0 0 0"/>
+    <geometry>
+      <mesh filename="file://$(find mycobot320_description)/meshes/link5_1.stl" scale="0.001 0.001 0.001"/>
+    </geometry>
+  </collision>
+</link>
+<link name="link6_1">
+  <inertial>
+    <origin xyz="0.009999999999999898 2.2737115904641891e-07 -8.11690367141793e-08" rpy="0 0 0"/>
     <mass value="0.6042068071016569"/>
-    <inertia ixx="0.00037" iyy="0.000205" izz="0.000205" ixy="-0.0" iyz="0.0" ixz="-0.0"/>
-  </inertial>
-  <visual>
-    <origin xyz="-0.130006 -0.06099 -0.529098" rpy="0 0 0"/>
-    <geometry>
-      <mesh filename="file://$(find mycobot320_description)/meshes/link6.stl" scale="0.001 0.001 0.001"/>
-    </geometry>
-    <material name="silver"/>
-  </visual>
-  <collision>
-    <origin xyz="-0.130006 -0.06099 -0.529098" rpy="0 0 0"/>
-    <geometry>
-      <mesh filename="file://$(find mycobot320_description)/meshes/link6.stl" scale="0.001 0.001 0.001"/>
-    </geometry>
-  </collision>
-</link>
-<link name="gripper_base">
-  <inertial>
-    <origin xyz="0.04130515061115911 0.010013488596629185 -4.428984489124321e-05" rpy="0 0 0"/>
+    <inertia ixx="0.00037" iyy="0.000205" izz="0.000205" ixy="0.0" iyz="-0.0" ixz="-0.0"/>
+  </inertial>
+  <visual>
+    <origin xyz="-0.13 -0.060191 -0.529761" rpy="0 0 0"/>
+    <geometry>
+      <mesh filename="file://$(find mycobot320_description)/meshes/link6_1.stl" scale="0.001 0.001 0.001"/>
+    </geometry>
+    <material name="silver"/>
+  </visual>
+  <collision>
+    <origin xyz="-0.13 -0.060191 -0.529761" rpy="0 0 0"/>
+    <geometry>
+      <mesh filename="file://$(find mycobot320_description)/meshes/link6_1.stl" scale="0.001 0.001 0.001"/>
+    </geometry>
+  </collision>
+</link>
+<link name="gripper_right2_1">
+  <inertial>
+    <origin xyz="0.03379863281685422 0.02246224440899991 0.002360087014586343" rpy="0 0 0"/>
+    <mass value="0.05940572970223046"/>
+    <inertia ixx="6e-06" iyy="1.8e-05" izz="2.1e-05" ixy="-7e-06" iyz="-1e-06" ixz="-2e-06"/>
+  </inertial>
+  <visual>
+    <origin xyz="-0.188135 -0.10458 -0.524876" rpy="0 0 0"/>
+    <geometry>
+      <mesh filename="file://$(find mycobot320_description)/meshes/gripper_right2_1.stl" scale="0.001 0.001 0.001"/>
+    </geometry>
+    <material name="silver"/>
+  </visual>
+  <collision>
+    <origin xyz="-0.188135 -0.10458 -0.524876" rpy="0 0 0"/>
+    <geometry>
+      <mesh filename="file://$(find mycobot320_description)/meshes/gripper_right2_1.stl" scale="0.001 0.001 0.001"/>
+    </geometry>
+  </collision>
+</link>
+<link name="gripper_right3_1">
+  <inertial>
+    <origin xyz="0.015740982452355473 0.01214544458691133 -0.0033499396529518277" rpy="0 0 0"/>
+    <mass value="0.08857210300231066"/>
+    <inertia ixx="1.6e-05" iyy="3.3e-05" izz="4.8e-05" ixy="-1.6e-05" iyz="-0.0" ixz="-0.0"/>
+  </inertial>
+  <visual>
+    <origin xyz="-0.2105 -0.078518 -0.540192" rpy="0 0 0"/>
+    <geometry>
+      <mesh filename="file://$(find mycobot320_description)/meshes/gripper_right3_1.stl" scale="0.001 0.001 0.001"/>
+    </geometry>
+    <material name="silver"/>
+  </visual>
+  <collision>
+    <origin xyz="-0.2105 -0.078518 -0.540192" rpy="0 0 0"/>
+    <geometry>
+      <mesh filename="file://$(find mycobot320_description)/meshes/gripper_right3_1.stl" scale="0.001 0.001 0.001"/>
+    </geometry>
+  </collision>
+</link>
+<link name="gripper_left3_1">
+  <inertial>
+    <origin xyz="0.015692604770214447 -0.012149863481161281 -0.003642405326842235" rpy="0 0 0"/>
+    <mass value="0.08842063664845463"/>
+    <inertia ixx="1.6e-05" iyy="3.3e-05" izz="4.8e-05" ixy="1.6e-05" iyz="-0.0" ixz="0.0"/>
+  </inertial>
+  <visual>
+    <origin xyz="-0.2105 -0.041878 -0.540214" rpy="0 0 0"/>
+    <geometry>
+      <mesh filename="file://$(find mycobot320_description)/meshes/gripper_left3_1.stl" scale="0.001 0.001 0.001"/>
+    </geometry>
+    <material name="silver"/>
+  </visual>
+  <collision>
+    <origin xyz="-0.2105 -0.041878 -0.540214" rpy="0 0 0"/>
+    <geometry>
+      <mesh filename="file://$(find mycobot320_description)/meshes/gripper_left3_1.stl" scale="0.001 0.001 0.001"/>
+    </geometry>
+  </collision>
+</link>
+<link name="gripper_left2_1">
+  <inertial>
+    <origin xyz="0.03246595180129555 -0.022600862626259127 -9.99896592168703e-06" rpy="0 0 0"/>
+    <mass value="0.055976918228274164"/>
+    <inertia ixx="6e-06" iyy="1.6e-05" izz="2e-05" ixy="7e-06" iyz="1e-06" ixz="-2e-06"/>
+  </inertial>
+  <visual>
+    <origin xyz="-0.188135 -0.015798 -0.52743" rpy="0 0 0"/>
+    <geometry>
+      <mesh filename="file://$(find mycobot320_description)/meshes/gripper_left2_1.stl" scale="0.001 0.001 0.001"/>
+    </geometry>
+    <material name="silver"/>
+  </visual>
+  <collision>
+    <origin xyz="-0.188135 -0.015798 -0.52743" rpy="0 0 0"/>
+    <geometry>
+      <mesh filename="file://$(find mycobot320_description)/meshes/gripper_left2_1.stl" scale="0.001 0.001 0.001"/>
+    </geometry>
+  </collision>
+</link>
+<link name="gripper_base_1">
+  <inertial>
+    <origin xyz="0.041301491018273684 5.606290499195893e-05 -0.010030403559479484" rpy="0 0 0"/>
     <mass value="1.169410692896674"/>
-    <inertia ixx="0.000963" iyy="0.001227" izz="0.000961" ixy="-6.1e-05" iyz="0.0" ixz="1e-06"/>
-  </inertial>
-  <visual>
-    <origin xyz="-0.150006 -0.060982 -0.529047" rpy="0 0 0"/>
-    <geometry>
-      <mesh filename="file://$(find mycobot320_description)/meshes/gripper_base.stl" scale="0.001 0.001 0.001"/>
-    </geometry>
-    <material name="silver"/>
-  </visual>
-  <collision>
-    <origin xyz="-0.150006 -0.060982 -0.529047" rpy="0 0 0"/>
-    <geometry>
-      <mesh filename="file://$(find mycobot320_description)/meshes/gripper_base.stl" scale="0.001 0.001 0.001"/>
-    </geometry>
-  </collision>
-</link>
-<link name="gripper_right3">
-  <inertial>
-    <origin xyz="0.019897445301458788 0.003328334846588371 -0.0008618172580167061" rpy="0 0 0"/>
-    <mass value="0.0884342899427992"/>
-    <inertia ixx="7e-06" iyy="4.8e-05" izz="4.2e-05" ixy="0.0" iyz="-0.0" ixz="6e-06"/>
-  </inertial>
-  <visual>
-    <origin xyz="-0.210547 -0.050521 -0.547218" rpy="0 0 0"/>
-    <geometry>
-      <mesh filename="file://$(find mycobot320_description)/meshes/gripper_right3.stl" scale="0.001 0.001 0.001"/>
-    </geometry>
-    <material name="silver"/>
-  </visual>
-  <collision>
-    <origin xyz="-0.210547 -0.050521 -0.547218" rpy="0 0 0"/>
-    <geometry>
-      <mesh filename="file://$(find mycobot320_description)/meshes/gripper_right3.stl" scale="0.001 0.001 0.001"/>
-    </geometry>
-  </collision>
-</link>
-<link name="gripper_right1">
-  <inertial>
-    <origin xyz="0.011640592022952256 0.003586474602388895 0.005141940843472637" rpy="0 0 0"/>
-    <mass value="0.09086983402456465"/>
-    <inertia ixx="1e-05" iyy="4e-05" izz="3.3e-05" ixy="-0.0" iyz="0.0" ixz="1.2e-05"/>
-  </inertial>
-  <visual>
-    <origin xyz="-0.269552 -0.050353 -0.537954" rpy="0 0 0"/>
-    <geometry>
-      <mesh filename="file://$(find mycobot320_description)/meshes/gripper_right1.stl" scale="0.001 0.001 0.001"/>
-    </geometry>
-    <material name="silver"/>
-  </visual>
-  <collision>
-    <origin xyz="-0.269552 -0.050353 -0.537954" rpy="0 0 0"/>
-    <geometry>
-      <mesh filename="file://$(find mycobot320_description)/meshes/gripper_right1.stl" scale="0.001 0.001 0.001"/>
-    </geometry>
-  </collision>
-</link>
-<link name="gripper_right2">
-  <inertial>
-    <origin xyz="0.039252999761462265 -0.00016291284147181007 -0.004528228598043582" rpy="0 0 0"/>
-    <mass value="0.05677395712192003"/>
-    <inertia ixx="3e-06" iyy="2e-05" izz="1.9e-05" ixy="2e-06" iyz="-0.0" ixz="4e-06"/>
-  </inertial>
-  <visual>
-    <origin xyz="-0.188253 -0.063338 -0.573343" rpy="0 0 0"/>
-    <geometry>
-      <mesh filename="file://$(find mycobot320_description)/meshes/gripper_right2.stl" scale="0.001 0.001 0.001"/>
-    </geometry>
-    <material name="silver"/>
-  </visual>
-  <collision>
-    <origin xyz="-0.188253 -0.063338 -0.573343" rpy="0 0 0"/>
-    <geometry>
-      <mesh filename="file://$(find mycobot320_description)/meshes/gripper_right2.stl" scale="0.001 0.001 0.001"/>
-    </geometry>
-  </collision>
-</link>
-<link name="gripper_left3">
-  <inertial>
-    <origin xyz="0.019874922365214265 0.0032052020362376143 0.0010863693067071356" rpy="0 0 0"/>
-    <mass value="0.08829596207620957"/>
-    <inertia ixx="7e-06" iyy="4.8e-05" izz="4.2e-05" ixy="-0.0" iyz="-0.0" ixz="-6e-06"/>
-  </inertial>
-  <visual>
-    <origin xyz="-0.210455 -0.05051 -0.510579" rpy="0 0 0"/>
-    <geometry>
-      <mesh filename="file://$(find mycobot320_description)/meshes/gripper_left3.stl" scale="0.001 0.001 0.001"/>
-    </geometry>
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