Commit message: 1

File: mycobot111_description/urdf/mycobot111.xacro (robot description, xacro)
@@ -26,7 +26,7 @@
 <link name="link1_1">
   <inertial>
-    <origin xyz="0.0068967662247303866 4.702325320090434e-17 0.055490186869056476" rpy="0 0 0"/>
+    <origin xyz="0.006896766224730428 4.7445558334983536e-17 0.055490186869056476" rpy="0 0 0"/>
     <mass value="3.4735206294395446"/>
-    <inertia ixx="0.004461" iyy="0.004757" izz="0.002424" ixy="0.0" iyz="0.0" ixz="-0.000777"/>
+    <inertia ixx="0.004461" iyy="0.004757" izz="0.002424" ixy="-0.0" iyz="0.0" ixz="-0.000777"/>
   </inertial>
   <visual>
