Commit message: change gripper tf

File: mycobot_description/urdf/mycobot.xacro (robot description, xacro)
@@ -24,14 +24,14 @@
   </collision>
 </link>
-<link name="link1">
-  <inertial>
-    <origin xyz="0.006896766224730391 -3.4711337724979696e-07 0.05549014255068621" rpy="0 0 0"/>
+<link name="link1_1">
+  <inertial>
+    <origin xyz="1.7818903264329774e-17 -0.006897113338107677 0.05549014255068621" rpy="0 0 0"/>
     <mass value="3.4735206294395446"/>
-    <inertia ixx="0.004461" iyy="0.004757" izz="0.002424" ixy="0.0" iyz="-0.0" ixz="-0.000777"/>
+    <inertia ixx="0.004757" iyy="0.004461" izz="0.002424" ixy="-0.0" iyz="0.000777" ixz="0.0"/>
   </inertial>
   <visual>
     <origin xyz="0.0 -0.060072 -0.114761" rpy="0 0 0"/>
     <geometry>
-      <mesh filename="file://$(find mycobot_description)/meshes/link1.stl" scale="0.001 0.001 0.001"/>
+      <mesh filename="file://$(find mycobot_description)/meshes/link1_1.stl" scale="0.001 0.001 0.001"/>
     </geometry>
     <material name="silver"/>
@@ -40,338 +40,406 @@
     <origin xyz="0.0 -0.060072 -0.114761" rpy="0 0 0"/>
     <geometry>
-      <mesh filename="file://$(find mycobot_description)/meshes/link1.stl" scale="0.001 0.001 0.001"/>
-    </geometry>
-  </collision>
-</link>
-<link name="link2">
-  <inertial>
-    <origin xyz="0.03690658575567238 -3.4711337713183577e-07 0.06799995568162978" rpy="0 0 0"/>
+      <mesh filename="file://$(find mycobot_description)/meshes/link1_1.stl" scale="0.001 0.001 0.001"/>
+    </geometry>
+  </collision>
+</link>
+<link name="link2_1">
+  <inertial>
+    <origin xyz="3.6106292522153246e-16 -0.03690693286904952 0.06799995568162978" rpy="0 0 0"/>
     <mass value="5.91988968680626"/>
-    <inertia ixx="0.0188" iyy="0.019335" izz="0.004161" ixy="0.0" iyz="0.0" ixz="0.0"/>
-  </inertial>
-  <visual>
-    <origin xyz="-0.045 -0.060072 -0.199761" rpy="0 0 0"/>
-    <geometry>
-      <mesh filename="file://$(find mycobot_description)/meshes/link2.stl" scale="0.001 0.001 0.001"/>
-    </geometry>
-    <material name="silver"/>
-  </visual>
-  <collision>
-    <origin xyz="-0.045 -0.060072 -0.199761" rpy="0 0 0"/>
-    <geometry>
-      <mesh filename="file://$(find mycobot_description)/meshes/link2.stl" scale="0.001 0.001 0.001"/>
-    </geometry>
-  </collision>
-</link>
-<link name="link3">
-  <inertial>
-    <origin xyz="-0.03502268825299208 -3.4711337702081346e-07 0.049499955681629404" rpy="0 0 0"/>
+    <inertia ixx="0.019335" iyy="0.0188" izz="0.004161" ixy="-0.0" iyz="-0.0" ixz="-0.0"/>
+  </inertial>
+  <visual>
+    <origin xyz="-0.0 -0.015072 -0.199761" rpy="0 0 0"/>
+    <geometry>
+      <mesh filename="file://$(find mycobot_description)/meshes/link2_1.stl" scale="0.001 0.001 0.001"/>
+    </geometry>
+    <material name="silver"/>
+  </visual>
+  <collision>
+    <origin xyz="-0.0 -0.015072 -0.199761" rpy="0 0 0"/>
+    <geometry>
+      <mesh filename="file://$(find mycobot_description)/meshes/link2_1.stl" scale="0.001 0.001 0.001"/>
+    </geometry>
+  </collision>
+</link>
+<link name="link3_1">
+  <inertial>
+    <origin xyz="4.97742590851401e-16 0.035022341139615054 0.04949995568162946" rpy="0 0 0"/>
     <mass value="4.802107093668197"/>
-    <inertia ixx="0.01014" iyy="0.010584" izz="0.003386" ixy="0.0" iyz="-0.0" ixz="0.0"/>
-  </inertial>
-  <visual>
-    <origin xyz="-0.045 -0.060072 -0.335761" rpy="0 0 0"/>
-    <geometry>
-      <mesh filename="file://$(find mycobot_description)/meshes/link3.stl" scale="0.001 0.001 0.001"/>
-    </geometry>
-    <material name="silver"/>
-  </visual>
-  <collision>
-    <origin xyz="-0.045 -0.060072 -0.335761" rpy="0 0 0"/>
-    <geometry>
-      <mesh filename="file://$(find mycobot_description)/meshes/link3.stl" scale="0.001 0.001 0.001"/>
-    </geometry>
-  </collision>
-</link>
-<link name="link4">
-  <inertial>
-    <origin xyz="0.03442387286919234 -3.4711337690979116e-07 0.010576082812437049" rpy="0 0 0"/>
+    <inertia ixx="0.010584" iyy="0.01014" izz="0.003386" ixy="-0.0" iyz="-0.0" ixz="-0.0"/>
+  </inertial>
+  <visual>
+    <origin xyz="-0.0 -0.015072 -0.335761" rpy="0 0 0"/>
+    <geometry>
+      <mesh filename="file://$(find mycobot_description)/meshes/link3_1.stl" scale="0.001 0.001 0.001"/>
+    </geometry>
+    <material name="silver"/>
+  </visual>
+  <collision>
+    <origin xyz="-0.0 -0.015072 -0.335761" rpy="0 0 0"/>
+    <geometry>
+      <mesh filename="file://$(find mycobot_description)/meshes/link3_1.stl" scale="0.001 0.001 0.001"/>
+    </geometry>
+  </collision>
+</link>
+<link name="link4_1">
+  <inertial>
+    <origin xyz="-0.010576127130807278 -0.0344242199825693 -4.431837047347287e-08" rpy="0 0 0"/>
     <mass value="2.265107015236222"/>
-    <inertia ixx="0.001595" iyy="0.001803" izz="0.001595" ixy="0.0" iyz="0.0" ixz="-0.000324"/>
-  </inertial>
-  <visual>
-    <origin xyz="-0.045 -0.060072 -0.434761" rpy="0 0 0"/>
-    <geometry>
-      <mesh filename="file://$(find mycobot_description)/meshes/link4.stl" scale="0.001 0.001 0.001"/>
-    </geometry>
-    <material name="silver"/>
-  </visual>
-  <collision>
-    <origin xyz="-0.045 -0.060072 -0.434761" rpy="0 0 0"/>
-    <geometry>
-      <mesh filename="file://$(find mycobot_description)/meshes/link4.stl" scale="0.001 0.001 0.001"/>
-    </geometry>
-  </collision>
-</link>
-<link name="link5">
-  <inertial>
-    <origin xyz="6.938893903907228e-17 -3.4711337680570775e-07 0.04211665218776295" rpy="0 0 0"/>
+    <inertia ixx="0.001595" iyy="0.001595" izz="0.001803" ixy="-0.000324" iyz="0.0" ixz="0.0"/>
+  </inertial>
+  <visual>
+    <origin xyz="-0.0 -0.015072 -0.434761" rpy="0 0 0"/>
+    <geometry>
+      <mesh filename="file://$(find mycobot_description)/meshes/link4_1.stl" scale="0.001 0.001 0.001"/>
+    </geometry>
+    <material name="silver"/>
+  </visual>
+  <collision>
+    <origin xyz="-0.0 -0.015072 -0.434761" rpy="0 0 0"/>
+    <geometry>
+      <mesh filename="file://$(find mycobot_description)/meshes/link4_1.stl" scale="0.001 0.001 0.001"/>
+    </geometry>
+  </collision>
+</link>
+<link name="link5_1">
+  <inertial>
+    <origin xyz="-0.04211669650613323 -3.4711337686468835e-07 -4.431837019591711e-08" rpy="0 0 0"/>
     <mass value="3.029827579494103"/>
-    <inertia ixx="0.0025" iyy="0.002976" izz="0.002441" ixy="0.0" iyz="-0.0" ixz="-0.0"/>
-  </inertial>
-  <visual>
-    <origin xyz="-0.09 -0.060072 -0.479761" rpy="0 0 0"/>
-    <geometry>
-      <mesh filename="file://$(find mycobot_description)/meshes/link5.stl" scale="0.001 0.001 0.001"/>
-    </geometry>
-    <material name="silver"/>
-  </visual>
-  <collision>
-    <origin xyz="-0.09 -0.060072 -0.479761" rpy="0 0 0"/>
-    <geometry>
-      <mesh filename="file://$(find mycobot_description)/meshes/link5.stl" scale="0.001 0.001 0.001"/>
-    </geometry>
-  </collision>
-</link>
-<link name="link6">
-  <inertial>
-    <origin xyz="0.010000000000000092 -3.471133767779522e-07 -4.4318370751028624e-08" rpy="0 0 0"/>
+    <inertia ixx="0.002441" iyy="0.002976" izz="0.0025" ixy="-0.0" iyz="0.0" ixz="-0.0"/>
+  </inertial>
+  <visual>
+    <origin xyz="0.045 0.029928 -0.434761" rpy="0 0 0"/>
+    <geometry>
+      <mesh filename="file://$(find mycobot_description)/meshes/link5_1.stl" scale="0.001 0.001 0.001"/>
+    </geometry>
+    <material name="silver"/>
+  </visual>
+  <collision>
+    <origin xyz="0.045 0.029928 -0.434761" rpy="0 0 0"/>
+    <geometry>
+      <mesh filename="file://$(find mycobot_description)/meshes/link5_1.stl" scale="0.001 0.001 0.001"/>
+    </geometry>
+  </collision>
+</link>
+<link name="link6_1">
+  <inertial>
+    <origin xyz="1.0130785099704553e-15 -3.4711337656284647e-07 0.009999955681629924" rpy="0 0 0"/>
     <mass value="0.6042068071016569"/>
-    <inertia ixx="0.00037" iyy="0.000205" izz="0.000205" ixy="0.0" iyz="0.0" ixz="0.0"/>
-  </inertial>
-  <visual>
-    <origin xyz="-0.13 -0.060072 -0.529761" rpy="0 0 0"/>
-    <geometry>
-      <mesh filename="file://$(find mycobot_description)/meshes/link6.stl" scale="0.001 0.001 0.001"/>
-    </geometry>
-    <material name="silver"/>
-  </visual>
-  <collision>
-    <origin xyz="-0.13 -0.060072 -0.529761" rpy="0 0 0"/>
-    <geometry>
-      <mesh filename="file://$(find mycobot_description)/meshes/link6.stl" scale="0.001 0.001 0.001"/>
-    </geometry>
-  </collision>
-</link>
-<link name="gripper_left1">
-  <inertial>
-    <origin xyz="0.011053321311780717 -0.005254043045734549 0.00013658058489207647" rpy="0 0 0"/>
-    <mass value="0.09307370524691046"/>
-    <inertia ixx="1e-05" iyy="3.5e-05" izz="4.2e-05" ixy="-1.3e-05" iyz="0.0" ixz="0.0"/>
-  </inertial>
-  <visual>
-    <origin xyz="-0.261438 -0.008607 -0.536903" rpy="0 0 0"/>
-    <geometry>
-      <mesh filename="file://$(find mycobot_description)/meshes/gripper_left1.stl" scale="0.001 0.001 0.001"/>
-    </geometry>
-    <material name="silver"/>
-  </visual>
-  <collision>
-    <origin xyz="-0.261438 -0.008607 -0.536903" rpy="0 0 0"/>
-    <geometry>
-      <mesh filename="file://$(find mycobot_description)/meshes/gripper_left1.stl" scale="0.001 0.001 0.001"/>
-    </geometry>
-  </collision>
-</link>
-<link name="gripper_right1">
-  <inertial>
-    <origin xyz="0.011064486332764245 0.00525722808018074 0.003559949036713861" rpy="0 0 0"/>
-    <mass value="0.0929857868716481"/>
-    <inertia ixx="1e-05" iyy="3.5e-05" izz="4.2e-05" ixy="1.3e-05" iyz="0.0" ixz="-0.0"/>
-  </inertial>
-  <visual>
-    <origin xyz="-0.261438 -0.111297 -0.533501" rpy="0 0 0"/>
-    <geometry>
-      <mesh filename="file://$(find mycobot_description)/meshes/gripper_right1.stl" scale="0.001 0.001 0.001"/>
-    </geometry>
-    <material name="silver"/>
-  </visual>
-  <collision>
-    <origin xyz="-0.261438 -0.111297 -0.533501" rpy="0 0 0"/>
-    <geometry>
-      <mesh filename="file://$(find mycobot_description)/meshes/gripper_right1.stl" scale="0.001 0.001 0.001"/>
-    </geometry>
-  </collision>
-</link>
-<link name="gripper_left3">
-  <inertial>
-    <origin xyz="0.01599044289886639 -0.012967874127836797 0.003475371537171479" rpy="0 0 0"/>
+    <inertia ixx="0.000205" iyy="0.000205" izz="0.00037" ixy="0.0" iyz="0.0" ixz="0.0"/>
+  </inertial>
+  <visual>
+    <origin xyz="0.095 0.029928 -0.474761" rpy="0 0 0"/>
+    <geometry>
+      <mesh filename="file://$(find mycobot_description)/meshes/link6_1.stl" scale="0.001 0.001 0.001"/>
+    </geometry>
+    <material name="silver"/>
+  </visual>
+  <collision>
+    <origin xyz="0.095 0.029928 -0.474761" rpy="0 0 0"/>
+    <geometry>
+      <mesh filename="file://$(find mycobot_description)/meshes/link6_1.stl" scale="0.001 0.001 0.001"/>
+    </geometry>
+  </collision>
+</link>
+<link name="gripper_left1_1">
+  <inertial>
+    <origin xyz="-0.0001366249032619532 -0.005254043045734361 0.011053276993410743" rpy="0 0 0"/>
+    <mass value="0.09307370524691048"/>
+    <inertia ixx="4.2e-05" iyy="3.5e-05" izz="1e-05" ixy="-0.0" iyz="-1.3e-05" ixz="-0.0"/>
+  </inertial>
+  <visual>
+    <origin xyz="0.102142 0.081393 -0.613499" rpy="0 0 0"/>
+    <geometry>
+      <mesh filename="file://$(find mycobot_description)/meshes/gripper_left1_1.stl" scale="0.001 0.001 0.001"/>
+    </geometry>
+    <material name="silver"/>
+  </visual>
+  <collision>
+    <origin xyz="0.102142 0.081393 -0.613499" rpy="0 0 0"/>
+    <geometry>
+      <mesh filename="file://$(find mycobot_description)/meshes/gripper_left1_1.stl" scale="0.001 0.001 0.001"/>
+    </geometry>
+  </collision>
+</link>
+<link name="gripper_right1_1">
+  <inertial>
+    <origin xyz="-0.003559993355084029 0.0052572280801808785 0.01106444201439416" rpy="0 0 0"/>
+    <mass value="0.09298578687164809"/>
+    <inertia ixx="4.2e-05" iyy="3.5e-05" izz="1e-05" ixy="-0.0" iyz="1.3e-05" ixz="0.0"/>
+  </inertial>
+  <visual>
+    <origin xyz="0.09874 -0.021297 -0.613499" rpy="0 0 0"/>
+    <geometry>
+      <mesh filename="file://$(find mycobot_description)/meshes/gripper_right1_1.stl" scale="0.001 0.001 0.001"/>
+    </geometry>
+    <material name="silver"/>
+  </visual>
+  <collision>
+    <origin xyz="0.09874 -0.021297 -0.613499" rpy="0 0 0"/>
+    <geometry>
+      <mesh filename="file://$(find mycobot_description)/meshes/gripper_right1_1.stl" scale="0.001 0.001 0.001"/>
+    </geometry>
+  </collision>
+</link>
+<link name="gripper_left3_1">
+  <inertial>
+    <origin xyz="-0.0034754158555415915 -0.012967874127836669 0.015990398580496223" rpy="0 0 0"/>
     <mass value="0.09059526730883062"/>
-    <inertia ixx="1.8e-05" iyy="3.3e-05" izz="5e-05" ixy="1.8e-05" iyz="0.0" ixz="-0.0"/>
-  </inertial>
-  <visual>
-    <origin xyz="-0.21039 -0.041612 -0.533403" rpy="0 0 0"/>
-    <geometry>
-      <mesh filename="file://$(find mycobot_description)/meshes/gripper_left3.stl" scale="0.001 0.001 0.001"/>
-    </geometry>
-    <material name="silver"/>
-  </visual>
-  <collision>
-    <origin xyz="-0.21039 -0.041612 -0.533403" rpy="0 0 0"/>
-    <geometry>
-      <mesh filename="file://$(find mycobot_description)/meshes/gripper_left3.stl" scale="0.001 0.001 0.001"/>
-    </geometry>
-  </collision>
-</link>
-<link name="gripper_right3">
-  <inertial>
-    <origin xyz="0.015989588845322006 0.012966613242614375 0.0035542257609944006" rpy="0 0 0"/>
+    <inertia ixx="5e-05" iyy="3.3e-05" izz="1.8e-05" ixy="-0.0" iyz="1.8e-05" ixz="0.0"/>
+  </inertial>
+  <visual>
+    <origin xyz="0.098642 0.048388 -0.562451" rpy="0 0 0"/>
+    <geometry>
+      <mesh filename="file://$(find mycobot_description)/meshes/gripper_left3_1.stl" scale="0.001 0.001 0.001"/>
+    </geometry>
+    <material name="silver"/>
+  </visual>
+  <collision>
+    <origin xyz="0.098642 0.048388 -0.562451" rpy="0 0 0"/>
+    <geometry>
+      <mesh filename="file://$(find mycobot_description)/meshes/gripper_left3_1.stl" scale="0.001 0.001 0.001"/>
+    </geometry>
+  </collision>
+</link>
+<link name="gripper_right3_1">
+  <inertial>
+    <origin xyz="-0.003554270079364527 0.012966613242614462 0.015989544526951893" rpy="0 0 0"/>
     <mass value="0.09058559783383588"/>
-    <inertia ixx="1.8e-05" iyy="3.3e-05" izz="5e-05" ixy="-1.8e-05" iyz="-0.0" ixz="-0.0"/>
-  </inertial>
-  <visual>
-    <origin xyz="-0.21039 -0.078292 -0.533403" rpy="0 0 0"/>
-    <geometry>
-      <mesh filename="file://$(find mycobot_description)/meshes/gripper_right3.stl" scale="0.001 0.001 0.001"/>
-    </geometry>
-    <material name="silver"/>
-  </visual>
-  <collision>
-    <origin xyz="-0.21039 -0.078292 -0.533403" rpy="0 0 0"/>
-    <geometry>
-      <mesh filename="file://$(find mycobot_description)/meshes/gripper_right3.stl" scale="0.001 0.001 0.001"/>
-    </geometry>
-  </collision>
-</link>
-<!-- <link name="gripper_right2">
-  <inertial>
-    <origin xyz="0.029939990495379626 0.020889826569869555 -0.00039518056690335257" rpy="0 0 0"/>
-    <mass value="0.05227728599311408"/>
-    <inertia ixx="6e-06" iyy="1.6e-05" izz="2e-05" ixy="-8e-06" iyz="-1e-06" ixz="-1e-06"/>
-  </inertial>
-  <visual>
-    <origin xyz="-0.188075 -0.104364 -0.526413" rpy="0 0 0"/>
-    <geometry>
-      <mesh filename="file://$(find mycobot_description)/meshes/gripper_right2.stl" scale="0.001 0.001 0.001"/>
-    </geometry>
-    <material name="silver"/>
-  </visual>
-  <collision>
-    <origin xyz="-0.188075 -0.104364 -0.526413" rpy="0 0 0"/>
-    <geometry>
-      <mesh filename="file://$(find mycobot_description)/meshes/gripper_right2.stl" scale="0.001 0.001 0.001"/>
-    </geometry>
-  </collision>
-</link> -->
-<!-- <link name="gripper_left2">
-  <inertial>
-    <origin xyz="0.03183851476317609 -0.022109126086089934 0.0008827048100953361" rpy="0 0 0"/>
-    <mass value="0.05612369952823833"/>
-    <inertia ixx="6e-06" iyy="1.7e-05" izz="2.1e-05" ixy="8e-06" iyz="1e-06" ixz="-2e-06"/>
-  </inertial>
-  <visual>
-    <origin xyz="-0.188075 -0.01558 -0.525913" rpy="0 0 0"/>
-    <geometry>
-      <mesh filename="file://$(find mycobot_description)/meshes/gripper_left2.stl" scale="0.001 0.001 0.001"/>
-    </geometry>
-    <material name="silver"/>
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