Commit message: edit mycobot_description
edit urdf(joint limits, mimic, rpy)

File: mycobot_description/urdf/mycobot.xacro (robot description, xacro)
@@ -2,6 +2,6 @@
 <robot name="mycobot" xmlns:xacro="http://www.ros.org/wiki/xacro">
 <xacro:include filename="$(find mycobot_description)/urdf/materials.xacro" />
-<xacro:include filename="$(find mycobot_description)/urdf/mycobot.trans" />
-<xacro:include filename="$(find mycobot_description)/urdf/mycobot.gazebo" />
+<!-- <xacro:include filename="$(find mycobot_description)/urdf/mycobot.trans" />
+<xacro:include filename="$(find mycobot_description)/urdf/mycobot.gazebo" /> -->
 <link name="base_link">
   <inertial>
@@ -24,5 +24,5 @@
   </collision>
 </link>
-<link name="link1_1">
+<link name="link1">
   <inertial>
     <origin xyz="0.006896766224730428 4.7445558334983536e-17 0.055490186869056476" rpy="0 0 0"/>
@@ -33,5 +33,5 @@
     <origin xyz="-0.0 -0.0 -0.11" rpy="0 0 0"/>
     <geometry>
-      <mesh filename="file://$(find mycobot_description)/meshes/link1_1.stl" scale="0.001 0.001 0.001"/>
+      <mesh filename="file://$(find mycobot_description)/meshes/link1.stl" scale="0.001 0.001 0.001"/>
     </geometry>
     <material name="silver"/>
@@ -40,9 +40,9 @@
     <origin xyz="-0.0 -0.0 -0.11" rpy="0 0 0"/>
     <geometry>
-      <mesh filename="file://$(find mycobot_description)/meshes/link1_1.stl" scale="0.001 0.001 0.001"/>
-    </geometry>
-  </collision>
-</link>
-<link name="link2_1">
+      <mesh filename="file://$(find mycobot_description)/meshes/link1.stl" scale="0.001 0.001 0.001"/>
+    </geometry>
+  </collision>
+</link>
+<link name="link2">
   <inertial>
     <origin xyz="0.03690658575567249 -1.0444649911926371e-16 0.06800000000000012" rpy="0 0 0"/>
@@ -53,5 +53,5 @@
     <origin xyz="-0.045 -0.0 -0.195" rpy="0 0 0"/>
     <geometry>
-      <mesh filename="file://$(find mycobot_description)/meshes/link2_1.stl" scale="0.001 0.001 0.001"/>
+      <mesh filename="file://$(find mycobot_description)/meshes/link2.stl" scale="0.001 0.001 0.001"/>
     </geometry>
     <material name="silver"/>
@@ -60,9 +60,9 @@
     <origin xyz="-0.045 -0.0 -0.195" rpy="0 0 0"/>
     <geometry>
-      <mesh filename="file://$(find mycobot_description)/meshes/link2_1.stl" scale="0.001 0.001 0.001"/>
-    </geometry>
-  </collision>
-</link>
-<link name="link3_1">
+      <mesh filename="file://$(find mycobot_description)/meshes/link2.stl" scale="0.001 0.001 0.001"/>
+    </geometry>
+  </collision>
+</link>
+<link name="link3">
   <inertial>
     <origin xyz="-0.035022688252992054 -8.56731250465993e-16 0.049500000000000155" rpy="0 0 0"/>
@@ -73,5 +73,5 @@
     <origin xyz="-0.045 0.0 -0.331" rpy="0 0 0"/>
     <geometry>
-      <mesh filename="file://$(find mycobot_description)/meshes/link3_1.stl" scale="0.001 0.001 0.001"/>
+      <mesh filename="file://$(find mycobot_description)/meshes/link3.stl" scale="0.001 0.001 0.001"/>
     </geometry>
     <material name="silver"/>
@@ -80,9 +80,9 @@
     <origin xyz="-0.045 0.0 -0.331" rpy="0 0 0"/>
     <geometry>
-      <mesh filename="file://$(find mycobot_description)/meshes/link3_1.stl" scale="0.001 0.001 0.001"/>
-    </geometry>
-  </collision>
-</link>
-<link name="link4_1">
+      <mesh filename="file://$(find mycobot_description)/meshes/link3.stl" scale="0.001 0.001 0.001"/>
+    </geometry>
+  </collision>
+</link>
+<link name="link4">
   <inertial>
     <origin xyz="0.03442387286919234 -1.62263567395975e-15 0.010576127130807855" rpy="0 0 0"/>
@@ -93,5 +93,5 @@
     <origin xyz="-0.045 0.0 -0.43" rpy="0 0 0"/>
     <geometry>
-      <mesh filename="file://$(find mycobot_description)/meshes/link4_1.stl" scale="0.001 0.001 0.001"/>
+      <mesh filename="file://$(find mycobot_description)/meshes/link4.stl" scale="0.001 0.001 0.001"/>
     </geometry>
     <material name="silver"/>
@@ -100,9 +100,9 @@
     <origin xyz="-0.045 0.0 -0.43" rpy="0 0 0"/>
     <geometry>
-      <mesh filename="file://$(find mycobot_description)/meshes/link4_1.stl" scale="0.001 0.001 0.001"/>
-    </geometry>
-  </collision>
-</link>
-<link name="link5_1">
+      <mesh filename="file://$(find mycobot_description)/meshes/link4.stl" scale="0.001 0.001 0.001"/>
+    </geometry>
+  </collision>
+</link>
+<link name="link5">
   <inertial>
     <origin xyz="4.163336342344337e-17 -2.2870367877634065e-15 0.04211669650613381" rpy="0 0 0"/>
@@ -113,5 +113,5 @@
     <origin xyz="-0.09 0.0 -0.475" rpy="0 0 0"/>
     <geometry>
-      <mesh filename="file://$(find mycobot_description)/meshes/link5_1.stl" scale="0.001 0.001 0.001"/>
+      <mesh filename="file://$(find mycobot_description)/meshes/link5.stl" scale="0.001 0.001 0.001"/>
     </geometry>
     <material name="silver"/>
@@ -120,9 +120,9 @@
     <origin xyz="-0.09 0.0 -0.475" rpy="0 0 0"/>
     <geometry>
-      <mesh filename="file://$(find mycobot_description)/meshes/link5_1.stl" scale="0.001 0.001 0.001"/>
-    </geometry>
-  </collision>
-</link>
-<link name="link6_1">
+      <mesh filename="file://$(find mycobot_description)/meshes/link5.stl" scale="0.001 0.001 0.001"/>
+    </geometry>
+  </collision>
+</link>
+<link name="link6">
   <inertial>
     <origin xyz="0.010000000000000009 -2.29263991248323e-15 0.0" rpy="0 0 0"/>
@@ -133,5 +133,5 @@
     <origin xyz="-0.13 0.0 -0.525" rpy="0 0 0"/>
     <geometry>
-      <mesh filename="file://$(find mycobot_description)/meshes/link6_1.stl" scale="0.001 0.001 0.001"/>
+      <mesh filename="file://$(find mycobot_description)/meshes/link6.stl" scale="0.001 0.001 0.001"/>
     </geometry>
     <material name="silver"/>
@@ -140,9 +140,9 @@
     <origin xyz="-0.13 0.0 -0.525" rpy="0 0 0"/>
     <geometry>
-      <mesh filename="file://$(find mycobot_description)/meshes/link6_1.stl" scale="0.001 0.001 0.001"/>
-    </geometry>
-  </collision>
-</link>
-<link name="gripper_base_1">
+      <mesh filename="file://$(find mycobot_description)/meshes/link6.stl" scale="0.001 0.001 0.001"/>
+    </geometry>
+  </collision>
+</link>
+<link name="gripper_base">
   <inertial>
     <origin xyz="0.0355664843149987 -0.0001756055492085692 0.008326821944589002" rpy="0 0 0"/>
@@ -153,5 +153,5 @@
     <origin xyz="-0.15 0.0 -0.525" rpy="0 0 0"/>
     <geometry>
-      <mesh filename="file://$(find mycobot_description)/meshes/gripper_base_1.stl" scale="0.001 0.001 0.001"/>
+      <mesh filename="file://$(find mycobot_description)/meshes/gripper_base.stl" scale="0.001 0.001 0.001"/>
     </geometry>
     <material name="silver"/>
@@ -160,9 +160,9 @@
     <origin xyz="-0.15 0.0 -0.525" rpy="0 0 0"/>
     <geometry>
-      <mesh filename="file://$(find mycobot_description)/meshes/gripper_base_1.stl" scale="0.001 0.001 0.001"/>
-    </geometry>
-  </collision>
-</link>
-<link name="gripper_right3_1">
+      <mesh filename="file://$(find mycobot_description)/meshes/gripper_base.stl" scale="0.001 0.001 0.001"/>
+    </geometry>
+  </collision>
+</link>
+<link name="gripper_right3">
   <inertial>
     <origin xyz="0.015989567569339613 0.012966960169895517 0.0035542407438502455" rpy="0 0 0"/>
@@ -173,5 +173,5 @@
     <origin xyz="-0.21039 -0.01822 -0.528642" rpy="0 0 0"/>
     <geometry>
-      <mesh filename="file://$(find mycobot_description)/meshes/gripper_right3_1.stl" scale="0.001 0.001 0.001"/>
+      <mesh filename="file://$(find mycobot_description)/meshes/gripper_right3.stl" scale="0.001 0.001 0.001"/>
     </geometry>
     <material name="silver"/>
@@ -180,9 +180,9 @@
     <origin xyz="-0.21039 -0.01822 -0.528642" rpy="0 0 0"/>
     <geometry>
-      <mesh filename="file://$(find mycobot_description)/meshes/gripper_right3_1.stl" scale="0.001 0.001 0.001"/>
-    </geometry>
-  </collision>
-</link>
-<link name="gripper_right1_1">
+      <mesh filename="file://$(find mycobot_description)/meshes/gripper_right3.stl" scale="0.001 0.001 0.001"/>
+    </geometry>
+  </collision>
+</link>
+<link name="gripper_right1">
   <inertial>
     <origin xyz="0.011064466442332721 0.005257573311972401 0.00355996955743465" rpy="0 0 0"/>
@@ -193,5 +193,5 @@
     <origin xyz="-0.261438 -0.051225 -0.52874" rpy="0 0 0"/>
     <geometry>
-      <mesh filename="file://$(find mycobot_description)/meshes/gripper_right1_1.stl" scale="0.001 0.001 0.001"/>
+      <mesh filename="file://$(find mycobot_description)/meshes/gripper_right1.stl" scale="0.001 0.001 0.001"/>
     </geometry>
     <material name="silver"/>
@@ -200,9 +200,9 @@
     <origin xyz="-0.261438 -0.051225 -0.52874" rpy="0 0 0"/>
     <geometry>
-      <mesh filename="file://$(find mycobot_description)/meshes/gripper_right1_1.stl" scale="0.001 0.001 0.001"/>
-    </geometry>
-  </collision>
-</link>
-<link name="gripper_left3_1">
+      <mesh filename="file://$(find mycobot_description)/meshes/gripper_right1.stl" scale="0.001 0.001 0.001"/>
+    </geometry>
+  </collision>
+</link>
+<link name="gripper_left3">
   <inertial>
     <origin xyz="0.0159904266297618 -0.012967523057109649 0.0034753903195801072" rpy="0 0 0"/>
@@ -213,5 +213,5 @@
     <origin xyz="-0.21039 0.01846 -0.528642" rpy="0 0 0"/>
     <geometry>
-      <mesh filename="file://$(find mycobot_description)/meshes/gripper_left3_1.stl" scale="0.001 0.001 0.001"/>
+      <mesh filename="file://$(find mycobot_description)/meshes/gripper_left3.stl" scale="0.001 0.001 0.001"/>
     </geometry>
     <material name="silver"/>
@@ -220,9 +220,9 @@
     <origin xyz="-0.21039 0.01846 -0.528642" rpy="0 0 0"/>
     <geometry>
-      <mesh filename="file://$(find mycobot_description)/meshes/gripper_left3_1.stl" scale="0.001 0.001 0.001"/>
-    </geometry>
-  </collision>
-</link>
-<link name="gripper_left1_1">
+      <mesh filename="file://$(find mycobot_description)/meshes/gripper_left3.stl" scale="0.001 0.001 0.001"/>
+    </geometry>
+  </collision>
+</link>
+<link name="gripper_left1">
   <inertial>
     <origin xyz="0.011053309239177689 -0.0052536917643599065 0.003636608039289002" rpy="0 0 0"/>
@@ -233,5 +233,5 @@
     <origin xyz="-0.261438 0.051465 -0.528642" rpy="0 0 0"/>
     <geometry>
-      <mesh filename="file://$(find mycobot_description)/meshes/gripper_left1_1.stl" scale="0.001 0.001 0.001"/>
+      <mesh filename="file://$(find mycobot_description)/meshes/gripper_left1.stl" scale="0.001 0.001 0.001"/>
     </geometry>
     <material name="silver"/>
@@ -240,5 +240,5 @@
     <origin xyz="-0.261438 0.051465 -0.528642" rpy="0 0 0"/>
     <geometry>
-      <mesh filename="file://$(find mycobot_description)/meshes/gripper_left1_1.stl" scale="0.001 0.001 0.001"/>
+      <mesh filename="file://$(find mycobot_description)/meshes/gripper_left1.stl" scale="0.001 0.001 0.001"/>
     </geometry>
   </collision>
@@ -248,5 +248,5 @@
   <origin xyz="0.0 0.0 0.11" rpy="0 0 0"/>
   <parent link="base_link"/>
-  <child link="link1_1"/>
+  <child link="link1"/>
   <axis xyz="0.0 0.0 1.0"/>
   <limit upper="2.792527" lower="-2.792527" effort="100" velocity="100"/>
@@ -254,6 +254,6 @@
 <joint name="joint2" type="revolute">
   <origin xyz="0.045 0.0 0.085" rpy="0 0 0"/>
-  <parent link="link1_1"/>
-  <child link="link2_1"/>
+  <parent link="link1"/>
+  <child link="link2"/>
   <axis xyz="1.0 0.0 0.0"/>
   <limit upper="2.792527" lower="-2.792527" effort="100" velocity="100"/>
@@ -261,6 +261,6 @@
 <joint name="joint3" type="revolute">
   <origin xyz="0.0 -0.0 0.136" rpy="0 0 0"/>
-  <parent link="link2_1"/>
-  <child link="link3_1"/>
+  <parent link="link2"/>
+  <child link="link3"/>
   <axis xyz="-1.0 -0.0 -0.0"/>
   <limit upper="2.792527" lower="-2.792527" effort="100" velocity="100"/>
@@ -268,6 +268,6 @@
 <joint name="joint4" type="revolute">
   <origin xyz="0.0 0.0 0.099" rpy="0 0 0"/>
-  <parent link="link3_1"/>
-  <child link="link4_1"/>
+  <parent link="link3"/>
+  <child link="link4"/>
   <axis xyz="1.0 -0.0 -0.0"/>
   <limit upper="2.792527" lower="-2.792527" effort="100" velocity="100"/>
@@ -275,6 +275,6 @@
 <joint name="joint5" type="revolute">
   <origin xyz="0.045 0.0 0.045" rpy="0 0 0"/>
-  <parent link="link4_1"/>
-  <child link="link5_1"/>
+  <parent link="link4"/>
+  <child link="link5"/>
   <axis xyz="-0.0 -0.0 1.0"/>
   <limit upper="2.792527" lower="-2.792527" effort="100" velocity="100"/>
@@ -282,6 +282,6 @@
 <joint name="joint6" type="revolute">
   <origin xyz="0.04 0.0 0.05" rpy="0 0 0"/>
-  <parent link="link5_1"/>
-  <child link="link6_1"/>
+  <parent link="link5"/>
+  <child link="link6"/>
   <axis xyz="1.0 0.0 0.0"/>
   <limit upper="2.792527" lower="-2.792527" effort="100" velocity="100"/>
@@ -289,34 +289,37 @@
 <joint name="gripper_base_to_link6" type="fixed">
   <origin xyz="0.02 0.0 0.0" rpy="0 0 0"/>
-  <parent link="link6_1"/>
-  <child link="gripper_base_1"/>
-</joint>
-<joint name="right3_to_base" type="revolute">
-  <origin xyz="0.06039 0.01822 0.003642" rpy="0 0 0"/>
-  <parent link="gripper_base_1"/>
-  <child link="gripper_right3_1"/>
+  <parent link="link6"/>
+  <child link="gripper_base"/>
+</joint>
+<joint name="gripper_controller" type="revolute">
+  <origin xyz="0.06039 0.01822 0.003642" rpy="0 0 -0.42"/> <!-- change rpy y to -0.42-->
+  <parent link="gripper_base"/>
+  <child link="gripper_right3"/>
   <axis xyz="0.0 0.0 -1.0"/>
-  <limit upper="0.698132" lower="0.0" effort="100" velocity="100"/>
-</joint>
-<joint name="right1_to_right3" type="revolute">
-  <origin xyz="0.051048 0.033005 9.8e-05" rpy="0 0 0"/>
-  <parent link="gripper_right3_1"/>
-  <child link="gripper_right1_1"/>
+  <limit upper="0.3" lower="-0.7" effort="100" velocity="100"/> <!-- change upper to 0.3 and lower to -0.7-->
+</joint>
+<joint name="gripper_right3_to_gripper_right1" type="revolute">
+  <origin xyz="0.051048 0.033005 9.8e-05" rpy="0 0 0.42"/> <!-- change rpy y to 0.42-->
+  <parent link="gripper_right3"/>
+  <child link="gripper_right1"/>
   <axis xyz="-0.0 -0.0 -1.0"/>
-  <limit upper="0.0" lower="-0.698132" effort="100" velocity="100"/>
-</joint>
-<joint name="left3_to_base" type="revolute">
-  <origin xyz="0.06039 -0.01846 0.003642" rpy="0 0 0"/>
-  <parent link="gripper_base_1"/>
-  <child link="gripper_left3_1"/>
+  <limit upper="0.7" lower="-0.3" effort="100" velocity="100"/> <!-- change upper to 0.7 and lower to -0.3-->
+  <mimic joint="gripper_controller" multiplier="-1" offset="0"/> <!-- add mimic and change multiplier to -1-->
+</joint>
+<joint name="gripper_base_to_gripper_left3" type="revolute">
+  <origin xyz="0.06039 -0.01846 0.003642" rpy="0 0 0.42"/> <!-- change rpy y to 0.42-->
+  <parent link="gripper_base"/>
+  <child link="gripper_left3"/>
   <axis xyz="0.0 0.0 -1.0"/>
-  <limit upper="0.0" lower="-0.698132" effort="100" velocity="100"/>
-</joint>
-<joint name="left1_to_left3" type="revolute">
-  <origin xyz="0.051048 -0.033005 0.0" rpy="0 0 0"/>
-  <parent link="gripper_left3_1"/>
-  <child link="gripper_left1_1"/>
+  <limit upper="0.7" lower="-0.3" effort="100" velocity="100"/> <!-- change upper to 0.7 and lower to -0.3-->
+  <mimic joint="gripper_controller" multiplier="-1" offset="0"/> <!-- add mimic and change multiplier to -1-->
+</joint>
+<joint name="gripper_left3_to_gripper_left1" type="revolute">
+  <origin xyz="0.051048 -0.033005 0.0" rpy="0 0 -0.42"/> <!-- change rpy y to -0.42-->
+  <parent link="gripper_left3"/>
+  <child link="gripper_left1"/>
   <axis xyz="-0.0 -0.0 -1.0"/>
-  <limit upper="0.698132" lower="0.0" effort="100" velocity="100"/>
+  <limit upper="0.3" lower="-0.7" effort="100" velocity="100"/> <!-- change upper to 0.3 and lower to -0.7-->
+  <mimic joint="gripper_controller" multiplier="1" offset="0"/> <!-- add mimic and change multiplier to 1-->
 </joint>
 </robot>
