Commit message: profile add

File: mycobot_description/urdf/mycobot.xacro (robot description, xacro)
@@ -2,324 +2,702 @@
 <robot name="mycobot" xmlns:xacro="http://www.ros.org/wiki/xacro">
 <xacro:include filename="$(find mycobot_description)/urdf/materials.xacro" />
-<!-- <xacro:include filename="$(find mycobot_description)/urdf/mycobot.trans" />
-<xacro:include filename="$(find mycobot_description)/urdf/mycobot.gazebo" /> -->
+<xacro:include filename="$(find mycobot_description)/urdf/mycobot.trans" />
+<xacro:include filename="$(find mycobot_description)/urdf/mycobot.gazebo" />
 <link name="base_link">
   <inertial>
-    <origin xyz="-1.3994637957346424e-08 -0.013751224256395762 0.04886454507234413" rpy="0 0 0"/>
+    <origin xyz="8.368053381880458e-07 -1.7610424648219707e-05 0.27252999856366134" rpy="0 0 0"/>
+    <mass value="8.34475627832778"/>
+    <inertia ixx="0.41971" iyy="0.457952" izz="0.39007" ixy="-1.6e-05" iyz="-2e-06" ixz="-0.0"/>
+  </inertial>
+  <visual>
+    <origin xyz="0 0 0" rpy="0 0 0"/>
+    <geometry>
+      <mesh filename="file://$(find mycobot_description)/meshes/base_link.stl" scale="0.001 0.001 0.001"/>
+    </geometry>
+    <material name="silver"/>
+  </visual>
+  <collision>
+    <origin xyz="0 0 0" rpy="0 0 0"/>
+    <geometry>
+      <mesh filename="file://$(find mycobot_description)/meshes/base_link.stl" scale="0.001 0.001 0.001"/>
+    </geometry>
+  </collision>
+</link>
+<link name="caster_3">
+  <inertial>
+    <origin xyz="-0.02857352949264516 -0.01151471005681412 -0.03043828110848307" rpy="0 0 0"/>
+    <mass value="0.18931422070235698"/>
+    <inertia ixx="5.5e-05" iyy="7.4e-05" izz="3.3e-05" ixy="-0.0" iyz="0.0" ixz="0.0"/>
+  </inertial>
+  <visual>
+    <origin xyz="-0.25 -0.2169 -0.058" rpy="0 0 0"/>
+    <geometry>
+      <mesh filename="file://$(find mycobot_description)/meshes/caster_3.stl" scale="0.001 0.001 0.001"/>
+    </geometry>
+    <material name="silver"/>
+  </visual>
+  <collision>
+    <origin xyz="-0.25 -0.2169 -0.058" rpy="0 0 0"/>
+    <geometry>
+      <mesh filename="file://$(find mycobot_description)/meshes/caster_3.stl" scale="0.001 0.001 0.001"/>
+    </geometry>
+  </collision>
+</link>
+<link name="caster_4">
+  <inertial>
+    <origin xyz="-0.028573529492625066 0.011514701707892594 -0.03043828110848334" rpy="0 0 0"/>
+    <mass value="0.18931422070235698"/>
+    <inertia ixx="5.5e-05" iyy="7.4e-05" izz="3.3e-05" ixy="-0.0" iyz="0.0" ixz="0.0"/>
+  </inertial>
+  <visual>
+    <origin xyz="-0.25 0.2169 -0.058" rpy="0 0 0"/>
+    <geometry>
+      <mesh filename="file://$(find mycobot_description)/meshes/caster_4.stl" scale="0.001 0.001 0.001"/>
+    </geometry>
+    <material name="silver"/>
+  </visual>
+  <collision>
+    <origin xyz="-0.25 0.2169 -0.058" rpy="0 0 0"/>
+    <geometry>
+      <mesh filename="file://$(find mycobot_description)/meshes/caster_4.stl" scale="0.001 0.001 0.001"/>
+    </geometry>
+  </collision>
+</link>
+<link name="caster_5">
+  <inertial>
+    <origin xyz="0.028573529330904346 0.01151470170789251 -0.0304382811084827" rpy="0 0 0"/>
+    <mass value="0.18931422070235698"/>
+    <inertia ixx="5.5e-05" iyy="7.4e-05" izz="3.3e-05" ixy="-0.0" iyz="0.0" ixz="0.0"/>
+  </inertial>
+  <visual>
+    <origin xyz="0.25 0.2169 -0.058" rpy="0 0 0"/>
+    <geometry>
+      <mesh filename="file://$(find mycobot_description)/meshes/caster_5.stl" scale="0.001 0.001 0.001"/>
+    </geometry>
+    <material name="silver"/>
+  </visual>
+  <collision>
+    <origin xyz="0.25 0.2169 -0.058" rpy="0 0 0"/>
+    <geometry>
+      <mesh filename="file://$(find mycobot_description)/meshes/caster_5.stl" scale="0.001 0.001 0.001"/>
+    </geometry>
+  </collision>
+</link>
+<link name="caster_6">
+  <inertial>
+    <origin xyz="0.02857352933088425 -0.01151471005681412 -0.030438281108482977" rpy="0 0 0"/>
+    <mass value="0.18931422070235698"/>
+    <inertia ixx="5.5e-05" iyy="7.4e-05" izz="3.3e-05" ixy="-0.0" iyz="0.0" ixz="0.0"/>
+  </inertial>
+  <visual>
+    <origin xyz="0.25 -0.2169 -0.058" rpy="0 0 0"/>
+    <geometry>
+      <mesh filename="file://$(find mycobot_description)/meshes/caster_6.stl" scale="0.001 0.001 0.001"/>
+    </geometry>
+    <material name="silver"/>
+  </visual>
+  <collision>
+    <origin xyz="0.25 -0.2169 -0.058" rpy="0 0 0"/>
+    <geometry>
+      <mesh filename="file://$(find mycobot_description)/meshes/caster_6.stl" scale="0.001 0.001 0.001"/>
+    </geometry>
+  </collision>
+</link>
+<link name="XL430_base_2">
+  <inertial>
+    <origin xyz="-0.008328504070776243 0.006321930521842017 0.014516362632086596" rpy="0 0 0"/>
+    <mass value="0.3239556630537195"/>
+    <inertia ixx="5e-05" iyy="7.9e-05" izz="8.6e-05" ixy="-0.0" iyz="0.0" ixz="0.0"/>
+  </inertial>
+  <visual>
+    <origin xyz="0.004 -0.198 -0.0855" rpy="0 0 0"/>
+    <geometry>
+      <mesh filename="file://$(find mycobot_description)/meshes/XL430_base_2.stl" scale="0.001 0.001 0.001"/>
+    </geometry>
+    <material name="silver"/>
+  </visual>
+  <collision>
+    <origin xyz="0.004 -0.198 -0.0855" rpy="0 0 0"/>
+    <geometry>
+      <mesh filename="file://$(find mycobot_description)/meshes/XL430_base_2.stl" scale="0.001 0.001 0.001"/>
+    </geometry>
+  </collision>
+</link>
+<link name="XL430_base_1">
+  <inertial>
+    <origin xyz="0.015671495929223667 -0.00632193052184804 0.014483637367895638" rpy="0 0 0"/>
+    <mass value="0.3239556630537195"/>
+    <inertia ixx="5e-05" iyy="7.9e-05" izz="8.6e-05" ixy="0.0" iyz="0.0" ixz="-0.0"/>
+  </inertial>
+  <visual>
+    <origin xyz="0.028 0.198 -0.0855" rpy="0 0 0"/>
+    <geometry>
+      <mesh filename="file://$(find mycobot_description)/meshes/XL430_base_1.stl" scale="0.001 0.001 0.001"/>
+    </geometry>
+    <material name="silver"/>
+  </visual>
+  <collision>
+    <origin xyz="0.028 0.198 -0.0855" rpy="0 0 0"/>
+    <geometry>
+      <mesh filename="file://$(find mycobot_description)/meshes/XL430_base_1.stl" scale="0.001 0.001 0.001"/>
+    </geometry>
+  </collision>
+</link>
+<link name="XL430_motor_1">
+  <inertial>
+    <origin xyz="-3.045443770730309e-06 -0.002385176775222958 6.646072581162343e-14" rpy="0 0 0"/>
+    <mass value="0.011770865349524429"/>
+    <inertia ixx="0.0" iyy="1e-06" izz="0.0" ixy="0.0" iyz="0.0" ixz="-0.0"/>
+  </inertial>
+  <visual>
+    <origin xyz="-0.0003 0.2188 -0.1" rpy="0 0 0"/>
+    <geometry>
+      <mesh filename="file://$(find mycobot_description)/meshes/XL430_motor_1.stl" scale="0.001 0.001 0.001"/>
+    </geometry>
+    <material name="silver"/>
+  </visual>
+  <collision>
+    <origin xyz="-0.0003 0.2188 -0.1" rpy="0 0 0"/>
+    <geometry>
+      <mesh filename="file://$(find mycobot_description)/meshes/XL430_motor_1.stl" scale="0.001 0.001 0.001"/>
+    </geometry>
+  </collision>
+</link>
+<link name="wheel_1">
+  <inertial>
+    <origin xyz="-0.005656851380657197 -0.013437856519626423 -0.005656982696146395" rpy="0 0 0"/>
+    <mass value="5.068160827641181"/>
+    <inertia ixx="0.014881" iyy="0.029142" izz="0.014881" ixy="0.0" iyz="0.0" ixz="-0.0"/>
+  </inertial>
+  <visual>
+    <origin xyz="-0.005957 0.2233 -0.105657" rpy="0 0 0"/>
+    <geometry>
+      <mesh filename="file://$(find mycobot_description)/meshes/wheel_1.stl" scale="0.001 0.001 0.001"/>
+    </geometry>
+    <material name="silver"/>
+  </visual>
+  <collision>
+    <origin xyz="-0.005957 0.2233 -0.105657" rpy="0 0 0"/>
+    <geometry>
+      <mesh filename="file://$(find mycobot_description)/meshes/wheel_1.stl" scale="0.001 0.001 0.001"/>
+    </geometry>
+  </collision>
+</link>
+<link name="XL430_motor_2">
+  <inertial>
+    <origin xyz="0.2077984717700098 -0.09411482322478323 -0.000300000000084219" rpy="0 0 0"/>
+    <mass value="0.011770865349524429"/>
+    <inertia ixx="0.0" iyy="1e-06" izz="0.0" ixy="-0.0" iyz="0.0" ixz="0.0"/>
+  </inertial>
+  <visual>
+    <origin xyz="0.2075 -0.3153 -0.1003" rpy="0 0 0"/>
+    <geometry>
+      <mesh filename="file://$(find mycobot_description)/meshes/XL430_motor_2.stl" scale="0.001 0.001 0.001"/>
+    </geometry>
+    <material name="silver"/>
+  </visual>
+  <collision>
+    <origin xyz="0.2075 -0.3153 -0.1003" rpy="0 0 0"/>
+    <geometry>
+      <mesh filename="file://$(find mycobot_description)/meshes/XL430_motor_2.stl" scale="0.001 0.001 0.001"/>
+    </geometry>
+  </collision>
+</link>
+<link name="wheel_3">
+  <inertial>
+    <origin xyz="-0.005655334166857521 0.46003785651962026 0.005656982696109328" rpy="0 0 0"/>
+    <mass value="5.068160827641181"/>
+    <inertia ixx="0.014881" iyy="0.029142" izz="0.014881" ixy="-0.0" iyz="0.0" ixz="0.0"/>
+  </inertial>
+  <visual>
+    <origin xyz="-0.005957 0.2233 -0.094343" rpy="0 0 0"/>
+    <geometry>
+      <mesh filename="file://$(find mycobot_description)/meshes/wheel_3.stl" scale="0.001 0.001 0.001"/>
+    </geometry>
+    <material name="silver"/>
+  </visual>
+  <collision>
+    <origin xyz="-0.005957 0.2233 -0.094343" rpy="0 0 0"/>
+    <geometry>
+      <mesh filename="file://$(find mycobot_description)/meshes/wheel_3.stl" scale="0.001 0.001 0.001"/>
+    </geometry>
+  </collision>
+</link>
+<link name="plate_1">
+  <inertial>
+    <origin xyz="2.349014429479716e-17 2.217469621428852e-14 0.009999999999990572" rpy="0 0 0"/>
+    <mass value="6.078748022419618"/>
+    <inertia ixx="0.018932" iyy="0.018932" izz="0.037458" ixy="0.0" iyz="0.0" ixz="0.0"/>
+  </inertial>
+  <visual>
+    <origin xyz="-0.0 0.0 -0.501" rpy="0 0 0"/>
+    <geometry>
+      <mesh filename="file://$(find mycobot_description)/meshes/plate_1.stl" scale="0.001 0.001 0.001"/>
+    </geometry>
+    <material name="silver"/>
+  </visual>
+  <collision>
+    <origin xyz="-0.0 0.0 -0.501" rpy="0 0 0"/>
+    <geometry>
+      <mesh filename="file://$(find mycobot_description)/meshes/plate_1.stl" scale="0.001 0.001 0.001"/>
+    </geometry>
+  </collision>
+</link>
+<link name="cobot_body_1">
+  <inertial>
+    <origin xyz="-1.3994638513012427e-08 -0.013751224256373267 0.04886454507233462" rpy="0 0 0"/>
     <mass value="12.899764355948896"/>
     <inertia ixx="0.033823" iyy="0.028162" izz="0.035033" ixy="0.0" iyz="-0.000755" ixz="0.0"/>
   </inertial>
   <visual>
-    <origin xyz="0 0 0" rpy="0 0 0"/>
-    <geometry>
-      <mesh filename="file://$(find mycobot_description)/meshes/base_link.stl" scale="0.001 0.001 0.001"/>
-    </geometry>
-    <material name="silver"/>
-  </visual>
-  <collision>
-    <origin xyz="0 0 0" rpy="0 0 0"/>
-    <geometry>
-      <mesh filename="file://$(find mycobot_description)/meshes/base_link.stl" scale="0.001 0.001 0.001"/>
-    </geometry>
-  </collision>
-</link>
-<link name="link1">
-  <inertial>
-    <origin xyz="0.006896766224730428 4.7445558334983536e-17 0.055490186869056476" rpy="0 0 0"/>
+    <origin xyz="-0.0 -0.0 -0.521" rpy="0 0 0"/>
+    <geometry>
+      <mesh filename="file://$(find mycobot_description)/meshes/cobot_body_1.stl" scale="0.001 0.001 0.001"/>
+    </geometry>
+    <material name="silver"/>
+  </visual>
+  <collision>
+    <origin xyz="-0.0 -0.0 -0.521" rpy="0 0 0"/>
+    <geometry>
+      <mesh filename="file://$(find mycobot_description)/meshes/cobot_body_1.stl" scale="0.001 0.001 0.001"/>
+    </geometry>
+  </collision>
+</link>
+<link name="baseArm_v1_1">
+  <inertial>
+    <origin xyz="0.0068967662247284124 2.2561127161268677e-14 0.05549018686904705" rpy="0 0 0"/>
     <mass value="3.4735206294395446"/>
-    <inertia ixx="0.004461" iyy="0.004757" izz="0.002424" ixy="-0.0" iyz="0.0" ixz="-0.000777"/>
-  </inertial>
-  <visual>
-    <origin xyz="-0.0 -0.0 -0.11" rpy="0 0 0"/>
-    <geometry>
-      <mesh filename="file://$(find mycobot_description)/meshes/link1.stl" scale="0.001 0.001 0.001"/>
-    </geometry>
-    <material name="silver"/>
-  </visual>
-  <collision>
-    <origin xyz="-0.0 -0.0 -0.11" rpy="0 0 0"/>
-    <geometry>
-      <mesh filename="file://$(find mycobot_description)/meshes/link1.stl" scale="0.001 0.001 0.001"/>
-    </geometry>
-  </collision>
-</link>
-<link name="link2">
-  <inertial>
-    <origin xyz="0.03690658575567249 -1.0444649911926371e-16 0.06800000000000012" rpy="0 0 0"/>
+    <inertia ixx="0.004461" iyy="0.004757" izz="0.002424" ixy="0.0" iyz="0.0" ixz="-0.000777"/>
+  </inertial>
+  <visual>
+    <origin xyz="0.0 -0.0 -0.631" rpy="0 0 0"/>
+    <geometry>
+      <mesh filename="file://$(find mycobot_description)/meshes/baseArm_v1_1.stl" scale="0.001 0.001 0.001"/>
+    </geometry>
+    <material name="silver"/>
+  </visual>
+  <collision>
+    <origin xyz="0.0 -0.0 -0.631" rpy="0 0 0"/>
+    <geometry>
+      <mesh filename="file://$(find mycobot_description)/meshes/baseArm_v1_1.stl" scale="0.001 0.001 0.001"/>
+    </geometry>
+  </collision>
+</link>
+<link name="lowerArm_v1_1">
+  <inertial>
+    <origin xyz="0.03690658575566909 2.2563486026873027e-14 0.06799999999999196" rpy="0 0 0"/>
     <mass value="5.91988968680626"/>
     <inertia ixx="0.0188" iyy="0.019335" izz="0.004161" ixy="0.0" iyz="0.0" ixz="0.0"/>
   </inertial>
   <visual>
-    <origin xyz="-0.045 -0.0 -0.195" rpy="0 0 0"/>
-    <geometry>
-      <mesh filename="file://$(find mycobot_description)/meshes/link2.stl" scale="0.001 0.001 0.001"/>
-    </geometry>
-    <material name="silver"/>
-  </visual>
-  <collision>
-    <origin xyz="-0.045 -0.0 -0.195" rpy="0 0 0"/>
-    <geometry>
-      <mesh filename="file://$(find mycobot_description)/meshes/link2.stl" scale="0.001 0.001 0.001"/>
-    </geometry>
-  </collision>
-</link>
-<link name="link3">
-  <inertial>
-    <origin xyz="-0.035022688252992054 -8.56731250465993e-16 0.049500000000000155" rpy="0 0 0"/>
+    <origin xyz="-0.045 -0.0 -0.716" rpy="0 0 0"/>
+    <geometry>
+      <mesh filename="file://$(find mycobot_description)/meshes/lowerArm_v1_1.stl" scale="0.001 0.001 0.001"/>
+    </geometry>
+    <material name="silver"/>
+  </visual>
+  <collision>
+    <origin xyz="-0.045 -0.0 -0.716" rpy="0 0 0"/>
+    <geometry>
+      <mesh filename="file://$(find mycobot_description)/meshes/lowerArm_v1_1.stl" scale="0.001 0.001 0.001"/>
+    </geometry>
+  </collision>
+</link>
+<link name="upperArm_v1_1">
+  <inertial>
+    <origin xyz="-0.035022688252996176 2.6167507160751738e-14 0.04949999999999111" rpy="0 0 0"/>
     <mass value="4.802107093668197"/>
-    <inertia ixx="0.01014" iyy="0.010584" izz="0.003386" ixy="-0.0" iyz="0.0" ixz="-0.0"/>
-  </inertial>
-  <visual>
-    <origin xyz="-0.045 0.0 -0.331" rpy="0 0 0"/>
-    <geometry>
-      <mesh filename="file://$(find mycobot_description)/meshes/link3.stl" scale="0.001 0.001 0.001"/>
-    </geometry>
-    <material name="silver"/>
-  </visual>
-  <collision>
-    <origin xyz="-0.045 0.0 -0.331" rpy="0 0 0"/>
-    <geometry>
-      <mesh filename="file://$(find mycobot_description)/meshes/link3.stl" scale="0.001 0.001 0.001"/>
-    </geometry>
-  </collision>
-</link>
-<link name="link4">
-  <inertial>
-    <origin xyz="0.03442387286919234 -1.62263567395975e-15 0.010576127130807855" rpy="0 0 0"/>
+    <inertia ixx="0.01014" iyy="0.010584" izz="0.003386" ixy="-0.0" iyz="-0.0" ixz="-0.0"/>
+  </inertial>
+  <visual>
+    <origin xyz="-0.045 -0.0 -0.852" rpy="0 0 0"/>
+    <geometry>
+      <mesh filename="file://$(find mycobot_description)/meshes/upperArm_v1_1.stl" scale="0.001 0.001 0.001"/>
+    </geometry>
+    <material name="silver"/>
+  </visual>
+  <collision>
+    <origin xyz="-0.045 -0.0 -0.852" rpy="0 0 0"/>
+    <geometry>
+      <mesh filename="file://$(find mycobot_description)/meshes/upperArm_v1_1.stl" scale="0.001 0.001 0.001"/>
+    </geometry>
+  </collision>
+</link>
+<link name="pitchArm_v1_1">
+  <inertial>
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
Commit message: edit wheel file(split another component
휠을 다른 컴포터넌트로 교체

File: mycobot_description/urdf/mycobot.xacro (robot description, xacro)
@@ -164,5 +164,5 @@
   </collision>
 </link>
-<link name="wheel_1">
+<link name="wheel_right_1">
   <inertial>
     <origin xyz="-0.005656851380657197 -0.013437856519626423 -0.005656982696146395" rpy="0 0 0"/>
@@ -173,5 +173,5 @@
     <origin xyz="-0.005957 0.2233 -0.105657" rpy="0 0 0"/>
     <geometry>
-      <mesh filename="file://$(find mycobot_description)/meshes/wheel_1.stl" scale="0.001 0.001 0.001"/>
+      <mesh filename="file://$(find mycobot_description)/meshes/wheel_right_1.stl" scale="0.001 0.001 0.001"/>
     </geometry>
     <material name="silver"/>
@@ -180,5 +180,5 @@
     <origin xyz="-0.005957 0.2233 -0.105657" rpy="0 0 0"/>
     <geometry>
-      <mesh filename="file://$(find mycobot_description)/meshes/wheel_1.stl" scale="0.001 0.001 0.001"/>
+      <mesh filename="file://$(find mycobot_description)/meshes/wheel_right_1.stl" scale="0.001 0.001 0.001"/>
     </geometry>
   </collision>
@@ -201,24 +201,4 @@
     <geometry>
       <mesh filename="file://$(find mycobot_description)/meshes/XL430_motor_2.stl" scale="0.001 0.001 0.001"/>
-    </geometry>
-  </collision>
-</link>
-<link name="wheel_3">
-  <inertial>
-    <origin xyz="-0.005655334166857521 0.46003785651962026 0.005656982696109328" rpy="0 0 0"/>
-    <mass value="5.068160827641181"/>
-    <inertia ixx="0.014881" iyy="0.029142" izz="0.014881" ixy="-0.0" iyz="0.0" ixz="0.0"/>
-  </inertial>
-  <visual>
-    <origin xyz="-0.005957 0.2233 -0.094343" rpy="0 0 0"/>
-    <geometry>
-      <mesh filename="file://$(find mycobot_description)/meshes/wheel_3.stl" scale="0.001 0.001 0.001"/>
-    </geometry>
-    <material name="silver"/>
-  </visual>
-  <collision>
-    <origin xyz="-0.005957 0.2233 -0.094343" rpy="0 0 0"/>
-    <geometry>
-      <mesh filename="file://$(find mycobot_description)/meshes/wheel_3.stl" scale="0.001 0.001 0.001"/>
     </geometry>
   </collision>
@@ -585,5 +565,5 @@
   <origin xyz="0.005657 -0.0045 0.005657" rpy="0 0 0"/>
   <parent link="XL430_motor_1"/>
-  <child link="wheel_1"/>
+  <child link="wheel_right_1"/>
 </joint>
 <joint name="Revolute 15" type="revolute">
@@ -593,9 +573,4 @@
   <axis xyz="0.0 1.0 -0.0"/>
   <limit upper="6.283185" lower="0.0" effort="100" velocity="100"/>
-</joint>
-<joint name="Rigid 16" type="fixed">
-  <origin xyz="0.213457 -0.5386 -0.005957" rpy="0 0 0"/>
-  <parent link="XL430_motor_2"/>
-  <child link="wheel_3"/>
 </joint>
 <joint name="Rigid 21" type="fixed">
