Commit message: edit component
다이나믹셀 다른 컴포넌트로 교체

File: mycobot_description/urdf/mycobot.xacro (robot description, xacro)
@@ -104,25 +104,5 @@
   </collision>
 </link>
-<link name="XL430_base_2">
-  <inertial>
-    <origin xyz="-0.008328504070776243 0.006321930521842017 0.014516362632086596" rpy="0 0 0"/>
-    <mass value="0.3239556630537195"/>
-    <inertia ixx="5e-05" iyy="7.9e-05" izz="8.6e-05" ixy="-0.0" iyz="0.0" ixz="0.0"/>
-  </inertial>
-  <visual>
-    <origin xyz="0.004 -0.198 -0.0855" rpy="0 0 0"/>
-    <geometry>
-      <mesh filename="file://$(find mycobot_description)/meshes/XL430_base_2.stl" scale="0.001 0.001 0.001"/>
-    </geometry>
-    <material name="silver"/>
-  </visual>
-  <collision>
-    <origin xyz="0.004 -0.198 -0.0855" rpy="0 0 0"/>
-    <geometry>
-      <mesh filename="file://$(find mycobot_description)/meshes/XL430_base_2.stl" scale="0.001 0.001 0.001"/>
-    </geometry>
-  </collision>
-</link>
-<link name="XL430_base_1">
+<link name="XL430_base_right_1">
   <inertial>
     <origin xyz="0.015671495929223667 -0.00632193052184804 0.014483637367895638" rpy="0 0 0"/>
@@ -133,5 +113,5 @@
     <origin xyz="0.028 0.198 -0.0855" rpy="0 0 0"/>
     <geometry>
-      <mesh filename="file://$(find mycobot_description)/meshes/XL430_base_1.stl" scale="0.001 0.001 0.001"/>
+      <mesh filename="file://$(find mycobot_description)/meshes/XL430_base_right_1.stl" scale="0.001 0.001 0.001"/>
     </geometry>
     <material name="silver"/>
@@ -140,9 +120,9 @@
     <origin xyz="0.028 0.198 -0.0855" rpy="0 0 0"/>
     <geometry>
-      <mesh filename="file://$(find mycobot_description)/meshes/XL430_base_1.stl" scale="0.001 0.001 0.001"/>
-    </geometry>
-  </collision>
-</link>
-<link name="XL430_motor_1">
+      <mesh filename="file://$(find mycobot_description)/meshes/XL430_base_right_1.stl" scale="0.001 0.001 0.001"/>
+    </geometry>
+  </collision>
+</link>
+<link name="XL430_motor_right_1">
   <inertial>
     <origin xyz="-3.045443770730309e-06 -0.002385176775222958 6.646072581162343e-14" rpy="0 0 0"/>
@@ -153,5 +133,5 @@
     <origin xyz="-0.0003 0.2188 -0.1" rpy="0 0 0"/>
     <geometry>
-      <mesh filename="file://$(find mycobot_description)/meshes/XL430_motor_1.stl" scale="0.001 0.001 0.001"/>
+      <mesh filename="file://$(find mycobot_description)/meshes/XL430_motor_right_1.stl" scale="0.001 0.001 0.001"/>
     </geometry>
     <material name="silver"/>
@@ -160,5 +140,5 @@
     <origin xyz="-0.0003 0.2188 -0.1" rpy="0 0 0"/>
     <geometry>
-      <mesh filename="file://$(find mycobot_description)/meshes/XL430_motor_1.stl" scale="0.001 0.001 0.001"/>
+      <mesh filename="file://$(find mycobot_description)/meshes/XL430_motor_right_1.stl" scale="0.001 0.001 0.001"/>
     </geometry>
   </collision>
@@ -184,24 +164,4 @@
   </collision>
 </link>
-<link name="XL430_motor_2">
-  <inertial>
-    <origin xyz="0.2077984717700098 -0.09411482322478323 -0.000300000000084219" rpy="0 0 0"/>
-    <mass value="0.011770865349524429"/>
-    <inertia ixx="0.0" iyy="1e-06" izz="0.0" ixy="-0.0" iyz="0.0" ixz="0.0"/>
-  </inertial>
-  <visual>
-    <origin xyz="0.2075 -0.3153 -0.1003" rpy="0 0 0"/>
-    <geometry>
-      <mesh filename="file://$(find mycobot_description)/meshes/XL430_motor_2.stl" scale="0.001 0.001 0.001"/>
-    </geometry>
-    <material name="silver"/>
-  </visual>
-  <collision>
-    <origin xyz="0.2075 -0.3153 -0.1003" rpy="0 0 0"/>
-    <geometry>
-      <mesh filename="file://$(find mycobot_description)/meshes/XL430_motor_2.stl" scale="0.001 0.001 0.001"/>
-    </geometry>
-  </collision>
-</link>
 <link name="plate_1">
   <inertial>
@@ -524,5 +484,44 @@
   </collision>
 </link>
-<!-- joint -->
+<link name="XL430_base_left_1">
+  <inertial>
+    <origin xyz="0.015671495929223758 0.006321930521842017 0.014516362632086596" rpy="0 0 0"/>
+    <mass value="0.3239556630537195"/>
+    <inertia ixx="5e-05" iyy="7.9e-05" izz="8.6e-05" ixy="-0.0" iyz="0.0" ixz="0.0"/>
+  </inertial>
+  <visual>
+    <origin xyz="0.028 -0.198 -0.0855" rpy="0 0 0"/>
+    <geometry>
+      <mesh filename="file://$(find mycobot_description)/meshes/XL430_base_left_1.stl" scale="0.001 0.001 0.001"/>
+    </geometry>
+    <material name="silver"/>
+  </visual>
+  <collision>
+    <origin xyz="0.028 -0.198 -0.0855" rpy="0 0 0"/>
+    <geometry>
+      <mesh filename="file://$(find mycobot_description)/meshes/XL430_base_left_1.stl" scale="0.001 0.001 0.001"/>
+    </geometry>
+  </collision>
+</link>
+<link name="XL430_motor_left_1">
+  <inertial>
+    <origin xyz="-3.0454437706458498e-06 0.0023851767752167963 -8.416878305439468e-14" rpy="0 0 0"/>
+    <mass value="0.011770865349524429"/>
+    <inertia ixx="0.0" iyy="1e-06" izz="0.0" ixy="-0.0" iyz="0.0" ixz="0.0"/>
+  </inertial>
+  <visual>
+    <origin xyz="-0.0003 -0.2188 -0.1" rpy="0 0 0"/>
+    <geometry>
+      <mesh filename="file://$(find mycobot_description)/meshes/XL430_motor_left_1.stl" scale="0.001 0.001 0.001"/>
+    </geometry>
+    <material name="silver"/>
+  </visual>
+  <collision>
+    <origin xyz="-0.0003 -0.2188 -0.1" rpy="0 0 0"/>
+    <geometry>
+      <mesh filename="file://$(find mycobot_description)/meshes/XL430_motor_left_1.stl" scale="0.001 0.001 0.001"/>
+    </geometry>
+  </collision>
+</link>
 <joint name="Rigid 5" type="fixed">
   <origin xyz="0.25 0.2169 0.058" rpy="0 0 0"/>
@@ -545,18 +544,13 @@
   <child link="caster_6"/>
 </joint>
-<joint name="Rigid 9" type="fixed">
-  <origin xyz="-0.004 0.198 0.0855" rpy="0 0 0"/>
-  <parent link="base_link"/>
-  <child link="XL430_base_2"/>
-</joint>
 <joint name="Rigid 11" type="fixed">
   <origin xyz="-0.028 -0.198 0.0855" rpy="0 0 0"/>
   <parent link="base_link"/>
-  <child link="XL430_base_1"/>
+  <child link="XL430_base_right_1"/>
 </joint>
 <joint name="Revolute 12" type="revolute">
   <origin xyz="0.0283 -0.0208 0.0145" rpy="0 0 0"/>
-  <parent link="XL430_base_1"/>
-  <child link="XL430_motor_1"/>
+  <parent link="XL430_base_right_1"/>
+  <child link="XL430_motor_right_1"/>
   <axis xyz="-0.0 -1.0 0.0"/>
   <limit upper="6.283185" lower="0.0" effort="100" velocity="100"/>
@@ -564,13 +558,6 @@
 <joint name="Rigid 14" type="fixed">
   <origin xyz="0.005657 -0.0045 0.005657" rpy="0 0 0"/>
-  <parent link="XL430_motor_1"/>
+  <parent link="XL430_motor_right_1"/>
   <child link="wheel_right_1"/>
-</joint>
-<joint name="Revolute 15" type="revolute">
-  <origin xyz="-0.2035 0.1173 0.0148" rpy="0 0 0"/>
-  <parent link="XL430_base_2"/>
-  <child link="XL430_motor_2"/>
-  <axis xyz="0.0 1.0 -0.0"/>
-  <limit upper="6.283185" lower="0.0" effort="100" velocity="100"/>
 </joint>
 <joint name="Rigid 21" type="fixed">
@@ -665,5 +652,4 @@
   <limit upper="0.3" lower="-0.7" effort="100" velocity="100"/> <!-- change upper to 0.3 and lower to -0.7-->
   <mimic joint="gripper_controller" multiplier="1" offset="0"/> <!-- add mimic and change multiplier to 1-->
-</joint>
 <joint name="Rigid 39" type="fixed">
   <origin xyz="0.0 0.0 0.11" rpy="0 0 0"/>
@@ -676,3 +662,15 @@
   <child link="camera_stand_1"/>
 </joint>
+<joint name="Rigid 42" type="fixed">
+  <origin xyz="-0.028 0.198 0.0855" rpy="0 0 0"/>
+  <parent link="base_link"/>
+  <child link="XL430_base_left_1"/>
+</joint>
+<joint name="Revolute 43" type="revolute">
+  <origin xyz="0.0283 0.0208 0.0145" rpy="0 0 0"/>
+  <parent link="XL430_base_left_1"/>
+  <child link="XL430_motor_left_1"/>
+  <axis xyz="0.0 1.0 -0.0"/>
+  <limit upper="6.283185" lower="0.0" effort="100" velocity="100"/>
+</joint>
 </robot>

Commit message: fixed error
휠과 모터 조인트 수정

File: mycobot_description/urdf/mycobot.xacro (robot description, xacro)
@@ -521,4 +521,24 @@
     <geometry>
       <mesh filename="file://$(find mycobot_description)/meshes/XL430_motor_left_1.stl" scale="0.001 0.001 0.001"/>
+    </geometry>
+  </collision>
+</link>
+<link name="wheel_left_1">
+  <inertial>
+    <origin xyz="-0.00565685138065711 0.01343785651962029 -0.0056570173038905935" rpy="0 0 0"/>
+    <mass value="5.068160827641181"/>
+    <inertia ixx="0.014881" iyy="0.029142" izz="0.014881" ixy="-0.0" iyz="0.0" ixz="0.0"/>
+  </inertial>
+  <visual>
+    <origin xyz="-0.005957 -0.2233 -0.105657" rpy="0 0 0"/>
+    <geometry>
+      <mesh filename="file://$(find mycobot_description)/meshes/wheel_left_1.stl" scale="0.001 0.001 0.001"/>
+    </geometry>
+    <material name="silver"/>
+  </visual>
+  <collision>
+    <origin xyz="-0.005957 -0.2233 -0.105657" rpy="0 0 0"/>
+    <geometry>
+      <mesh filename="file://$(find mycobot_description)/meshes/wheel_left_1.stl" scale="0.001 0.001 0.001"/>
     </geometry>
   </collision>
@@ -652,4 +672,5 @@
   <limit upper="0.3" lower="-0.7" effort="100" velocity="100"/> <!-- change upper to 0.3 and lower to -0.7-->
   <mimic joint="gripper_controller" multiplier="1" offset="0"/> <!-- add mimic and change multiplier to 1-->
+</joint>
 <joint name="Rigid 39" type="fixed">
   <origin xyz="0.0 0.0 0.11" rpy="0 0 0"/>
@@ -674,3 +695,8 @@
   <limit upper="6.283185" lower="0.0" effort="100" velocity="100"/>
 </joint>
+<joint name="Rigid 44" type="fixed">
+  <origin xyz="0.005657 0.0045 0.005657" rpy="0 0 0"/>
+  <parent link="XL430_motor_left_1"/>
+  <child link="wheel_left_1"/>
+</joint>
 </robot>

Commit message: edit joint
조인트 순서 변경(좌우 휠이 슬라이더 위로 오게 수정, 조인트 이름 변경)

File: mycobot_description/urdf/mycobot.xacro (robot description, xacro)
@@ -569,5 +569,12 @@
   <child link="XL430_base_right_1"/>
 </joint>
-<joint name="Revolute 12" type="revolute">
+<joint name="wheel_left" type="revolute">
+  <origin xyz="0.0283 0.0208 0.0145" rpy="0 0 0"/>
+  <parent link="XL430_base_left_1"/>
+  <child link="XL430_motor_left_1"/>
+  <axis xyz="0.0 1.0 -0.0"/>
+  <limit upper="6.283185" lower="0.0" effort="100" velocity="100"/>
+</joint>
+<joint name="wheel_right" type="revolute">
   <origin xyz="0.0283 -0.0208 0.0145" rpy="0 0 0"/>
   <parent link="XL430_base_right_1"/>
@@ -688,11 +695,4 @@
   <child link="XL430_base_left_1"/>
 </joint>
-<joint name="Revolute 43" type="revolute">
-  <origin xyz="0.0283 0.0208 0.0145" rpy="0 0 0"/>
-  <parent link="XL430_base_left_1"/>
-  <child link="XL430_motor_left_1"/>
-  <axis xyz="0.0 1.0 -0.0"/>
-  <limit upper="6.283185" lower="0.0" effort="100" velocity="100"/>
-</joint>
 <joint name="Rigid 44" type="fixed">
   <origin xyz="0.005657 0.0045 0.005657" rpy="0 0 0"/>

Commit message: edit joint
그리퍼 컨트롤 mimic 조인트 멀티플라이어 값 수정

File: mycobot_description/urdf/mycobot.xacro (robot description, xacro)
@@ -662,5 +662,5 @@
   <axis xyz="0.0 -0.0 1.0"/>
   <limit upper="0.7" lower="-0.3" effort="100" velocity="100"/> <!-- change upper to 0.7 and lower to -0.3-->
-  <mimic joint="gripper_controller" multiplier="-1" offset="0"/> <!-- add mimic and change multiplier to -1-->
+  <mimic joint="gripper_controller" multiplier="1" offset="0"/> <!-- add mimic and change multiplier to -1-->
 </joint>
 <joint name="Revolute 33" type="revolute">
@@ -678,5 +678,5 @@
   <axis xyz="0.0 0.0 1.0"/>
   <limit upper="0.3" lower="-0.7" effort="100" velocity="100"/> <!-- change upper to 0.3 and lower to -0.7-->
-  <mimic joint="gripper_controller" multiplier="1" offset="0"/> <!-- add mimic and change multiplier to 1-->
+  <mimic joint="gripper_controller" multiplier="-1" offset="0"/> <!-- add mimic and change multiplier to 1-->
 </joint>
 <joint name="Rigid 39" type="fixed">

Commit message: edit joint
mycobot joint 이름 변경, continous -> revolute 변경

File: mycobot_description/urdf/mycobot.xacro (robot description, xacro)
@@ -598,5 +598,5 @@
   <child link="cobot_body_1"/>
 </joint>
-<joint name="Revolute 24" type="revolute">
+<joint name="Revolute 1" type="revolute">
   <origin xyz="-0.0 0.0 0.11" rpy="0 0 0"/>
   <parent link="cobot_body_1"/>
@@ -605,5 +605,5 @@
   <limit upper="2.792527" lower="-2.792527" effort="100" velocity="100"/>
 </joint>
-<joint name="Revolute 25" type="revolute">
+<joint name="Revolute 2" type="revolute">
   <origin xyz="0.045 0.0 0.085" rpy="0 0 0"/>
   <parent link="baseArm_v1_1"/>
@@ -612,11 +612,12 @@
   <limit upper="2.792527" lower="-2.792527" effort="100" velocity="100"/>
 </joint>
-<joint name="Revolute 26" type="continuous">
+<joint name="Revolute 3" type="revolute">
   <origin xyz="0.0 0.0 0.136" rpy="0 0 0"/>
   <parent link="lowerArm_v1_1"/>
   <child link="upperArm_v1_1"/>
   <axis xyz="-1.0 0.0 -0.0"/>
-</joint>
-<joint name="Revolute 27" type="revolute">
+  <limit upper="2.792527" lower="-2.792527" effort="100" velocity="100"/>
+</joint>
+<joint name="Revolute 4" type="revolute">
   <origin xyz="0.0 0.0 0.099" rpy="0 0 0"/>
   <parent link="upperArm_v1_1"/>
@@ -625,5 +626,5 @@
   <limit upper="2.792527" lower="-2.792527" effort="100" velocity="100"/>
 </joint>
-<joint name="Revolute 28" type="revolute">
+<joint name="Revolute 5" type="revolute">
   <origin xyz="0.045 0.0 0.045" rpy="0 0 0"/>
   <parent link="pitchArm_v1_1"/>
@@ -632,5 +633,5 @@
   <limit upper="2.792527" lower="-2.792527" effort="100" velocity="100"/>
 </joint>
-<joint name="Revolute 29" type="revolute">
+<joint name="Revolute 6" type="revolute">
   <origin xyz="0.04 0.0 0.05" rpy="0 0 0"/>
   <parent link="rollArm_v1_1"/>
