Commit message: change stl name, delete gazebo file

File: mycobot_description/urdf/mycobot.xacro (robot description, xacro)
@@ -24,5 +24,5 @@
   </collision>
 </link>
-<link name="caster_3">
+<link name="caster_1">
   <inertial>
     <origin xyz="-0.02857352949264516 -0.01151471005681412 -0.03043828110848307" rpy="0 0 0"/>
@@ -33,5 +33,5 @@
     <origin xyz="-0.25 -0.2169 -0.058" rpy="0 0 0"/>
     <geometry>
-      <mesh filename="file://$(find mycobot_description)/meshes/caster_3.stl" scale="0.001 0.001 0.001"/>
+      <mesh filename="file://$(find mycobot_description)/meshes/caster_1.stl" scale="0.001 0.001 0.001"/>
     </geometry>
     <material name="silver"/>
@@ -40,9 +40,9 @@
     <origin xyz="-0.25 -0.2169 -0.058" rpy="0 0 0"/>
     <geometry>
-      <mesh filename="file://$(find mycobot_description)/meshes/caster_3.stl" scale="0.001 0.001 0.001"/>
-    </geometry>
-  </collision>
-</link>
-<link name="caster_4">
+      <mesh filename="file://$(find mycobot_description)/meshes/caster_1.stl" scale="0.001 0.001 0.001"/>
+    </geometry>
+  </collision>
+</link>
+<link name="caster_2">
   <inertial>
     <origin xyz="-0.028573529492625066 0.011514701707892594 -0.03043828110848334" rpy="0 0 0"/>
@@ -53,5 +53,5 @@
     <origin xyz="-0.25 0.2169 -0.058" rpy="0 0 0"/>
     <geometry>
-      <mesh filename="file://$(find mycobot_description)/meshes/caster_4.stl" scale="0.001 0.001 0.001"/>
+      <mesh filename="file://$(find mycobot_description)/meshes/caster_2.stl" scale="0.001 0.001 0.001"/>
     </geometry>
     <material name="silver"/>
@@ -60,9 +60,9 @@
     <origin xyz="-0.25 0.2169 -0.058" rpy="0 0 0"/>
     <geometry>
-      <mesh filename="file://$(find mycobot_description)/meshes/caster_4.stl" scale="0.001 0.001 0.001"/>
-    </geometry>
-  </collision>
-</link>
-<link name="caster_5">
+      <mesh filename="file://$(find mycobot_description)/meshes/caster_2.stl" scale="0.001 0.001 0.001"/>
+    </geometry>
+  </collision>
+</link>
+<link name="caster_3">
   <inertial>
     <origin xyz="0.028573529330904346 0.01151470170789251 -0.0304382811084827" rpy="0 0 0"/>
@@ -73,5 +73,5 @@
     <origin xyz="0.25 0.2169 -0.058" rpy="0 0 0"/>
     <geometry>
-      <mesh filename="file://$(find mycobot_description)/meshes/caster_5.stl" scale="0.001 0.001 0.001"/>
+      <mesh filename="file://$(find mycobot_description)/meshes/caster_3.stl" scale="0.001 0.001 0.001"/>
     </geometry>
     <material name="silver"/>
@@ -80,9 +80,9 @@
     <origin xyz="0.25 0.2169 -0.058" rpy="0 0 0"/>
     <geometry>
-      <mesh filename="file://$(find mycobot_description)/meshes/caster_5.stl" scale="0.001 0.001 0.001"/>
-    </geometry>
-  </collision>
-</link>
-<link name="caster_6">
+      <mesh filename="file://$(find mycobot_description)/meshes/caster_3.stl" scale="0.001 0.001 0.001"/>
+    </geometry>
+  </collision>
+</link>
+<link name="caster_4">
   <inertial>
     <origin xyz="0.02857352933088425 -0.01151471005681412 -0.030438281108482977" rpy="0 0 0"/>
@@ -93,5 +93,5 @@
     <origin xyz="0.25 -0.2169 -0.058" rpy="0 0 0"/>
     <geometry>
-      <mesh filename="file://$(find mycobot_description)/meshes/caster_6.stl" scale="0.001 0.001 0.001"/>
+      <mesh filename="file://$(find mycobot_description)/meshes/caster_4.stl" scale="0.001 0.001 0.001"/>
     </geometry>
     <material name="silver"/>
@@ -100,9 +100,9 @@
     <origin xyz="0.25 -0.2169 -0.058" rpy="0 0 0"/>
     <geometry>
-      <mesh filename="file://$(find mycobot_description)/meshes/caster_6.stl" scale="0.001 0.001 0.001"/>
-    </geometry>
-  </collision>
-</link>
-<link name="XL430_base_right_1">
+      <mesh filename="file://$(find mycobot_description)/meshes/caster_4.stl" scale="0.001 0.001 0.001"/>
+    </geometry>
+  </collision>
+</link>
+<link name="XL430_base_right">
   <inertial>
     <origin xyz="0.015671495929223667 -0.00632193052184804 0.014483637367895638" rpy="0 0 0"/>
@@ -113,5 +113,5 @@
     <origin xyz="0.028 0.198 -0.0855" rpy="0 0 0"/>
     <geometry>
-      <mesh filename="file://$(find mycobot_description)/meshes/XL430_base_right_1.stl" scale="0.001 0.001 0.001"/>
+      <mesh filename="file://$(find mycobot_description)/meshes/XL430_base_right.stl" scale="0.001 0.001 0.001"/>
     </geometry>
     <material name="silver"/>
@@ -120,9 +120,9 @@
     <origin xyz="0.028 0.198 -0.0855" rpy="0 0 0"/>
     <geometry>
-      <mesh filename="file://$(find mycobot_description)/meshes/XL430_base_right_1.stl" scale="0.001 0.001 0.001"/>
-    </geometry>
-  </collision>
-</link>
-<link name="XL430_motor_right_1">
+      <mesh filename="file://$(find mycobot_description)/meshes/XL430_base_right.stl" scale="0.001 0.001 0.001"/>
+    </geometry>
+  </collision>
+</link>
+<link name="XL430_motor_right">
   <inertial>
     <origin xyz="-3.045443770730309e-06 -0.002385176775222958 6.646072581162343e-14" rpy="0 0 0"/>
@@ -133,5 +133,5 @@
     <origin xyz="-0.0003 0.2188 -0.1" rpy="0 0 0"/>
     <geometry>
-      <mesh filename="file://$(find mycobot_description)/meshes/XL430_motor_right_1.stl" scale="0.001 0.001 0.001"/>
+      <mesh filename="file://$(find mycobot_description)/meshes/XL430_motor_right.stl" scale="0.001 0.001 0.001"/>
     </geometry>
     <material name="silver"/>
@@ -140,9 +140,9 @@
     <origin xyz="-0.0003 0.2188 -0.1" rpy="0 0 0"/>
     <geometry>
-      <mesh filename="file://$(find mycobot_description)/meshes/XL430_motor_right_1.stl" scale="0.001 0.001 0.001"/>
-    </geometry>
-  </collision>
-</link>
-<link name="wheel_right_1">
+      <mesh filename="file://$(find mycobot_description)/meshes/XL430_motor_right.stl" scale="0.001 0.001 0.001"/>
+    </geometry>
+  </collision>
+</link>
+<link name="wheel_right">
   <inertial>
     <origin xyz="-0.005656851380657197 -0.013437856519626423 -0.005656982696146395" rpy="0 0 0"/>
@@ -153,5 +153,5 @@
     <origin xyz="-0.005957 0.2233 -0.105657" rpy="0 0 0"/>
     <geometry>
-      <mesh filename="file://$(find mycobot_description)/meshes/wheel_right_1.stl" scale="0.001 0.001 0.001"/>
+      <mesh filename="file://$(find mycobot_description)/meshes/wheel_right.stl" scale="0.001 0.001 0.001"/>
     </geometry>
     <material name="silver"/>
@@ -160,9 +160,9 @@
     <origin xyz="-0.005957 0.2233 -0.105657" rpy="0 0 0"/>
     <geometry>
-      <mesh filename="file://$(find mycobot_description)/meshes/wheel_right_1.stl" scale="0.001 0.001 0.001"/>
-    </geometry>
-  </collision>
-</link>
-<link name="plate_1">
+      <mesh filename="file://$(find mycobot_description)/meshes/wheel_right.stl" scale="0.001 0.001 0.001"/>
+    </geometry>
+  </collision>
+</link>
+<link name="plate">
   <inertial>
     <origin xyz="2.349014429479716e-17 2.217469621428852e-14 0.009999999999990572" rpy="0 0 0"/>
@@ -173,5 +173,5 @@
     <origin xyz="-0.0 0.0 -0.501" rpy="0 0 0"/>
     <geometry>
-      <mesh filename="file://$(find mycobot_description)/meshes/plate_1.stl" scale="0.001 0.001 0.001"/>
+      <mesh filename="file://$(find mycobot_description)/meshes/plate.stl" scale="0.001 0.001 0.001"/>
     </geometry>
     <material name="silver"/>
@@ -180,9 +180,9 @@
     <origin xyz="-0.0 0.0 -0.501" rpy="0 0 0"/>
     <geometry>
-      <mesh filename="file://$(find mycobot_description)/meshes/plate_1.stl" scale="0.001 0.001 0.001"/>
-    </geometry>
-  </collision>
-</link>
-<link name="cobot_body_1">
+      <mesh filename="file://$(find mycobot_description)/meshes/plate.stl" scale="0.001 0.001 0.001"/>
+    </geometry>
+  </collision>
+</link>
+<link name="cobot_body">
   <inertial>
     <origin xyz="-1.3994638513012427e-08 -0.013751224256373267 0.04886454507233462" rpy="0 0 0"/>
@@ -193,5 +193,5 @@
     <origin xyz="-0.0 -0.0 -0.521" rpy="0 0 0"/>
     <geometry>
-      <mesh filename="file://$(find mycobot_description)/meshes/cobot_body_1.stl" scale="0.001 0.001 0.001"/>
+      <mesh filename="file://$(find mycobot_description)/meshes/cobot_body.stl" scale="0.001 0.001 0.001"/>
     </geometry>
     <material name="silver"/>
@@ -200,9 +200,9 @@
     <origin xyz="-0.0 -0.0 -0.521" rpy="0 0 0"/>
     <geometry>
-      <mesh filename="file://$(find mycobot_description)/meshes/cobot_body_1.stl" scale="0.001 0.001 0.001"/>
-    </geometry>
-  </collision>
-</link>
-<link name="baseArm_v1_1">
+      <mesh filename="file://$(find mycobot_description)/meshes/cobot_body.stl" scale="0.001 0.001 0.001"/>
+    </geometry>
+  </collision>
+</link>
+<link name="baseArm">
   <inertial>
     <origin xyz="0.0068967662247284124 2.2561127161268677e-14 0.05549018686904705" rpy="0 0 0"/>
@@ -213,5 +213,5 @@
     <origin xyz="0.0 -0.0 -0.631" rpy="0 0 0"/>
     <geometry>
-      <mesh filename="file://$(find mycobot_description)/meshes/baseArm_v1_1.stl" scale="0.001 0.001 0.001"/>
+      <mesh filename="file://$(find mycobot_description)/meshes/baseArm.stl" scale="0.001 0.001 0.001"/>
     </geometry>
     <material name="silver"/>
@@ -220,9 +220,9 @@
     <origin xyz="0.0 -0.0 -0.631" rpy="0 0 0"/>
     <geometry>
-      <mesh filename="file://$(find mycobot_description)/meshes/baseArm_v1_1.stl" scale="0.001 0.001 0.001"/>
-    </geometry>
-  </collision>
-</link>
-<link name="lowerArm_v1_1">
+      <mesh filename="file://$(find mycobot_description)/meshes/baseArm.stl" scale="0.001 0.001 0.001"/>
+    </geometry>
+  </collision>
+</link>
+<link name="lowerArm">
   <inertial>
     <origin xyz="0.03690658575566909 2.2563486026873027e-14 0.06799999999999196" rpy="0 0 0"/>
@@ -233,5 +233,5 @@
     <origin xyz="-0.045 -0.0 -0.716" rpy="0 0 0"/>
     <geometry>
-      <mesh filename="file://$(find mycobot_description)/meshes/lowerArm_v1_1.stl" scale="0.001 0.001 0.001"/>
+      <mesh filename="file://$(find mycobot_description)/meshes/lowerArm.stl" scale="0.001 0.001 0.001"/>
     </geometry>
     <material name="silver"/>
@@ -240,9 +240,9 @@
     <origin xyz="-0.045 -0.0 -0.716" rpy="0 0 0"/>
     <geometry>
-      <mesh filename="file://$(find mycobot_description)/meshes/lowerArm_v1_1.stl" scale="0.001 0.001 0.001"/>
-    </geometry>
-  </collision>
-</link>
-<link name="upperArm_v1_1">
+      <mesh filename="file://$(find mycobot_description)/meshes/lowerArm.stl" scale="0.001 0.001 0.001"/>
+    </geometry>
+  </collision>
+</link>
+<link name="upperArm">
   <inertial>
     <origin xyz="-0.035022688252996176 2.6167507160751738e-14 0.04949999999999111" rpy="0 0 0"/>
@@ -253,5 +253,5 @@
     <origin xyz="-0.045 -0.0 -0.852" rpy="0 0 0"/>
     <geometry>
-      <mesh filename="file://$(find mycobot_description)/meshes/upperArm_v1_1.stl" scale="0.001 0.001 0.001"/>
+      <mesh filename="file://$(find mycobot_description)/meshes/upperArm.stl" scale="0.001 0.001 0.001"/>
     </geometry>
     <material name="silver"/>
@@ -260,9 +260,9 @@
     <origin xyz="-0.045 -0.0 -0.852" rpy="0 0 0"/>
     <geometry>
-      <mesh filename="file://$(find mycobot_description)/meshes/upperArm_v1_1.stl" scale="0.001 0.001 0.001"/>
-    </geometry>
-  </collision>
-</link>
-<link name="pitchArm_v1_1">
+      <mesh filename="file://$(find mycobot_description)/meshes/upperArm.stl" scale="0.001 0.001 0.001"/>
+    </geometry>
+  </collision>
+</link>
+<link name="pitchArm">
   <inertial>
     <origin xyz="0.0344238728691882 2.9930072914790985e-14 0.010576127130799029" rpy="0 0 0"/>
@@ -273,5 +273,5 @@
     <origin xyz="-0.045 -0.0 -0.951" rpy="0 0 0"/>
     <geometry>
-      <mesh filename="file://$(find mycobot_description)/meshes/pitchArm_v1_1.stl" scale="0.001 0.001 0.001"/>
+      <mesh filename="file://$(find mycobot_description)/meshes/pitchArm.stl" scale="0.001 0.001 0.001"/>
     </geometry>
     <material name="silver"/>
@@ -280,9 +280,9 @@
     <origin xyz="-0.045 -0.0 -0.951" rpy="0 0 0"/>
     <geometry>
-      <mesh filename="file://$(find mycobot_description)/meshes/pitchArm_v1_1.stl" scale="0.001 0.001 0.001"/>
-    </geometry>
-  </collision>
-</link>
-<link name="rollArm_v1_1">
+      <mesh filename="file://$(find mycobot_description)/meshes/pitchArm.stl" scale="0.001 0.001 0.001"/>
+    </geometry>
+  </collision>
+</link>
+<link name="rollArm">
   <inertial>
     <origin xyz="-4.052314039881821e-15 3.104263161282912e-14 0.04211669650612482" rpy="0 0 0"/>
@@ -293,5 +293,5 @@
     <origin xyz="-0.09 -0.0 -0.996" rpy="0 0 0"/>
     <geometry>
-      <mesh filename="file://$(find mycobot_description)/meshes/rollArm_v1_1.stl" scale="0.001 0.001 0.001"/>
+      <mesh filename="file://$(find mycobot_description)/meshes/rollArm.stl" scale="0.001 0.001 0.001"/>
     </geometry>
     <material name="silver"/>
@@ -300,9 +300,9 @@
     <origin xyz="-0.09 -0.0 -0.996" rpy="0 0 0"/>
     <geometry>
-      <mesh filename="file://$(find mycobot_description)/meshes/rollArm_v1_1.stl" scale="0.001 0.001 0.001"/>
-    </geometry>
-  </collision>
-</link>
-<link name="gripperArm_v1_1">
+      <mesh filename="file://$(find mycobot_description)/meshes/rollArm.stl" scale="0.001 0.001 0.001"/>
+    </geometry>
+  </collision>
+</link>
+<link name="gripperArm">
   <inertial>
     <origin xyz="0.009999999999995929 3.104852866283627e-14 -9.325873406851315e-15" rpy="0 0 0"/>
@@ -313,5 +313,5 @@
     <origin xyz="-0.13 -0.0 -1.046" rpy="0 0 0"/>
     <geometry>
-      <mesh filename="file://$(find mycobot_description)/meshes/gripperArm_v1_1.stl" scale="0.001 0.001 0.001"/>
+      <mesh filename="file://$(find mycobot_description)/meshes/gripperArm.stl" scale="0.001 0.001 0.001"/>
     </geometry>
     <material name="silver"/>
@@ -320,9 +320,9 @@
     <origin xyz="-0.13 -0.0 -1.046" rpy="0 0 0"/>
     <geometry>
-      <mesh filename="file://$(find mycobot_description)/meshes/gripperArm_v1_1.stl" scale="0.001 0.001 0.001"/>
-    </geometry>
-  </collision>
-</link>
-<link name="cobot_camera_1">
+      <mesh filename="file://$(find mycobot_description)/meshes/gripperArm.stl" scale="0.001 0.001 0.001"/>
+    </geometry>
+  </collision>
+</link>
+<link name="cobot_camera">
   <inertial>
     <origin xyz="0.004999999999995952 3.105530767256797e-14 0.02345781668822733" rpy="0 0 0"/>
@@ -333,5 +333,5 @@
     <origin xyz="-0.15 -0.0 -1.046" rpy="0 0 0"/>
     <geometry>
-      <mesh filename="file://$(find mycobot_description)/meshes/cobot_camera_1.stl" scale="0.001 0.001 0.001"/>
+      <mesh filename="file://$(find mycobot_description)/meshes/cobot_camera.stl" scale="0.001 0.001 0.001"/>
     </geometry>
     <material name="silver"/>
@@ -340,9 +340,9 @@
     <origin xyz="-0.15 -0.0 -1.046" rpy="0 0 0"/>
     <geometry>
-      <mesh filename="file://$(find mycobot_description)/meshes/cobot_camera_1.stl" scale="0.001 0.001 0.001"/>
-    </geometry>
-  </collision>
-</link>
-<link name="gripper_base_1">
+      <mesh filename="file://$(find mycobot_description)/meshes/cobot_camera.stl" scale="0.001 0.001 0.001"/>
+    </geometry>
+  </collision>
+</link>
+<link name="gripper_base">
   <inertial>
     <origin xyz="0.035566484314994706 -0.00017560554917522554 0.00832682194458001" rpy="0 0 0"/>
@@ -353,5 +353,5 @@
     <origin xyz="-0.16 -0.0 -1.046" rpy="0 0 0"/>
     <geometry>
-      <mesh filename="file://$(find mycobot_description)/meshes/gripper_base_1.stl" scale="0.001 0.001 0.001"/>
+      <mesh filename="file://$(find mycobot_description)/meshes/gripper_base.stl" scale="0.001 0.001 0.001"/>
     </geometry>
     <material name="silver"/>
@@ -360,9 +360,9 @@
     <origin xyz="-0.16 -0.0 -1.046" rpy="0 0 0"/>
     <geometry>
-      <mesh filename="file://$(find mycobot_description)/meshes/gripper_base_1.stl" scale="0.001 0.001 0.001"/>
-    </geometry>
-  </collision>
-</link>
-<link name="gripper_left3_1">
+      <mesh filename="file://$(find mycobot_description)/meshes/gripper_base.stl" scale="0.001 0.001 0.001"/>
+    </geometry>
+  </collision>
+</link>
+<link name="gripper_left3">
   <inertial>
     <origin xyz="0.015990426629757803 -0.012967523057076307 0.0034753903195710034" rpy="0 0 0"/>
@@ -373,5 +373,5 @@
     <origin xyz="-0.22039 0.01846 -1.049642" rpy="0 0 0"/>
     <geometry>
-      <mesh filename="file://$(find mycobot_description)/meshes/gripper_left3_1.stl" scale="0.001 0.001 0.001"/>
+      <mesh filename="file://$(find mycobot_description)/meshes/gripper_left3.stl" scale="0.001 0.001 0.001"/>
     </geometry>
     <material name="silver"/>
@@ -380,9 +380,9 @@
     <origin xyz="-0.22039 0.01846 -1.049642" rpy="0 0 0"/>
     <geometry>
-      <mesh filename="file://$(find mycobot_description)/meshes/gripper_left3_1.stl" scale="0.001 0.001 0.001"/>
-    </geometry>
-  </collision>
-</link>
-<link name="gripper_left1_1">
+      <mesh filename="file://$(find mycobot_description)/meshes/gripper_left3.stl" scale="0.001 0.001 0.001"/>
+    </geometry>
+  </collision>
+</link>
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
Commit message: modify link names

File: mycobot_description/urdf/mycobot.xacro (robot description, xacro)
@@ -102,5 +102,5 @@
   </collision>
 </link>
-<link name="XL430_base_right">
+<link name="base_right">
   <inertial>
     <origin xyz="0.015671495929223667 -0.00632193052184804 0.014483637367895638" rpy="0 0 0"/>
@@ -122,5 +122,5 @@
   </collision>
 </link>
-<link name="XL430_motor_right">
+<link name="motor_right">
   <inertial>
     <origin xyz="-3.045443770730309e-06 -0.002385176775222958 6.646072581162343e-14" rpy="0 0 0"/>
@@ -162,5 +162,5 @@
   </collision>
 </link>
-<link name="plate">
+<link name="base_plate">
   <inertial>
     <origin xyz="2.349014429479716e-17 2.217469621428852e-14 0.009999999999990572" rpy="0 0 0"/>
@@ -442,5 +442,5 @@
   </collision>
 </link>
-<link name="Intel_Realsense_D435">
+<link name="camera_link">
   <inertial>
     <origin xyz="0.0015201693083259915 -5.299270958027507e-07 0.012451799923456464" rpy="0 0 0"/>
@@ -482,5 +482,5 @@
   </collision>
 </link>
-<link name="XL430_base_left">
+<link name="base_left">
   <inertial>
     <origin xyz="0.015671495929223758 0.006321930521842017 0.014516362632086596" rpy="0 0 0"/>
@@ -502,5 +502,5 @@
   </collision>
 </link>
-<link name="XL430_motor_left">
+<link name="motor_left">
   <inertial>
     <origin xyz="-3.0454437706458498e-06 0.0023851767752167963 -8.416878305439468e-14" rpy="0 0 0"/>
@@ -566,10 +566,10 @@
   <origin xyz="-0.028 -0.198 0.0855" rpy="0 0 0"/>
   <parent link="base_link"/>
-  <child link="XL430_base_right"/>
+  <child link="base_right"/>
 </joint>
 <joint name="wheel_left" type="revolute">
   <origin xyz="0.0283 0.0208 0.0145" rpy="0 0 0"/>
-  <parent link="XL430_base_left"/>
-  <child link="XL430_motor_left"/>
+  <parent link="base_left"/>
+  <child link="motor_left"/>
   <axis xyz="0.0 1.0 -0.0"/>
   <limit upper="6.283185" lower="0.0" effort="100" velocity="100"/>
@@ -577,6 +577,6 @@
 <joint name="wheel_right" type="revolute">
   <origin xyz="0.0283 -0.0208 0.0145" rpy="0 0 0"/>
-  <parent link="XL430_base_right"/>
-  <child link="XL430_motor_right"/>
+  <parent link="base_right"/>
+  <child link="motor_right"/>
   <axis xyz="-0.0 -1.0 0.0"/>
   <limit upper="6.283185" lower="0.0" effort="100" velocity="100"/>
@@ -584,5 +584,5 @@
 <joint name="Rigid 14" type="fixed">
   <origin xyz="0.005657 -0.0045 0.005657" rpy="0 0 0"/>
-  <parent link="XL430_motor_right"/>
+  <parent link="motor_right"/>
   <child link="wheel_right"/>
 </joint>
@@ -590,9 +590,9 @@
   <origin xyz="0.0 0.0 0.501" rpy="0 0 0"/>
   <parent link="base_link"/>
-  <child link="plate"/>
+  <child link="base_plate"/>
 </joint>
 <joint name="Rigid 23" type="fixed">
   <origin xyz="0.0 0.0 0.02" rpy="0 0 0"/>
-  <parent link="plate"/>
+  <parent link="base_plate"/>
   <child link="cobot_body"/>
 </joint>
@@ -683,5 +683,5 @@
   <origin xyz="0.0 0.0 0.11" rpy="0 0 0"/>
   <parent link="camera_stand"/>
-  <child link="Intel_Realsense_D435"/>
+  <child link="camera_link"/>
 </joint>
 <joint name="Rigid 40" type="fixed">
@@ -693,9 +693,9 @@
   <origin xyz="-0.028 0.198 0.0855" rpy="0 0 0"/>
   <parent link="base_link"/>
-  <child link="XL430_base_left"/>
+  <child link="base_left"/>
 </joint>
 <joint name="Rigid 44" type="fixed">
   <origin xyz="0.005657 0.0045 0.005657" rpy="0 0 0"/>
-  <parent link="XL430_motor_left"/>
+  <parent link="motor_left"/>
   <child link="wheel_left"/>
 </joint>
