Commit message: edit camera joint
카메라 조인트 수정, urdf fixed error

File: moiro_description/urdf/moiro.xacro (robot description, xacro)
@@ -6,7 +6,7 @@
 <link name="base_link">
   <inertial>
-    <origin xyz="0.005819797182780474 -0.0010588947341958668 0.274544607630003" rpy="0 0 0"/>
-    <mass value="8.753439823620923"/>
-    <inertia ixx="0.441696" iyy="0.493187" izz="0.405783" ixy="0.002051" iyz="0.002233" ixz="-0.012182"/>
+    <origin xyz="0.005355263561054088 -0.0009743746798552673 0.2595502059875776" rpy="0 0 0"/>
+    <mass value="9.51274328475089"/>
+    <inertia ixx="0.485755" iyy="0.519524" izz="0.426856" ixy="0.002055" iyz="0.002374" ixz="-0.012946"/>
   </inertial>
   <visual>
@@ -24,5 +24,5 @@
   </collision>
 </link>
-<link name="baseArm_v1">
+<link name="basearm">
   <inertial>
     <origin xyz="0.006896766224728663 -2.0858239854097905e-15 0.05549018686904683" rpy="0 0 0"/>
@@ -33,5 +33,5 @@
     <origin xyz="0.0 0.0 -0.609" rpy="0 0 0"/>
     <geometry>
-      <mesh filename="file://$(find moiro_description)/meshes/baseArm_v1.stl" scale="0.001 0.001 0.001"/>
+      <mesh filename="file://$(find moiro_description)/meshes/basearm.stl" scale="0.001 0.001 0.001"/>
     </geometry>
     <material name="silver"/>
@@ -40,9 +40,9 @@
     <origin xyz="0.0 0.0 -0.609" rpy="0 0 0"/>
     <geometry>
-      <mesh filename="file://$(find moiro_description)/meshes/baseArm_v1.stl" scale="0.001 0.001 0.001"/>
-    </geometry>
-  </collision>
-</link>
-<link name="lowerArm_v1">
+      <mesh filename="file://$(find moiro_description)/meshes/basearm.stl" scale="0.001 0.001 0.001"/>
+    </geometry>
+  </collision>
+</link>
+<link name="lowerarm">
   <inertial>
     <origin xyz="0.036906585755669324 -2.1012286881994426e-15 0.06799999999999129" rpy="0 0 0"/>
@@ -53,5 +53,5 @@
     <origin xyz="-0.045 0.0 -0.694" rpy="0 0 0"/>
     <geometry>
-      <mesh filename="file://$(find moiro_description)/meshes/lowerArm_v1.stl" scale="0.001 0.001 0.001"/>
+      <mesh filename="file://$(find moiro_description)/meshes/lowerarm.stl" scale="0.001 0.001 0.001"/>
     </geometry>
     <material name="silver"/>
@@ -60,9 +60,9 @@
     <origin xyz="-0.045 0.0 -0.694" rpy="0 0 0"/>
     <geometry>
-      <mesh filename="file://$(find moiro_description)/meshes/lowerArm_v1.stl" scale="0.001 0.001 0.001"/>
-    </geometry>
-  </collision>
-</link>
-<link name="upperArm_v1">
+      <mesh filename="file://$(find moiro_description)/meshes/lowerarm.stl" scale="0.001 0.001 0.001"/>
+    </geometry>
+  </collision>
+</link>
+<link name="upperarm">
   <inertial>
     <origin xyz="-0.03502268825299596 1.5066088373264134e-15 0.04949999999999122" rpy="0 0 0"/>
@@ -73,5 +73,5 @@
     <origin xyz="-0.045 0.0 -0.83" rpy="0 0 0"/>
     <geometry>
-      <mesh filename="file://$(find moiro_description)/meshes/upperArm_v1.stl" scale="0.001 0.001 0.001"/>
+      <mesh filename="file://$(find moiro_description)/meshes/upperarm.stl" scale="0.001 0.001 0.001"/>
     </geometry>
     <material name="silver"/>
@@ -80,9 +80,9 @@
     <origin xyz="-0.045 0.0 -0.83" rpy="0 0 0"/>
     <geometry>
-      <mesh filename="file://$(find moiro_description)/meshes/upperArm_v1.stl" scale="0.001 0.001 0.001"/>
-    </geometry>
-  </collision>
-</link>
-<link name="pitchArm_v1">
+      <mesh filename="file://$(find moiro_description)/meshes/upperarm.stl" scale="0.001 0.001 0.001"/>
+    </geometry>
+  </collision>
+</link>
+<link name="pitcharm">
   <inertial>
     <origin xyz="0.034423872869188424 5.2920035523095135e-15 0.010576127130799362" rpy="0 0 0"/>
@@ -93,5 +93,5 @@
     <origin xyz="-0.045 -0.0 -0.929" rpy="0 0 0"/>
     <geometry>
-      <mesh filename="file://$(find moiro_description)/meshes/pitchArm_v1.stl" scale="0.001 0.001 0.001"/>
+      <mesh filename="file://$(find moiro_description)/meshes/pitcharm.stl" scale="0.001 0.001 0.001"/>
     </geometry>
     <material name="silver"/>
@@ -100,9 +100,9 @@
     <origin xyz="-0.045 -0.0 -0.929" rpy="0 0 0"/>
     <geometry>
-      <mesh filename="file://$(find moiro_description)/meshes/pitchArm_v1.stl" scale="0.001 0.001 0.001"/>
-    </geometry>
-  </collision>
-</link>
-<link name="rollArm">
+      <mesh filename="file://$(find moiro_description)/meshes/pitcharm.stl" scale="0.001 0.001 0.001"/>
+    </geometry>
+  </collision>
+</link>
+<link name="rollarm">
   <inertial>
     <origin xyz="-3.802513859341161e-15 6.3512715451656364e-15 0.042116696506125484" rpy="0 0 0"/>
@@ -113,5 +113,5 @@
     <origin xyz="-0.09 -0.0 -0.974" rpy="0 0 0"/>
     <geometry>
-      <mesh filename="file://$(find moiro_description)/meshes/rollArm.stl" scale="0.001 0.001 0.001"/>
+      <mesh filename="file://$(find moiro_description)/meshes/rollarm.stl" scale="0.001 0.001 0.001"/>
     </geometry>
     <material name="silver"/>
@@ -120,9 +120,9 @@
     <origin xyz="-0.09 -0.0 -0.974" rpy="0 0 0"/>
     <geometry>
-      <mesh filename="file://$(find moiro_description)/meshes/rollArm.stl" scale="0.001 0.001 0.001"/>
-    </geometry>
-  </collision>
-</link>
-<link name="gripperArm">
+      <mesh filename="file://$(find moiro_description)/meshes/rollarm.stl" scale="0.001 0.001 0.001"/>
+    </geometry>
+  </collision>
+</link>
+<link name="gripperarm">
   <inertial>
     <origin xyz="0.00999999999999615 6.341593916658894e-15 -9.103828801926284e-15" rpy="0 0 0"/>
@@ -133,5 +133,5 @@
     <origin xyz="-0.13 -0.0 -1.024" rpy="0 0 0"/>
     <geometry>
-      <mesh filename="file://$(find moiro_description)/meshes/gripperArm.stl" scale="0.001 0.001 0.001"/>
+      <mesh filename="file://$(find moiro_description)/meshes/gripperarm.stl" scale="0.001 0.001 0.001"/>
     </geometry>
     <material name="silver"/>
@@ -140,5 +140,5 @@
     <origin xyz="-0.13 -0.0 -1.024" rpy="0 0 0"/>
     <geometry>
-      <mesh filename="file://$(find moiro_description)/meshes/gripperArm.stl" scale="0.001 0.001 0.001"/>
+      <mesh filename="file://$(find moiro_description)/meshes/gripperarm.stl" scale="0.001 0.001 0.001"/>
     </geometry>
   </collision>
@@ -146,7 +146,7 @@
 <link name="cobot_camera">
   <inertial>
-    <origin xyz="0.004999999999996174 6.363947604904578e-15 0.023457816688227107" rpy="0 0 0"/>
-    <mass value="0.5631767017754145"/>
-    <inertia ixx="0.000724" iyy="0.000514" izz="0.000219" ixy="-0.0" iyz="-0.0" ixz="0.0"/>
+    <origin xyz="0.004999999999996174 6.363947604904578e-15 0.023457816688226885" rpy="0 0 0"/>
+    <mass value="0.07891648050356126"/>
+    <inertia ixx="0.000101" iyy="7.2e-05" izz="3.1e-05" ixy="-0.0" iyz="-0.0" ixz="0.0"/>
   </inertial>
   <visual>
@@ -167,6 +167,6 @@
   <inertial>
     <origin xyz="0.035566484314994956 -0.00017560554919991735 0.008326821944580676" rpy="0 0 0"/>
-    <mass value="0.5510932173775136"/>
-    <inertia ixx="0.000508" iyy="0.00049" izz="0.000702" ixy="0.0" iyz="0.0" ixz="-0.000104"/>
+    <mass value="0.0772232533904796"/>
+    <inertia ixx="7.1e-05" iyy="6.9e-05" izz="9.8e-05" ixy="0.0" iyz="0.0" ixz="-1.5e-05"/>
   </inertial>
   <visual>
@@ -186,7 +186,7 @@
 <link name="gripper_left3">
   <inertial>
-    <origin xyz="0.015990426629758026 -0.012967523057101037 0.0034753903195710034" rpy="0 0 0"/>
-    <mass value="0.09059526730883281"/>
-    <inertia ixx="1.8e-05" iyy="3.3e-05" izz="5e-05" ixy="1.8e-05" iyz="0.0" ixz="-0.0"/>
+    <origin xyz="0.015990426629758026 -0.012967523057101044 0.0034753903195707814" rpy="0 0 0"/>
+    <mass value="0.012694878221619885"/>
+    <inertia ixx="2e-06" iyy="5e-06" izz="7e-06" ixy="3e-06" iyz="0.0" ixz="-0.0"/>
   </inertial>
   <visual>
@@ -207,6 +207,6 @@
   <inertial>
     <origin xyz="0.011053309239173859 -0.005253691764351268 0.0001366080392810609" rpy="0 0 0"/>
-    <mass value="0.09307370524687981"/>
-    <inertia ixx="1e-05" iyy="3.5e-05" izz="4.2e-05" ixy="-1.3e-05" iyz="0.0" ixz="0.0"/>
+    <mass value="0.013042175257524559"/>
+    <inertia ixx="1e-06" iyy="5e-06" izz="6e-06" ixy="-2e-06" iyz="0.0" ixz="0.0"/>
   </inertial>
   <visual>
@@ -227,6 +227,6 @@
   <inertial>
     <origin xyz="0.01599042559398811 0.012967524435816866 0.0035248809278745075" rpy="0 0 0"/>
-    <mass value="0.09059526730883281"/>
-    <inertia ixx="1.8e-05" iyy="3.3e-05" izz="5e-05" ixy="-1.8e-05" iyz="0.0" ixz="0.0"/>
+    <mass value="0.012694878221619885"/>
+    <inertia ixx="2e-06" iyy="5e-06" izz="7e-06" ixy="-3e-06" iyz="0.0" ixz="0.0"/>
   </inertial>
   <visual>
@@ -247,6 +247,6 @@
   <inertial>
     <origin xyz="0.011053308203403722 0.0052536931430675685 -0.00013633679183122638" rpy="0 0 0"/>
-    <mass value="0.09307370524687981"/>
-    <inertia ixx="1e-05" iyy="3.5e-05" izz="4.2e-05" ixy="1.3e-05" iyz="0.0" ixz="-0.0"/>
+    <mass value="0.013042175257524559"/>
+    <inertia ixx="1e-06" iyy="5e-06" izz="6e-06" ixy="2e-06" iyz="0.0" ixz="-0.0"/>
   </inertial>
   <visual>
@@ -261,24 +261,4 @@
     <geometry>
       <mesh filename="file://$(find moiro_description)/meshes/gripper_right1.stl" scale="0.001 0.001 0.001"/>
-    </geometry>
-  </collision>
-</link>
-<link name="motor_left">
-  <inertial>
-    <origin xyz="0.016114155240641678 0.006913170455318668 0.014515788868055365" rpy="0 0 0"/>
-    <mass value="0.33572652306107803"/>
-    <inertia ixx="5.4e-05" iyy="8.2e-05" izz="9.1e-05" ixy="-3e-06" iyz="0.0" ixz="0.0"/>
-  </inertial>
-  <visual>
-    <origin xyz="0.028 -0.198 -0.0855" rpy="0 0 0"/>
-    <geometry>
-      <mesh filename="file://$(find moiro_description)/meshes/motor_left.stl" scale="0.001 0.001 0.001"/>
-    </geometry>
-    <material name="silver"/>
-  </visual>
-  <collision>
-    <origin xyz="0.028 -0.198 -0.0855" rpy="0 0 0"/>
-    <geometry>
-      <mesh filename="file://$(find moiro_description)/meshes/motor_left.stl" scale="0.001 0.001 0.001"/>
     </geometry>
   </collision>
@@ -304,12 +284,132 @@
   </collision>
 </link>
+<link name="wheel_right">
+  <inertial>
+    <origin xyz="7.185686845753172e-07 -0.013441732021015451 6.740004032668168e-08" rpy="0 0 0"/>
+    <mass value="0.6403675217821955"/>
+    <inertia ixx="0.00197" iyy="0.003862" izz="0.00197" ixy="0.0" iyz="0.0" ixz="-0.0"/>
+  </inertial>
+  <visual>
+    <origin xyz="-0.000298 0.2233 -0.1055" rpy="0 0 0"/>
+    <geometry>
+      <mesh filename="file://$(find moiro_description)/meshes/wheel_right.stl" scale="0.001 0.001 0.001"/>
+    </geometry>
+    <material name="silver"/>
+  </visual>
+  <collision>
+    <origin xyz="-0.000298 0.2233 -0.1055" rpy="0 0 0"/>
+    <geometry>
+      <mesh filename="file://$(find moiro_description)/meshes/wheel_right.stl" scale="0.001 0.001 0.001"/>
+    </geometry>
+  </collision>
+</link>
+<link name="wheel_left">
+  <inertial>
+    <origin xyz="5.370332256415832e-07 0.013441732021011232 2.8938916790677283e-08" rpy="0 0 0"/>
+    <mass value="0.6403675217821955"/>
+    <inertia ixx="0.00197" iyy="0.003862" izz="0.00197" ixy="-0.0" iyz="0.0" ixz="0.0"/>
+  </inertial>
+  <visual>
+    <origin xyz="-0.000298 -0.2233 -0.1055" rpy="0 0 0"/>
+    <geometry>
+      <mesh filename="file://$(find moiro_description)/meshes/wheel_left.stl" scale="0.001 0.001 0.001"/>
+    </geometry>
+    <material name="silver"/>
+  </visual>
+  <collision>
+    <origin xyz="-0.000298 -0.2233 -0.1055" rpy="0 0 0"/>
+    <geometry>
+      <mesh filename="file://$(find moiro_description)/meshes/wheel_left.stl" scale="0.001 0.001 0.001"/>
+    </geometry>
+  </collision>
+</link>
+<link name="caster_4">
+  <inertial>
+    <origin xyz="-0.020672705075060666 -0.0093964574939722 -0.02565460037687653" rpy="0 0 0"/>
+    <mass value="0.14564908217460187"/>
+    <inertia ixx="4.1e-05" iyy="5.4e-05" izz="2.2e-05" ixy="0.0" iyz="0.0" ixz="0.0"/>
+  </inertial>
+  <visual>
+    <origin xyz="-0.238132 0.037118 -0.058" rpy="0 0 0"/>
+    <geometry>
+      <mesh filename="file://$(find moiro_description)/meshes/caster_4.stl" scale="0.001 0.001 0.001"/>
+    </geometry>
+    <material name="silver"/>
+  </visual>
+  <collision>
+    <origin xyz="-0.238132 0.037118 -0.058" rpy="0 0 0"/>
+    <geometry>
+      <mesh filename="file://$(find moiro_description)/meshes/caster_4.stl" scale="0.001 0.001 0.001"/>
+    </geometry>
+  </collision>
+</link>
+<link name="caster_3">
+  <inertial>
+    <origin xyz="-0.02067270507506075 0.006390241409318889 -0.02565460037687651" rpy="0 0 0"/>
+    <mass value="0.14564908217460187"/>
+    <inertia ixx="4.1e-05" iyy="5.4e-05" izz="2.2e-05" ixy="0.0" iyz="0.0" ixz="0.0"/>
+  </inertial>
+  <visual>
+    <origin xyz="-0.238132 -0.040529 -0.058" rpy="0 0 0"/>
+    <geometry>
+      <mesh filename="file://$(find moiro_description)/meshes/caster_3.stl" scale="0.001 0.001 0.001"/>
+    </geometry>
+    <material name="silver"/>
+  </visual>
+  <collision>
+    <origin xyz="-0.238132 -0.040529 -0.058" rpy="0 0 0"/>
+    <geometry>
+      <mesh filename="file://$(find moiro_description)/meshes/caster_3.stl" scale="0.001 0.001 0.001"/>
+    </geometry>
+  </collision>
+</link>
+<link name="caster_6">
+  <inertial>
+    <origin xyz="0.02067255115624625 0.009396455766248653 -0.02565460037687644" rpy="0 0 0"/>
+    <mass value="0.14564908217460187"/>
+    <inertia ixx="4.1e-05" iyy="5.4e-05" izz="2.2e-05" ixy="0.0" iyz="0.0" ixz="0.0"/>
+  </inertial>
+  <visual>
+    <origin xyz="0.238132 -0.037118 -0.058" rpy="0 0 0"/>
+    <geometry>
+      <mesh filename="file://$(find moiro_description)/meshes/caster_6.stl" scale="0.001 0.001 0.001"/>
+    </geometry>
+    <material name="silver"/>
+  </visual>
+  <collision>
+    <origin xyz="0.238132 -0.037118 -0.058" rpy="0 0 0"/>
+    <geometry>
+      <mesh filename="file://$(find moiro_description)/meshes/caster_6.stl" scale="0.001 0.001 0.001"/>
+    </geometry>
+  </collision>
+</link>
+<link name="caster_5">
+  <inertial>
+    <origin xyz="0.02067255115624622 -0.006390243137041694 -0.025654600376876474" rpy="0 0 0"/>
+    <mass value="0.14564908217460187"/>
+    <inertia ixx="4.1e-05" iyy="5.4e-05" izz="2.2e-05" ixy="0.0" iyz="0.0" ixz="0.0"/>
+  </inertial>
+  <visual>
+    <origin xyz="0.238132 0.040529 -0.058" rpy="0 0 0"/>
+    <geometry>
+      <mesh filename="file://$(find moiro_description)/meshes/caster_5.stl" scale="0.001 0.001 0.001"/>
+    </geometry>
+    <material name="silver"/>
+  </visual>
+  <collision>
+    <origin xyz="0.238132 0.040529 -0.058" rpy="0 0 0"/>
+    <geometry>
+      <mesh filename="file://$(find moiro_description)/meshes/caster_5.stl" scale="0.001 0.001 0.001"/>
+    </geometry>
+  </collision>
+</link>
 <link name="motor_right">
   <inertial>
-    <origin xyz="-0.00788584475935841 -0.006913170455324746 0.014484211131926869" rpy="0 0 0"/>
-    <mass value="0.3357265230610785"/>
-    <inertia ixx="5.4e-05" iyy="8.2e-05" izz="9.1e-05" ixy="3e-06" iyz="0.0" ixz="-0.0"/>
-  </inertial>
-  <visual>
-    <origin xyz="0.004 0.198 -0.0855" rpy="0 0 0"/>
+    <origin xyz="-0.00788584475935802 -0.006913170455323303 0.01448421113192662" rpy="0 0 0"/>
+    <mass value="0.055170345827871496"/>
+    <inertia ixx="9e-06" iyy="1.3e-05" izz="1.5e-05" ixy="0.0" iyz="0.0" ixz="-0.0"/>
+  </inertial>
+  <visual>
+    <origin xyz="0.004 0.198 -0.091" rpy="0 0 0"/>
     <geometry>
       <mesh filename="file://$(find moiro_description)/meshes/motor_right.stl" scale="0.001 0.001 0.001"/>
@@ -318,5 +418,5 @@
   </visual>
   <collision>
-    <origin xyz="0.004 0.198 -0.0855" rpy="0 0 0"/>
+    <origin xyz="0.004 0.198 -0.091" rpy="0 0 0"/>
     <geometry>
       <mesh filename="file://$(find moiro_description)/meshes/motor_right.stl" scale="0.001 0.001 0.001"/>
@@ -324,121 +424,41 @@
   </collision>
 </link>
-<link name="wheel_right">
-  <inertial>
-    <origin xyz="7.185686850442346e-07 -0.013441732021016534 6.740003920258086e-08" rpy="0 0 0"/>
-    <mass value="5.405252737623909"/>
-    <inertia ixx="0.01663" iyy="0.032598" izz="0.01663" ixy="0.0" iyz="0.0" ixz="-0.0"/>
-  </inertial>
-  <visual>
-    <origin xyz="-0.000298 0.2233 -0.1" rpy="0 0 0"/>
-    <geometry>
-      <mesh filename="file://$(find moiro_description)/meshes/wheel_right.stl" scale="0.001 0.001 0.001"/>
-    </geometry>
-    <material name="silver"/>
-  </visual>
-  <collision>
-    <origin xyz="-0.000298 0.2233 -0.1" rpy="0 0 0"/>
-    <geometry>
-      <mesh filename="file://$(find moiro_description)/meshes/wheel_right.stl" scale="0.001 0.001 0.001"/>
-    </geometry>
-  </collision>
-</link>
-<link name="wheel_left">
-  <inertial>
-    <origin xyz="-0.23429985498871683 -0.07855826797899002 -0.0003000192286679165" rpy="0 0 0"/>
-    <mass value="5.405252737623909"/>
-    <inertia ixx="0.01663" iyy="0.032598" izz="0.01663" ixy="-0.0" iyz="0.0" ixz="0.0"/>
-  </inertial>
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
Commit message: edit camera joint pitch

File: moiro_description/urdf/moiro.xacro (robot description, xacro)
@@ -446,7 +446,7 @@
 <link name="camera_zig">
   <inertial>
-    <origin xyz="-0.0032513672191570864 0.04404933875225113 0.031685069930480037" rpy="0 0 0"/>
+    <origin xyz="0.01453009991903656 0.044049338752250145 0.028344157098708522" rpy="0 0 0"/>
     <mass value="0.059863707592883605"/>
-    <inertia ixx="8.3e-05" iyy="4.8e-05" izz="6.1e-05" ixy="0.0" iyz="-5e-06" ixz="2e-05"/>
+    <inertia ixx="9.5e-05" iyy="4.8e-05" izz="4.9e-05" ixy="-3e-06" iyz="-5e-06" ixz="-2e-06"/>
   </inertial>
   <visual>
@@ -466,10 +466,10 @@
 <link name="camera_link">
   <inertial>
-    <origin xyz="0.010233937750200123 -5.299843264592978e-07 0.006588359530641186" rpy="0 0 0"/>
+    <origin xyz="0.012171542279409253 -5.299843283462433e-07 -4.8580261040487294e-05" rpy="0 0 0"/>
     <mass value="0.37833297071846606"/>
-    <inertia ixx="0.000239" iyy="3.5e-05" izz="0.000239" ixy="-0.0" iyz="0.0" ixz="-1e-06"/>
-  </inertial>
-  <visual>
-    <origin xyz="-0.242995 -0.00175 -0.564912" rpy="0 0 0"/>
+    <inertia ixx="0.000238" iyy="3.5e-05" izz="0.00024" ixy="-0.0" iyz="0.0" ixz="0.0"/>
+  </inertial>
+  <visual>
+    <origin xyz="-0.26675 -0.00175 -0.561285" rpy="0 0 0"/>
     <geometry>
       <mesh filename="file://$(find moiro_description)/meshes/camera_link.stl" scale="0.001 0.001 0.001"/>
@@ -478,5 +478,5 @@
   </visual>
   <collision>
-    <origin xyz="-0.242995 -0.00175 -0.564912" rpy="0 0 0"/>
+    <origin xyz="-0.26675 -0.00175 -0.561285" rpy="0 0 0"/>
     <geometry>
       <mesh filename="file://$(find moiro_description)/meshes/camera_link.stl" scale="0.001 0.001 0.001"/>
@@ -504,5 +504,4 @@
   </collision>
 </link>
-<!-- joint -->
 <joint name="Revolute 1" type="revolute">
   <origin xyz="0.0 0.0 0.09" rpy="0 0 0"/>
@@ -632,15 +631,15 @@
   <child link="motor_left"/>
 </joint>
-<joint name="joint_zig" type="fixed">
-  <origin xyz="0.24875 -0.045 0.523" rpy="0 0 0"/>
+<joint name="joint_camera" type="fixed">
+  <origin xyz="0.24875 -0.045 0.523" rpy="0 -0.575959 0"/>
   <parent link="base_link"/>
   <child link="camera_zig"/>
 </joint>
-<joint name="joint_camera" type="fixed">
-  <origin xyz="-0.005755 0.04675 0.041912" rpy="0 0 0"/>
+<joint name="Rigid 70" type="fixed">
+  <origin xyz="0.018 0.04675 0.038285" rpy="0 0 0"/>
   <parent link="camera_zig"/>
   <child link="camera_link"/>
 </joint>
-<joint name="base_plate_joint" type="fixed">
+<joint name="Rigid 71" type="fixed">
   <origin xyz="0.0 0.0 0.501" rpy="0 0 0"/>
   <parent link="base_link"/>

Commit message: add base_scan

File: moiro_description/urdf/moiro.xacro (robot description, xacro)
@@ -6,7 +6,7 @@
 <link name="base_link">
   <inertial>
-    <origin xyz="0.005355263561054088 -0.0009743746798552673 0.2595502059875776" rpy="0 0 0"/>
-    <mass value="9.51274328475089"/>
-    <inertia ixx="0.485755" iyy="0.519524" izz="0.426856" ixy="0.002055" iyz="0.002374" ixz="-0.012946"/>
+    <origin xyz="0.005150955585676035 -0.0009334785499818622 0.2594629875523824" rpy="0 0 0"/>
+    <mass value="9.890849791423904"/>
+    <inertia ixx="0.48614" iyy="0.520086" izz="0.427787" ixy="0.002057" iyz="0.002374" ixz="-0.01295"/>
   </inertial>
   <visual>
@@ -501,4 +501,24 @@
     <geometry>
       <mesh filename="file://$(find moiro_description)/meshes/base_plate.stl" scale="0.001 0.001 0.001"/>
+    </geometry>
+  </collision>
+</link>
+<link name="base_scan">
+  <inertial>
+    <origin xyz="1.4890131030019722e-05 -0.008617362464656674 0.01114526026515611" rpy="0 0 0"/>
+    <mass value="0.4177280575470181"/>
+    <inertia ixx="0.000281" iyy="0.000143" izz="0.000351" ixy="-0.0" iyz="-3.9e-05" ixz="-0.0"/>
+  </inertial>
+  <visual>
+    <origin xyz="0.000412 -0.003127 -0.271745" rpy="0 0 0"/>
+    <geometry>
+      <mesh filename="file://$(find moiro_description)/meshes/base_scan.stl" scale="0.001 0.001 0.001"/>
+    </geometry>
+    <material name="silver"/>
+  </visual>
+  <collision>
+    <origin xyz="0.000412 -0.003127 -0.271745" rpy="0 0 0"/>
+    <geometry>
+      <mesh filename="file://$(find moiro_description)/meshes/base_scan.stl" scale="0.001 0.001 0.001"/>
     </geometry>
   </collision>
@@ -641,8 +661,13 @@
   <child link="camera_link"/>
 </joint>
-<joint name="Rigid 71" type="fixed">
+<joint name="Rigid 74" type="fixed">
   <origin xyz="0.0 0.0 0.501" rpy="0 0 0"/>
   <parent link="base_link"/>
   <child link="base_plate"/>
 </joint>
+<joint name="joint_base_scan" type="fixed">
+  <origin xyz="-0.000412 0.003127 0.271745" rpy="0 0 0"/>
+  <parent link="base_link"/>
+  <child link="base_scan"/>
+</joint>
 </robot>
