Commit message: edit link, joint, add bracket
브라켓 추가, base_link 위치 수정, imu_link 추가

File: moiro_description/urdf/moiro.xacro (robot description, xacro)
@@ -4,9 +4,13 @@
 <xacro:include filename="$(find moiro_description)/urdf/moiro.trans" />
 <xacro:include filename="$(find moiro_description)/urdf/moiro.gazebo" />
+<!-- 240529 오후 12시 수정
+1. mycobot에 부착하는 카메라 링크, 브라켓 추가,
+2. imu_link 추가
+3. base_link 위치 수정 -->
 <link name="base_link">
   <inertial>
-    <origin xyz="0.005150955585676035 -0.0009334785499818622 0.2594629875523824" rpy="0 0 0"/>
-    <mass value="9.890849791423904"/>
-    <inertia ixx="0.48614" iyy="0.520086" izz="0.427787" ixy="0.002057" iyz="0.002374" ixz="-0.01295"/>
+    <origin xyz="0.004418404192394108 -0.0009320583420061628 0.2493907147199333" rpy="0 0 0"/>
+    <mass value="10.314151582114752"/>
+    <inertia ixx="0.498632" iyy="0.533352" izz="0.429421" ixy="0.002003" iyz="0.002378" ixz="-0.014194"/>
   </inertial>
   <visual>
@@ -26,10 +30,10 @@
 <link name="basearm">
   <inertial>
-    <origin xyz="0.006896766224728663 -2.0858239854097905e-15 0.05549018686904683" rpy="0 0 0"/>
+    <origin xyz="0.006896766224728663 -2.0863790969221033e-15 0.05549018686904683" rpy="0 0 0"/>
     <mass value="3.4735206294395446"/>
     <inertia ixx="0.004461" iyy="0.004757" izz="0.002424" ixy="0.0" iyz="0.0" ixz="-0.000777"/>
   </inertial>
   <visual>
-    <origin xyz="0.0 0.0 -0.609" rpy="0 0 0"/>
+    <origin xyz="0.0 0.0 -0.606" rpy="0 0 0"/>
     <geometry>
       <mesh filename="file://$(find moiro_description)/meshes/basearm.stl" scale="0.001 0.001 0.001"/>
@@ -38,5 +42,5 @@
   </visual>
   <collision>
-    <origin xyz="0.0 0.0 -0.609" rpy="0 0 0"/>
+    <origin xyz="0.0 0.0 -0.606" rpy="0 0 0"/>
     <geometry>
       <mesh filename="file://$(find moiro_description)/meshes/basearm.stl" scale="0.001 0.001 0.001"/>
@@ -46,10 +50,10 @@
 <link name="lowerarm">
   <inertial>
-    <origin xyz="0.036906585755669324 -2.1012286881994426e-15 0.06799999999999129" rpy="0 0 0"/>
+    <origin xyz="0.036906585755669324 -2.1017837997117547e-15 0.06799999999999129" rpy="0 0 0"/>
     <mass value="5.91988968680626"/>
     <inertia ixx="0.0188" iyy="0.019335" izz="0.004161" ixy="-0.0" iyz="0.0" ixz="0.0"/>
   </inertial>
   <visual>
-    <origin xyz="-0.045 0.0 -0.694" rpy="0 0 0"/>
+    <origin xyz="-0.045 0.0 -0.691" rpy="0 0 0"/>
     <geometry>
       <mesh filename="file://$(find moiro_description)/meshes/lowerarm.stl" scale="0.001 0.001 0.001"/>
@@ -58,5 +62,5 @@
   </visual>
   <collision>
-    <origin xyz="-0.045 0.0 -0.694" rpy="0 0 0"/>
+    <origin xyz="-0.045 0.0 -0.691" rpy="0 0 0"/>
     <geometry>
       <mesh filename="file://$(find moiro_description)/meshes/lowerarm.stl" scale="0.001 0.001 0.001"/>
@@ -66,10 +70,10 @@
 <link name="upperarm">
   <inertial>
-    <origin xyz="-0.03502268825299596 1.5066088373264134e-15 0.04949999999999122" rpy="0 0 0"/>
+    <origin xyz="-0.03502268825299596 1.5060537258141013e-15 0.04949999999999133" rpy="0 0 0"/>
     <mass value="4.802107093668197"/>
-    <inertia ixx="0.01014" iyy="0.010584" izz="0.003386" ixy="-0.0" iyz="-0.0" ixz="0.0"/>
-  </inertial>
-  <visual>
-    <origin xyz="-0.045 0.0 -0.83" rpy="0 0 0"/>
+    <inertia ixx="0.01014" iyy="0.010584" izz="0.003386" ixy="-0.0" iyz="-0.0" ixz="-0.0"/>
+  </inertial>
+  <visual>
+    <origin xyz="-0.045 0.0 -0.827" rpy="0 0 0"/>
     <geometry>
       <mesh filename="file://$(find moiro_description)/meshes/upperarm.stl" scale="0.001 0.001 0.001"/>
@@ -78,5 +82,5 @@
   </visual>
   <collision>
-    <origin xyz="-0.045 0.0 -0.83" rpy="0 0 0"/>
+    <origin xyz="-0.045 0.0 -0.827" rpy="0 0 0"/>
     <geometry>
       <mesh filename="file://$(find moiro_description)/meshes/upperarm.stl" scale="0.001 0.001 0.001"/>
@@ -86,10 +90,10 @@
 <link name="pitcharm">
   <inertial>
-    <origin xyz="0.034423872869188424 5.2920035523095135e-15 0.010576127130799362" rpy="0 0 0"/>
+    <origin xyz="0.034423872869188424 5.291448440797201e-15 0.010576127130799362" rpy="0 0 0"/>
     <mass value="2.265107015236222"/>
     <inertia ixx="0.001595" iyy="0.001803" izz="0.001595" ixy="-0.0" iyz="-0.0" ixz="-0.000324"/>
   </inertial>
   <visual>
-    <origin xyz="-0.045 -0.0 -0.929" rpy="0 0 0"/>
+    <origin xyz="-0.045 -0.0 -0.926" rpy="0 0 0"/>
     <geometry>
       <mesh filename="file://$(find moiro_description)/meshes/pitcharm.stl" scale="0.001 0.001 0.001"/>
@@ -98,5 +102,5 @@
   </visual>
   <collision>
-    <origin xyz="-0.045 -0.0 -0.929" rpy="0 0 0"/>
+    <origin xyz="-0.045 -0.0 -0.926" rpy="0 0 0"/>
     <geometry>
       <mesh filename="file://$(find moiro_description)/meshes/pitcharm.stl" scale="0.001 0.001 0.001"/>
@@ -106,10 +110,10 @@
 <link name="rollarm">
   <inertial>
-    <origin xyz="-3.802513859341161e-15 6.3512715451656364e-15 0.042116696506125484" rpy="0 0 0"/>
+    <origin xyz="-3.816391647148976e-15 6.350716433653324e-15 0.042116696506125595" rpy="0 0 0"/>
     <mass value="3.029827579494103"/>
     <inertia ixx="0.0025" iyy="0.002976" izz="0.002441" ixy="-0.0" iyz="-0.0" ixz="0.0"/>
   </inertial>
   <visual>
-    <origin xyz="-0.09 -0.0 -0.974" rpy="0 0 0"/>
+    <origin xyz="-0.09 -0.0 -0.971" rpy="0 0 0"/>
     <geometry>
       <mesh filename="file://$(find moiro_description)/meshes/rollarm.stl" scale="0.001 0.001 0.001"/>
@@ -118,5 +122,5 @@
   </visual>
   <collision>
-    <origin xyz="-0.09 -0.0 -0.974" rpy="0 0 0"/>
+    <origin xyz="-0.09 -0.0 -0.971" rpy="0 0 0"/>
     <geometry>
       <mesh filename="file://$(find moiro_description)/meshes/rollarm.stl" scale="0.001 0.001 0.001"/>
@@ -126,10 +130,10 @@
 <link name="gripperarm">
   <inertial>
-    <origin xyz="0.00999999999999615 6.341593916658894e-15 -9.103828801926284e-15" rpy="0 0 0"/>
+    <origin xyz="0.00999999999999615 6.341038805146582e-15 -9.103828801926284e-15" rpy="0 0 0"/>
     <mass value="0.6042068071016569"/>
     <inertia ixx="0.00037" iyy="0.000205" izz="0.000205" ixy="-0.0" iyz="0.0" ixz="-0.0"/>
   </inertial>
   <visual>
-    <origin xyz="-0.13 -0.0 -1.024" rpy="0 0 0"/>
+    <origin xyz="-0.13 -0.0 -1.021" rpy="0 0 0"/>
     <geometry>
       <mesh filename="file://$(find moiro_description)/meshes/gripperarm.stl" scale="0.001 0.001 0.001"/>
@@ -138,5 +142,5 @@
   </visual>
   <collision>
-    <origin xyz="-0.13 -0.0 -1.024" rpy="0 0 0"/>
+    <origin xyz="-0.13 -0.0 -1.021" rpy="0 0 0"/>
     <geometry>
       <mesh filename="file://$(find moiro_description)/meshes/gripperarm.stl" scale="0.001 0.001 0.001"/>
@@ -146,10 +150,10 @@
 <link name="cobot_camera">
   <inertial>
-    <origin xyz="0.004999999999996174 6.363947604904578e-15 0.023457816688226885" rpy="0 0 0"/>
-    <mass value="0.07891648050356126"/>
-    <inertia ixx="0.000101" iyy="7.2e-05" izz="3.1e-05" ixy="-0.0" iyz="-0.0" ixz="0.0"/>
-  </inertial>
-  <visual>
-    <origin xyz="-0.15 -0.0 -1.024" rpy="0 0 0"/>
+    <origin xyz="0.017423960091247193 0.003253426631193808 0.005819385718719872" rpy="0 0 0"/>
+    <mass value="0.21027144182469326"/>
+    <inertia ixx="0.000387" iyy="0.000194" izz="0.000246" ixy="-5e-06" iyz="2e-06" ixz="1.9e-05"/>
+  </inertial>
+  <visual>
+    <origin xyz="-0.15 -0.0 -1.021" rpy="0 0 0"/>
     <geometry>
       <mesh filename="file://$(find moiro_description)/meshes/cobot_camera.stl" scale="0.001 0.001 0.001"/>
@@ -158,5 +162,5 @@
   </visual>
   <collision>
-    <origin xyz="-0.15 -0.0 -1.024" rpy="0 0 0"/>
+    <origin xyz="-0.15 -0.0 -1.021" rpy="0 0 0"/>
     <geometry>
       <mesh filename="file://$(find moiro_description)/meshes/cobot_camera.stl" scale="0.001 0.001 0.001"/>
@@ -164,112 +168,12 @@
   </collision>
 </link>
-<link name="gripper_base">
-  <inertial>
-    <origin xyz="0.035566484314994956 -0.00017560554919991735 0.008326821944580676" rpy="0 0 0"/>
-    <mass value="0.0772232533904796"/>
-    <inertia ixx="7.1e-05" iyy="6.9e-05" izz="9.8e-05" ixy="0.0" iyz="0.0" ixz="-1.5e-05"/>
-  </inertial>
-  <visual>
-    <origin xyz="-0.16 -0.0 -1.024" rpy="0 0 0"/>
-    <geometry>
-      <mesh filename="file://$(find moiro_description)/meshes/gripper_base.stl" scale="0.001 0.001 0.001"/>
-    </geometry>
-    <material name="silver"/>
-  </visual>
-  <collision>
-    <origin xyz="-0.16 -0.0 -1.024" rpy="0 0 0"/>
-    <geometry>
-      <mesh filename="file://$(find moiro_description)/meshes/gripper_base.stl" scale="0.001 0.001 0.001"/>
-    </geometry>
-  </collision>
-</link>
-<link name="gripper_left3">
-  <inertial>
-    <origin xyz="0.015990426629758026 -0.012967523057101044 0.0034753903195707814" rpy="0 0 0"/>
-    <mass value="0.012694878221619885"/>
-    <inertia ixx="2e-06" iyy="5e-06" izz="7e-06" ixy="3e-06" iyz="0.0" ixz="-0.0"/>
-  </inertial>
-  <visual>
-    <origin xyz="-0.22039 0.01846 -1.027642" rpy="0 0 0"/>
-    <geometry>
-      <mesh filename="file://$(find moiro_description)/meshes/gripper_left3.stl" scale="0.001 0.001 0.001"/>
-    </geometry>
-    <material name="silver"/>
-  </visual>
-  <collision>
-    <origin xyz="-0.22039 0.01846 -1.027642" rpy="0 0 0"/>
-    <geometry>
-      <mesh filename="file://$(find moiro_description)/meshes/gripper_left3.stl" scale="0.001 0.001 0.001"/>
-    </geometry>
-  </collision>
-</link>
-<link name="gripper_left1">
-  <inertial>
-    <origin xyz="0.011053309239173859 -0.005253691764351268 0.0001366080392810609" rpy="0 0 0"/>
-    <mass value="0.013042175257524559"/>
-    <inertia ixx="1e-06" iyy="5e-06" izz="6e-06" ixy="-2e-06" iyz="0.0" ixz="0.0"/>
-  </inertial>
-  <visual>
-    <origin xyz="-0.271438 0.051465 -1.031142" rpy="0 0 0"/>
-    <geometry>
-      <mesh filename="file://$(find moiro_description)/meshes/gripper_left1.stl" scale="0.001 0.001 0.001"/>
-    </geometry>
-    <material name="silver"/>
-  </visual>
-  <collision>
-    <origin xyz="-0.271438 0.051465 -1.031142" rpy="0 0 0"/>
-    <geometry>
-      <mesh filename="file://$(find moiro_description)/meshes/gripper_left1.stl" scale="0.001 0.001 0.001"/>
-    </geometry>
-  </collision>
-</link>
-<link name="gripper_right3">
-  <inertial>
-    <origin xyz="0.01599042559398811 0.012967524435816866 0.0035248809278745075" rpy="0 0 0"/>
-    <mass value="0.012694878221619885"/>
-    <inertia ixx="2e-06" iyy="5e-06" izz="7e-06" ixy="-3e-06" iyz="0.0" ixz="0.0"/>
-  </inertial>
-  <visual>
-    <origin xyz="-0.22039 -0.01822 -1.027642" rpy="0 0 0"/>
-    <geometry>
-      <mesh filename="file://$(find moiro_description)/meshes/gripper_right3.stl" scale="0.001 0.001 0.001"/>
-    </geometry>
-    <material name="silver"/>
-  </visual>
-  <collision>
-    <origin xyz="-0.22039 -0.01822 -1.027642" rpy="0 0 0"/>
-    <geometry>
-      <mesh filename="file://$(find moiro_description)/meshes/gripper_right3.stl" scale="0.001 0.001 0.001"/>
-    </geometry>
-  </collision>
-</link>
-<link name="gripper_right1">
-  <inertial>
-    <origin xyz="0.011053308203403722 0.0052536931430675685 -0.00013633679183122638" rpy="0 0 0"/>
-    <mass value="0.013042175257524559"/>
-    <inertia ixx="1e-06" iyy="5e-06" izz="6e-06" ixy="2e-06" iyz="0.0" ixz="-0.0"/>
-  </inertial>
-  <visual>
-    <origin xyz="-0.271438 -0.051225 -1.031142" rpy="0 0 0"/>
-    <geometry>
-      <mesh filename="file://$(find moiro_description)/meshes/gripper_right1.stl" scale="0.001 0.001 0.001"/>
-    </geometry>
-    <material name="silver"/>
-  </visual>
-  <collision>
-    <origin xyz="-0.271438 -0.051225 -1.031142" rpy="0 0 0"/>
-    <geometry>
-      <mesh filename="file://$(find moiro_description)/meshes/gripper_right1.stl" scale="0.001 0.001 0.001"/>
-    </geometry>
-  </collision>
-</link>
 <link name="cobot_body">
   <inertial>
-    <origin xyz="-2.1294138884612695e-08 -0.012465741614899743 0.0436047733772541" rpy="0 0 0"/>
+    <origin xyz="-2.1294138884612695e-08 -0.012465741614899743 0.04360477337725388" rpy="0 0 0"/>
     <mass value="9.352590646947165"/>
     <inertia ixx="0.020014" iyy="0.013492" izz="0.021572" ixy="-0.0" iyz="-0.000111" ixz="-0.0"/>
   </inertial>
   <visual>
-    <origin xyz="0.0 0.0 -0.519" rpy="0 0 0"/>
+    <origin xyz="0.0 0.0 -0.516" rpy="0 0 0"/>
     <geometry>
       <mesh filename="file://$(find moiro_description)/meshes/cobot_body.stl" scale="0.001 0.001 0.001"/>
@@ -278,5 +182,5 @@
   </visual>
   <collision>
-    <origin xyz="0.0 0.0 -0.519" rpy="0 0 0"/>
+    <origin xyz="0.0 0.0 -0.516" rpy="0 0 0"/>
     <geometry>
       <mesh filename="file://$(find moiro_description)/meshes/cobot_body.stl" scale="0.001 0.001 0.001"/>
@@ -286,10 +190,10 @@
 <link name="wheel_right">
   <inertial>
-    <origin xyz="7.185686845753172e-07 -0.013441732021015451 6.740004032668168e-08" rpy="0 0 0"/>
+    <origin xyz="7.185686845753172e-07 -0.013441732021015451 6.740004027117052e-08" rpy="0 0 0"/>
     <mass value="0.6403675217821955"/>
     <inertia ixx="0.00197" iyy="0.003862" izz="0.00197" ixy="0.0" iyz="0.0" ixz="-0.0"/>
   </inertial>
   <visual>
-    <origin xyz="-0.000298 0.2233 -0.1055" rpy="0 0 0"/>
+    <origin xyz="-0.000298 0.2233 -0.1025" rpy="0 0 0"/>
     <geometry>
       <mesh filename="file://$(find moiro_description)/meshes/wheel_right.stl" scale="0.001 0.001 0.001"/>
@@ -298,5 +202,5 @@
   </visual>
   <collision>
-    <origin xyz="-0.000298 0.2233 -0.1055" rpy="0 0 0"/>
+    <origin xyz="-0.000298 0.2233 -0.1025" rpy="0 0 0"/>
     <geometry>
       <mesh filename="file://$(find moiro_description)/meshes/wheel_right.stl" scale="0.001 0.001 0.001"/>
@@ -306,10 +210,10 @@
 <link name="wheel_left">
   <inertial>
-    <origin xyz="5.370332256415832e-07 0.013441732021011232 2.8938916790677283e-08" rpy="0 0 0"/>
+    <origin xyz="5.370332256415832e-07 0.013441732021011232 2.8938916707410556e-08" rpy="0 0 0"/>
     <mass value="0.6403675217821955"/>
     <inertia ixx="0.00197" iyy="0.003862" izz="0.00197" ixy="-0.0" iyz="0.0" ixz="0.0"/>
   </inertial>
   <visual>
-    <origin xyz="-0.000298 -0.2233 -0.1055" rpy="0 0 0"/>
+    <origin xyz="-0.000298 -0.2233 -0.1025" rpy="0 0 0"/>
     <geometry>
       <mesh filename="file://$(find moiro_description)/meshes/wheel_left.stl" scale="0.001 0.001 0.001"/>
@@ -318,5 +222,5 @@
   </visual>
   <collision>
-    <origin xyz="-0.000298 -0.2233 -0.1055" rpy="0 0 0"/>
+    <origin xyz="-0.000298 -0.2233 -0.1025" rpy="0 0 0"/>
     <geometry>
       <mesh filename="file://$(find moiro_description)/meshes/wheel_left.stl" scale="0.001 0.001 0.001"/>
@@ -326,10 +230,10 @@
 <link name="caster_4">
   <inertial>
-    <origin xyz="-0.020672705075060666 -0.0093964574939722 -0.02565460037687653" rpy="0 0 0"/>
+    <origin xyz="-0.02067270507506061 -0.009396457493972207 -0.11565460037687654" rpy="0 0 0"/>
     <mass value="0.14564908217460187"/>
     <inertia ixx="4.1e-05" iyy="5.4e-05" izz="2.2e-05" ixy="0.0" iyz="0.0" ixz="0.0"/>
   </inertial>
   <visual>
-    <origin xyz="-0.238132 0.037118 -0.058" rpy="0 0 0"/>
+    <origin xyz="-0.238132 0.037118 -0.145" rpy="0 0 0"/>
     <geometry>
       <mesh filename="file://$(find moiro_description)/meshes/caster_4.stl" scale="0.001 0.001 0.001"/>
@@ -338,5 +242,5 @@
   </visual>
   <collision>
-    <origin xyz="-0.238132 0.037118 -0.058" rpy="0 0 0"/>
+    <origin xyz="-0.238132 0.037118 -0.145" rpy="0 0 0"/>
     <geometry>
       <mesh filename="file://$(find moiro_description)/meshes/caster_4.stl" scale="0.001 0.001 0.001"/>
@@ -346,10 +250,10 @@
 <link name="caster_3">
   <inertial>
-    <origin xyz="-0.02067270507506075 0.006390241409318889 -0.02565460037687651" rpy="0 0 0"/>
+    <origin xyz="-0.02067270507506072 0.006390241409318889 -0.025654600376876516" rpy="0 0 0"/>
     <mass value="0.14564908217460187"/>
     <inertia ixx="4.1e-05" iyy="5.4e-05" izz="2.2e-05" ixy="0.0" iyz="0.0" ixz="0.0"/>
   </inertial>
   <visual>
-    <origin xyz="-0.238132 -0.040529 -0.058" rpy="0 0 0"/>
+    <origin xyz="-0.238132 -0.040529 -0.055" rpy="0 0 0"/>
     <geometry>
       <mesh filename="file://$(find moiro_description)/meshes/caster_3.stl" scale="0.001 0.001 0.001"/>
@@ -358,5 +262,5 @@
   </visual>
   <collision>
-    <origin xyz="-0.238132 -0.040529 -0.058" rpy="0 0 0"/>
+    <origin xyz="-0.238132 -0.040529 -0.055" rpy="0 0 0"/>
     <geometry>
       <mesh filename="file://$(find moiro_description)/meshes/caster_3.stl" scale="0.001 0.001 0.001"/>
@@ -366,10 +270,10 @@
 <link name="caster_6">
   <inertial>
-    <origin xyz="0.02067255115624625 0.009396455766248653 -0.02565460037687644" rpy="0 0 0"/>
+    <origin xyz="0.020672551156246277 0.009396455766248653 -0.11565460037687647" rpy="0 0 0"/>
     <mass value="0.14564908217460187"/>
     <inertia ixx="4.1e-05" iyy="5.4e-05" izz="2.2e-05" ixy="0.0" iyz="0.0" ixz="0.0"/>
   </inertial>
   <visual>
-    <origin xyz="0.238132 -0.037118 -0.058" rpy="0 0 0"/>
+    <origin xyz="0.238132 -0.037118 -0.145" rpy="0 0 0"/>
     <geometry>
       <mesh filename="file://$(find moiro_description)/meshes/caster_6.stl" scale="0.001 0.001 0.001"/>
@@ -378,5 +282,5 @@
   </visual>
   <collision>
-    <origin xyz="0.238132 -0.037118 -0.058" rpy="0 0 0"/>
+    <origin xyz="0.238132 -0.037118 -0.145" rpy="0 0 0"/>
     <geometry>
       <mesh filename="file://$(find moiro_description)/meshes/caster_6.stl" scale="0.001 0.001 0.001"/>
@@ -386,10 +290,10 @@
 <link name="caster_5">
   <inertial>
-    <origin xyz="0.02067255115624622 -0.006390243137041694 -0.025654600376876474" rpy="0 0 0"/>
+    <origin xyz="0.02067255115624625 -0.006390243137041701 -0.1156546003768765" rpy="0 0 0"/>
     <mass value="0.14564908217460187"/>
     <inertia ixx="4.1e-05" iyy="5.4e-05" izz="2.2e-05" ixy="0.0" iyz="0.0" ixz="0.0"/>
   </inertial>
   <visual>
-    <origin xyz="0.238132 0.040529 -0.058" rpy="0 0 0"/>
+    <origin xyz="0.238132 0.040529 -0.145" rpy="0 0 0"/>
     <geometry>
       <mesh filename="file://$(find moiro_description)/meshes/caster_5.stl" scale="0.001 0.001 0.001"/>
@@ -398,5 +302,5 @@
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