Commit message: try_to_edit_base_link_position

File: moiro_description/urdf/moiro.xacro (robot description, xacro)
@@ -24,5 +24,5 @@
   </collision>
 </link>
-<link name="basearm">
+<link name="basearm_1">
   <inertial>
     <origin xyz="0.006896766224728663 -2.0863790969221033e-15 0.05549018686904683" rpy="0 0 0"/>
@@ -33,5 +33,5 @@
     <origin xyz="0.0 0.0 -0.606" rpy="0 0 0"/>
     <geometry>
-      <mesh filename="file://$(find moiro_description)/meshes/basearm.stl" scale="0.001 0.001 0.001"/>
+      <mesh filename="file://$(find moiro_description)/meshes/basearm_1.stl" scale="0.001 0.001 0.001"/>
     </geometry>
     <material name="silver"/>
@@ -40,9 +40,9 @@
     <origin xyz="0.0 0.0 -0.606" rpy="0 0 0"/>
     <geometry>
-      <mesh filename="file://$(find moiro_description)/meshes/basearm.stl" scale="0.001 0.001 0.001"/>
-    </geometry>
-  </collision>
-</link>
-<link name="lowerarm">
+      <mesh filename="file://$(find moiro_description)/meshes/basearm_1.stl" scale="0.001 0.001 0.001"/>
+    </geometry>
+  </collision>
+</link>
+<link name="lowerarm_1">
   <inertial>
     <origin xyz="0.036906585755669324 -2.1017837997117547e-15 0.06799999999999129" rpy="0 0 0"/>
@@ -53,5 +53,5 @@
     <origin xyz="-0.045 0.0 -0.691" rpy="0 0 0"/>
     <geometry>
-      <mesh filename="file://$(find moiro_description)/meshes/lowerarm.stl" scale="0.001 0.001 0.001"/>
+      <mesh filename="file://$(find moiro_description)/meshes/lowerarm_1.stl" scale="0.001 0.001 0.001"/>
     </geometry>
     <material name="silver"/>
@@ -60,9 +60,9 @@
     <origin xyz="-0.045 0.0 -0.691" rpy="0 0 0"/>
     <geometry>
-      <mesh filename="file://$(find moiro_description)/meshes/lowerarm.stl" scale="0.001 0.001 0.001"/>
-    </geometry>
-  </collision>
-</link>
-<link name="upperarm">
+      <mesh filename="file://$(find moiro_description)/meshes/lowerarm_1.stl" scale="0.001 0.001 0.001"/>
+    </geometry>
+  </collision>
+</link>
+<link name="upperarm_1">
   <inertial>
     <origin xyz="-0.03502268825299596 1.5060537258141013e-15 0.04949999999999133" rpy="0 0 0"/>
@@ -73,5 +73,5 @@
     <origin xyz="-0.045 0.0 -0.827" rpy="0 0 0"/>
     <geometry>
-      <mesh filename="file://$(find moiro_description)/meshes/upperarm.stl" scale="0.001 0.001 0.001"/>
+      <mesh filename="file://$(find moiro_description)/meshes/upperarm_1.stl" scale="0.001 0.001 0.001"/>
     </geometry>
     <material name="silver"/>
@@ -80,9 +80,9 @@
     <origin xyz="-0.045 0.0 -0.827" rpy="0 0 0"/>
     <geometry>
-      <mesh filename="file://$(find moiro_description)/meshes/upperarm.stl" scale="0.001 0.001 0.001"/>
-    </geometry>
-  </collision>
-</link>
-<link name="pitcharm">
+      <mesh filename="file://$(find moiro_description)/meshes/upperarm_1.stl" scale="0.001 0.001 0.001"/>
+    </geometry>
+  </collision>
+</link>
+<link name="pitcharm_1">
   <inertial>
     <origin xyz="0.034423872869188424 5.291448440797201e-15 0.010576127130799362" rpy="0 0 0"/>
@@ -93,5 +93,5 @@
     <origin xyz="-0.045 -0.0 -0.926" rpy="0 0 0"/>
     <geometry>
-      <mesh filename="file://$(find moiro_description)/meshes/pitcharm.stl" scale="0.001 0.001 0.001"/>
+      <mesh filename="file://$(find moiro_description)/meshes/pitcharm_1.stl" scale="0.001 0.001 0.001"/>
     </geometry>
     <material name="silver"/>
@@ -100,9 +100,9 @@
     <origin xyz="-0.045 -0.0 -0.926" rpy="0 0 0"/>
     <geometry>
-      <mesh filename="file://$(find moiro_description)/meshes/pitcharm.stl" scale="0.001 0.001 0.001"/>
-    </geometry>
-  </collision>
-</link>
-<link name="rollarm">
+      <mesh filename="file://$(find moiro_description)/meshes/pitcharm_1.stl" scale="0.001 0.001 0.001"/>
+    </geometry>
+  </collision>
+</link>
+<link name="rollarm_1">
   <inertial>
     <origin xyz="-3.816391647148976e-15 6.350716433653324e-15 0.042116696506125595" rpy="0 0 0"/>
@@ -113,5 +113,5 @@
     <origin xyz="-0.09 -0.0 -0.971" rpy="0 0 0"/>
     <geometry>
-      <mesh filename="file://$(find moiro_description)/meshes/rollarm.stl" scale="0.001 0.001 0.001"/>
+      <mesh filename="file://$(find moiro_description)/meshes/rollarm_1.stl" scale="0.001 0.001 0.001"/>
     </geometry>
     <material name="silver"/>
@@ -120,9 +120,9 @@
     <origin xyz="-0.09 -0.0 -0.971" rpy="0 0 0"/>
     <geometry>
-      <mesh filename="file://$(find moiro_description)/meshes/rollarm.stl" scale="0.001 0.001 0.001"/>
-    </geometry>
-  </collision>
-</link>
-<link name="gripperarm">
+      <mesh filename="file://$(find moiro_description)/meshes/rollarm_1.stl" scale="0.001 0.001 0.001"/>
+    </geometry>
+  </collision>
+</link>
+<link name="gripperarm_1">
   <inertial>
     <origin xyz="0.00999999999999615 6.341038805146582e-15 -9.103828801926284e-15" rpy="0 0 0"/>
@@ -133,5 +133,5 @@
     <origin xyz="-0.13 -0.0 -1.021" rpy="0 0 0"/>
     <geometry>
-      <mesh filename="file://$(find moiro_description)/meshes/gripperarm.stl" scale="0.001 0.001 0.001"/>
+      <mesh filename="file://$(find moiro_description)/meshes/gripperarm_1.stl" scale="0.001 0.001 0.001"/>
     </geometry>
     <material name="silver"/>
@@ -140,9 +140,9 @@
     <origin xyz="-0.13 -0.0 -1.021" rpy="0 0 0"/>
     <geometry>
-      <mesh filename="file://$(find moiro_description)/meshes/gripperarm.stl" scale="0.001 0.001 0.001"/>
-    </geometry>
-  </collision>
-</link>
-<link name="cobot_camera">
+      <mesh filename="file://$(find moiro_description)/meshes/gripperarm_1.stl" scale="0.001 0.001 0.001"/>
+    </geometry>
+  </collision>
+</link>
+<link name="cobot_camera_1">
   <inertial>
     <origin xyz="0.017423960091247193 0.003253426631193808 0.005819385718719872" rpy="0 0 0"/>
@@ -153,5 +153,5 @@
     <origin xyz="-0.15 -0.0 -1.021" rpy="0 0 0"/>
     <geometry>
-      <mesh filename="file://$(find moiro_description)/meshes/cobot_camera.stl" scale="0.001 0.001 0.001"/>
+      <mesh filename="file://$(find moiro_description)/meshes/cobot_camera_1.stl" scale="0.001 0.001 0.001"/>
     </geometry>
     <material name="silver"/>
@@ -160,9 +160,9 @@
     <origin xyz="-0.15 -0.0 -1.021" rpy="0 0 0"/>
     <geometry>
-      <mesh filename="file://$(find moiro_description)/meshes/cobot_camera.stl" scale="0.001 0.001 0.001"/>
-    </geometry>
-  </collision>
-</link>
-<link name="cobot_body">
+      <mesh filename="file://$(find moiro_description)/meshes/cobot_camera_1.stl" scale="0.001 0.001 0.001"/>
+    </geometry>
+  </collision>
+</link>
+<link name="cobot_body_1">
   <inertial>
     <origin xyz="-2.1294138884612695e-08 -0.012465741614899743 0.04360477337725388" rpy="0 0 0"/>
@@ -173,5 +173,5 @@
     <origin xyz="0.0 0.0 -0.516" rpy="0 0 0"/>
     <geometry>
-      <mesh filename="file://$(find moiro_description)/meshes/cobot_body.stl" scale="0.001 0.001 0.001"/>
+      <mesh filename="file://$(find moiro_description)/meshes/cobot_body_1.stl" scale="0.001 0.001 0.001"/>
     </geometry>
     <material name="silver"/>
@@ -180,9 +180,9 @@
     <origin xyz="0.0 0.0 -0.516" rpy="0 0 0"/>
     <geometry>
-      <mesh filename="file://$(find moiro_description)/meshes/cobot_body.stl" scale="0.001 0.001 0.001"/>
-    </geometry>
-  </collision>
-</link>
-<link name="wheel_right">
+      <mesh filename="file://$(find moiro_description)/meshes/cobot_body_1.stl" scale="0.001 0.001 0.001"/>
+    </geometry>
+  </collision>
+</link>
+<link name="wheel_right_1">
   <inertial>
     <origin xyz="7.185686845753172e-07 -0.013441732021015451 6.740004027117052e-08" rpy="0 0 0"/>
@@ -193,5 +193,5 @@
     <origin xyz="-0.000298 0.2233 -0.1025" rpy="0 0 0"/>
     <geometry>
-      <mesh filename="file://$(find moiro_description)/meshes/wheel_right.stl" scale="0.001 0.001 0.001"/>
+      <mesh filename="file://$(find moiro_description)/meshes/wheel_right_1.stl" scale="0.001 0.001 0.001"/>
     </geometry>
     <material name="silver"/>
@@ -200,9 +200,9 @@
     <origin xyz="-0.000298 0.2233 -0.1025" rpy="0 0 0"/>
     <geometry>
-      <mesh filename="file://$(find moiro_description)/meshes/wheel_right.stl" scale="0.001 0.001 0.001"/>
-    </geometry>
-  </collision>
-</link>
-<link name="wheel_left">
+      <mesh filename="file://$(find moiro_description)/meshes/wheel_right_1.stl" scale="0.001 0.001 0.001"/>
+    </geometry>
+  </collision>
+</link>
+<link name="wheel_left_1">
   <inertial>
     <origin xyz="5.370332256415832e-07 0.013441732021011232 2.8938916707410556e-08" rpy="0 0 0"/>
@@ -213,5 +213,5 @@
     <origin xyz="-0.000298 -0.2233 -0.1025" rpy="0 0 0"/>
     <geometry>
-      <mesh filename="file://$(find moiro_description)/meshes/wheel_left.stl" scale="0.001 0.001 0.001"/>
+      <mesh filename="file://$(find moiro_description)/meshes/wheel_left_1.stl" scale="0.001 0.001 0.001"/>
     </geometry>
     <material name="silver"/>
@@ -220,9 +220,9 @@
     <origin xyz="-0.000298 -0.2233 -0.1025" rpy="0 0 0"/>
     <geometry>
-      <mesh filename="file://$(find moiro_description)/meshes/wheel_left.stl" scale="0.001 0.001 0.001"/>
-    </geometry>
-  </collision>
-</link>
-<link name="camera_zig">
+      <mesh filename="file://$(find moiro_description)/meshes/wheel_left_1.stl" scale="0.001 0.001 0.001"/>
+    </geometry>
+  </collision>
+</link>
+<link name="camera_zig_1">
   <inertial>
     <origin xyz="0.014530099919036615 0.044049338752250145 0.028344157098708633" rpy="0 0 0"/>
@@ -233,5 +233,5 @@
     <origin xyz="-0.24875 0.045 -0.52" rpy="0 0 0"/>
     <geometry>
-      <mesh filename="file://$(find moiro_description)/meshes/camera_zig.stl" scale="0.001 0.001 0.001"/>
+      <mesh filename="file://$(find moiro_description)/meshes/camera_zig_1.stl" scale="0.001 0.001 0.001"/>
     </geometry>
     <material name="silver"/>
@@ -240,9 +240,9 @@
     <origin xyz="-0.24875 0.045 -0.52" rpy="0 0 0"/>
     <geometry>
-      <mesh filename="file://$(find moiro_description)/meshes/camera_zig.stl" scale="0.001 0.001 0.001"/>
-    </geometry>
-  </collision>
-</link>
-<link name="imu_link">
+      <mesh filename="file://$(find moiro_description)/meshes/camera_zig_1.stl" scale="0.001 0.001 0.001"/>
+    </geometry>
+  </collision>
+</link>
+<link name="imu_link_1">
   <inertial>
     <origin xyz="-0.04153434985377516 -0.031630029317067154 0.002586806247330431" rpy="0 0 0"/>
@@ -253,5 +253,5 @@
     <origin xyz="-0.048037 -0.045 -0.1" rpy="0 0 0"/>
     <geometry>
-      <mesh filename="file://$(find moiro_description)/meshes/imu_link.stl" scale="0.001 0.001 0.001"/>
+      <mesh filename="file://$(find moiro_description)/meshes/imu_link_1.stl" scale="0.001 0.001 0.001"/>
     </geometry>
     <material name="silver"/>
@@ -260,9 +260,9 @@
     <origin xyz="-0.048037 -0.045 -0.1" rpy="0 0 0"/>
     <geometry>
-      <mesh filename="file://$(find moiro_description)/meshes/imu_link.stl" scale="0.001 0.001 0.001"/>
-    </geometry>
-  </collision>
-</link>
-<link name="camera_link">
+      <mesh filename="file://$(find moiro_description)/meshes/imu_link_1.stl" scale="0.001 0.001 0.001"/>
+    </geometry>
+  </collision>
+</link>
+<link name="camera_link_1">
   <inertial>
     <origin xyz="0.012171550992974123 1.5521819223018093e-06 -4.879803335100519e-05" rpy="0 0 0"/>
@@ -273,5 +273,5 @@
     <origin xyz="-0.26675 -0.00175 -0.558285" rpy="0 0 0"/>
     <geometry>
-      <mesh filename="file://$(find moiro_description)/meshes/camera_link.stl" scale="0.001 0.001 0.001"/>
+      <mesh filename="file://$(find moiro_description)/meshes/camera_link_1.stl" scale="0.001 0.001 0.001"/>
     </geometry>
     <material name="silver"/>
@@ -280,5 +280,5 @@
     <origin xyz="-0.26675 -0.00175 -0.558285" rpy="0 0 0"/>
     <geometry>
-      <mesh filename="file://$(find moiro_description)/meshes/camera_link.stl" scale="0.001 0.001 0.001"/>
+      <mesh filename="file://$(find moiro_description)/meshes/camera_link_1.stl" scale="0.001 0.001 0.001"/>
     </geometry>
   </collision>
@@ -364,5 +364,5 @@
   </collision>
 </link>
-<link name="motor_right">
+<link name="motor_right_1">
   <inertial>
     <origin xyz="-0.00788584475935802 -0.006913170455323331 0.014484211131926578" rpy="0 0 0"/>
@@ -373,5 +373,5 @@
     <origin xyz="0.004 0.198 -0.088" rpy="0 0 0"/>
     <geometry>
-      <mesh filename="file://$(find moiro_description)/meshes/motor_right.stl" scale="0.001 0.001 0.001"/>
+      <mesh filename="file://$(find moiro_description)/meshes/motor_right_1.stl" scale="0.001 0.001 0.001"/>
     </geometry>
     <material name="silver"/>
@@ -380,9 +380,9 @@
     <origin xyz="0.004 0.198 -0.088" rpy="0 0 0"/>
     <geometry>
-      <mesh filename="file://$(find moiro_description)/meshes/motor_right.stl" scale="0.001 0.001 0.001"/>
-    </geometry>
-  </collision>
-</link>
-<link name="motor_left">
+      <mesh filename="file://$(find moiro_description)/meshes/motor_right_1.stl" scale="0.001 0.001 0.001"/>
+    </geometry>
+  </collision>
+</link>
+<link name="motor_left_1">
   <inertial>
     <origin xyz="-0.007885844759358442 0.006913170455319778 0.014515788868055449" rpy="0 0 0"/>
@@ -393,5 +393,5 @@
     <origin xyz="0.004 -0.198 -0.088" rpy="0 0 0"/>
     <geometry>
-      <mesh filename="file://$(find moiro_description)/meshes/motor_left.stl" scale="0.001 0.001 0.001"/>
+      <mesh filename="file://$(find moiro_description)/meshes/motor_left_1.stl" scale="0.001 0.001 0.001"/>
     </geometry>
     <material name="silver"/>
@@ -400,9 +400,9 @@
     <origin xyz="0.004 -0.198 -0.088" rpy="0 0 0"/>
     <geometry>
-      <mesh filename="file://$(find moiro_description)/meshes/motor_left.stl" scale="0.001 0.001 0.001"/>
-    </geometry>
-  </collision>
-</link>
-<link name="base_plate">
+      <mesh filename="file://$(find moiro_description)/meshes/motor_left_1.stl" scale="0.001 0.001 0.001"/>
+    </geometry>
+  </collision>
+</link>
+<link name="base_plate_1">
   <inertial>
     <origin xyz="3.024732238173218e-08 -0.020354187478525226 0.008984617763925118" rpy="0 0 0"/>
@@ -413,5 +413,5 @@
     <origin xyz="-0.0 0.0 -0.498" rpy="0 0 0"/>
     <geometry>
-      <mesh filename="file://$(find moiro_description)/meshes/base_plate.stl" scale="0.001 0.001 0.001"/>
+      <mesh filename="file://$(find moiro_description)/meshes/base_plate_1.stl" scale="0.001 0.001 0.001"/>
     </geometry>
     <material name="silver"/>
@@ -420,5 +420,25 @@
     <origin xyz="-0.0 0.0 -0.498" rpy="0 0 0"/>
     <geometry>
-      <mesh filename="file://$(find moiro_description)/meshes/base_plate.stl" scale="0.001 0.001 0.001"/>
+      <mesh filename="file://$(find moiro_description)/meshes/base_plate_1.stl" scale="0.001 0.001 0.001"/>
+    </geometry>
+  </collision>
+</link>
+<link name="base_scan_1">
+  <inertial>
+    <origin xyz="1.4890131030027799e-05 -0.008617362464656688 0.011145262430183378" rpy="0 0 0"/>
+    <mass value="0.4177280575470181"/>
+    <inertia ixx="0.000281" iyy="0.000143" izz="0.000351" ixy="-0.0" iyz="-3.9e-05" ixz="-0.0"/>
+  </inertial>
+  <visual>
+    <origin xyz="0.000412 -0.003127 -0.268745" rpy="0 0 0"/>
+    <geometry>
+      <mesh filename="file://$(find moiro_description)/meshes/base_scan_1.stl" scale="0.001 0.001 0.001"/>
+    </geometry>
+    <material name="silver"/>
+  </visual>
+  <collision>
+    <origin xyz="0.000412 -0.003127 -0.268745" rpy="0 0 0"/>
+    <geometry>
+      <mesh filename="file://$(find moiro_description)/meshes/base_scan_1.stl" scale="0.001 0.001 0.001"/>
     </geometry>
   </collision>
@@ -426,6 +446,6 @@
 <joint name="mycobot_joint_1" type="revolute">
   <origin xyz="0.0 0.0 0.09" rpy="0 0 0"/>
-  <parent link="cobot_body"/>
-  <child link="basearm"/>
+  <parent link="cobot_body_1"/>
+  <child link="basearm_1"/>
   <axis xyz="-0.0 0.0 1.0"/>
   <limit upper="2.792527" lower="-2.792527" effort="100" velocity="100"/>
@@ -433,6 +453,6 @@
 <joint name="mycobot_joint_2" type="revolute">
   <origin xyz="0.045 0.0 0.085" rpy="0 0 0"/>
-  <parent link="basearm"/>
-  <child link="lowerarm"/>
+  <parent link="basearm_1"/>
+  <child link="lowerarm_1"/>
   <axis xyz="1.0 0.0 0.0"/>
   <limit upper="2.792527" lower="-2.792527" effort="100" velocity="100"/>
@@ -440,6 +460,6 @@
 <joint name="mycobot_joint_3" type="revolute">
   <origin xyz="0.0 0.0 0.136" rpy="0 0 0"/>
-  <parent link="lowerarm"/>
-  <child link="upperarm"/>
+  <parent link="lowerarm_1"/>
+  <child link="upperarm_1"/>
   <axis xyz="-1.0 -0.0 -0.0"/>
   <limit upper="2.792527" lower="-2.792527" effort="100" velocity="100"/>
@@ -447,6 +467,6 @@
 <joint name="mycobot_joint_4" type="revolute">
   <origin xyz="0.0 0.0 0.099" rpy="0 0 0"/>
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
Commit message: Update moiro.xacro

File: moiro_description/urdf/moiro.xacro (robot description, xacro)
@@ -11,5 +11,5 @@
   </inertial>
   <visual>
-    <origin xyz="0 0 0" rpy="0 0 0"/>
+    <origin xyz="0 0 -0.09" rpy="0 0 0"/>
     <geometry>
       <mesh filename="file://$(find moiro_description)/meshes/base_link.stl" scale="0.001 0.001 0.001"/>
@@ -18,5 +18,5 @@
   </visual>
   <collision>
-    <origin xyz="0 0 0" rpy="0 0 0"/>
+    <origin xyz="0 0 -0.09" rpy="0 0 0"/>
     <geometry>
       <mesh filename="file://$(find moiro_description)/meshes/base_link.stl" scale="0.001 0.001 0.001"/>
@@ -509,10 +509,10 @@
 </joint>
 <joint name="joint_camera" type="fixed">
-  <origin xyz="0.24875 -0.045 0.52" rpy="0 0 0"/>
+  <origin xyz="0.24875 -0.045 0.43" rpy="0 0 0"/>
   <parent link="base_link"/>
   <child link="camera_zig_1"/>
 </joint>
 <joint name="imu_joint" type="fixed">
-  <origin xyz="0.048037 0.045 0.1" rpy="0 0 0"/>
+  <origin xyz="0.048037 0.045 0.01" rpy="0 0 0"/>
   <parent link="base_link"/>
   <child link="imu_link_1"/>
@@ -524,40 +524,40 @@
 </joint>
 <joint name="Rigid 79" type="fixed">
-  <origin xyz="-0.238132 0.037118 0.145" rpy="0 0 0"/>
+  <origin xyz="-0.238132 0.037118 0.055" rpy="0 0 0"/>
   <parent link="base_link"/>
   <child link="caster_6"/>
 </joint>
 <joint name="Rigid 80" type="fixed">
-  <origin xyz="-0.238132 -0.037118 0.145" rpy="0 0 0"/>
+  <origin xyz="-0.238132 -0.037118 0.055" rpy="0 0 0"/>
   <parent link="base_link"/>
   <child link="caster_5"/>
 </joint>
 <joint name="Rigid 81" type="fixed">
-  <origin xyz="0.238132 -0.037118 0.145" rpy="0 0 0"/>
+  <origin xyz="0.238132 -0.037118 0.055" rpy="0 0 0"/>
   <parent link="base_link"/>
   <child link="caster_4"/>
 </joint>
 <joint name="Rigid 82" type="fixed">
-  <origin xyz="0.238132 0.037118 0.055" rpy="0 0 0"/>
+  <origin xyz="0.238132 0.037118 -0.035" rpy="0 0 0"/>
   <parent link="base_link"/>
   <child link="caster_3"/>
 </joint>
 <joint name="Rigid 83" type="fixed">
-  <origin xyz="-0.004 -0.198 0.088" rpy="0 0 0"/>
+  <origin xyz="-0.004 -0.198 -0.002" rpy="0 0 0"/>
   <parent link="base_link"/>
   <child link="motor_right_1"/>
 </joint>
 <joint name="Rigid 84" type="fixed">
-  <origin xyz="-0.004 0.198 0.088" rpy="0 0 0"/>
+  <origin xyz="-0.004 0.198 -0.002" rpy="0 0 0"/>
   <parent link="base_link"/>
   <child link="motor_left_1"/>
 </joint>
 <joint name="Rigid 85" type="fixed">
-  <origin xyz="0.0 0.0 0.498" rpy="0 0 0"/>
+  <origin xyz="0.0 0.0 0.408" rpy="0 0 0"/>
   <parent link="base_link"/>
   <child link="base_plate_1"/>
 </joint>
 <joint name="Rigid 86" type="fixed">
-  <origin xyz="-0.000412 0.003127 0.268745" rpy="0 0 0"/>
+  <origin xyz="-0.000412 0.003127 0.178745" rpy="0 0 0"/>
   <parent link="base_link"/>
   <child link="base_scan_1"/>
