Commit message: add base_footprint, change mycobot link name

File: moiro_description/urdf/moiro.xacro (robot description, xacro)
@@ -4,12 +4,19 @@
 <xacro:include filename="$(find moiro_description)/urdf/moiro.trans" />
 <xacro:include filename="$(find moiro_description)/urdf/moiro.gazebo" />
+<!-- base_footprint 추가 base_link의 좌표는 0 0 0 -->
+<link name="base_footprint"/>
+<joint name="base_joint" type="fixed">
+  <parent link="base_footprint"/>
+  <child link="base_link" />
+  <origin xyz="0 0 0.090" rpy="0 0 0"/>
+</joint>
 <link name="base_link">
   <inertial>
-    <origin xyz="0.004418404192394108 -0.0009320583420061628 0.2493907147199333" rpy="0 0 0"/>
+    <origin xyz="0.004418404804107676 -0.0009320583374515539 0.24939071509061012" rpy="0 0 0"/>
     <mass value="10.314151582114752"/>
     <inertia ixx="0.498632" iyy="0.533352" izz="0.429421" ixy="0.002003" iyz="0.002378" ixz="-0.014194"/>
   </inertial>
   <visual>
-    <origin xyz="0 0 -0.09" rpy="0 0 0"/>
+    <origin xyz="0 0 0" rpy="0 0 0"/>
     <geometry>
       <mesh filename="file://$(find moiro_description)/meshes/base_link.stl" scale="0.001 0.001 0.001"/>
@@ -18,5 +25,5 @@
   </visual>
   <collision>
-    <origin xyz="0 0 -0.09" rpy="0 0 0"/>
+    <origin xyz="0 0 0" rpy="0 0 0"/>
     <geometry>
       <mesh filename="file://$(find moiro_description)/meshes/base_link.stl" scale="0.001 0.001 0.001"/>
@@ -24,5 +31,5 @@
   </collision>
 </link>
-<link name="basearm_1">
+<link name="link1">
   <inertial>
     <origin xyz="0.006896766224728663 -2.0863790969221033e-15 0.05549018686904683" rpy="0 0 0"/>
@@ -33,5 +40,5 @@
     <origin xyz="0.0 0.0 -0.606" rpy="0 0 0"/>
     <geometry>
-      <mesh filename="file://$(find moiro_description)/meshes/basearm_1.stl" scale="0.001 0.001 0.001"/>
+      <mesh filename="file://$(find moiro_description)/meshes/link1.stl" scale="0.001 0.001 0.001"/>
     </geometry>
     <material name="silver"/>
@@ -40,9 +47,9 @@
     <origin xyz="0.0 0.0 -0.606" rpy="0 0 0"/>
     <geometry>
-      <mesh filename="file://$(find moiro_description)/meshes/basearm_1.stl" scale="0.001 0.001 0.001"/>
-    </geometry>
-  </collision>
-</link>
-<link name="lowerarm_1">
+      <mesh filename="file://$(find moiro_description)/meshes/link1.stl" scale="0.001 0.001 0.001"/>
+    </geometry>
+  </collision>
+</link>
+<link name="link2">
   <inertial>
     <origin xyz="0.036906585755669324 -2.1017837997117547e-15 0.06799999999999129" rpy="0 0 0"/>
@@ -53,5 +60,5 @@
     <origin xyz="-0.045 0.0 -0.691" rpy="0 0 0"/>
     <geometry>
-      <mesh filename="file://$(find moiro_description)/meshes/lowerarm_1.stl" scale="0.001 0.001 0.001"/>
+      <mesh filename="file://$(find moiro_description)/meshes/link2.stl" scale="0.001 0.001 0.001"/>
     </geometry>
     <material name="silver"/>
@@ -60,9 +67,9 @@
     <origin xyz="-0.045 0.0 -0.691" rpy="0 0 0"/>
     <geometry>
-      <mesh filename="file://$(find moiro_description)/meshes/lowerarm_1.stl" scale="0.001 0.001 0.001"/>
-    </geometry>
-  </collision>
-</link>
-<link name="upperarm_1">
+      <mesh filename="file://$(find moiro_description)/meshes/link2.stl" scale="0.001 0.001 0.001"/>
+    </geometry>
+  </collision>
+</link>
+<link name="link3">
   <inertial>
     <origin xyz="-0.03502268825299596 1.5060537258141013e-15 0.04949999999999133" rpy="0 0 0"/>
@@ -73,5 +80,5 @@
     <origin xyz="-0.045 0.0 -0.827" rpy="0 0 0"/>
     <geometry>
-      <mesh filename="file://$(find moiro_description)/meshes/upperarm_1.stl" scale="0.001 0.001 0.001"/>
+      <mesh filename="file://$(find moiro_description)/meshes/link3.stl" scale="0.001 0.001 0.001"/>
     </geometry>
     <material name="silver"/>
@@ -80,9 +87,9 @@
     <origin xyz="-0.045 0.0 -0.827" rpy="0 0 0"/>
     <geometry>
-      <mesh filename="file://$(find moiro_description)/meshes/upperarm_1.stl" scale="0.001 0.001 0.001"/>
-    </geometry>
-  </collision>
-</link>
-<link name="pitcharm_1">
+      <mesh filename="file://$(find moiro_description)/meshes/link3.stl" scale="0.001 0.001 0.001"/>
+    </geometry>
+  </collision>
+</link>
+<link name="link4">
   <inertial>
     <origin xyz="0.034423872869188424 5.291448440797201e-15 0.010576127130799362" rpy="0 0 0"/>
@@ -93,5 +100,5 @@
     <origin xyz="-0.045 -0.0 -0.926" rpy="0 0 0"/>
     <geometry>
-      <mesh filename="file://$(find moiro_description)/meshes/pitcharm_1.stl" scale="0.001 0.001 0.001"/>
+      <mesh filename="file://$(find moiro_description)/meshes/link4.stl" scale="0.001 0.001 0.001"/>
     </geometry>
     <material name="silver"/>
@@ -100,9 +107,9 @@
     <origin xyz="-0.045 -0.0 -0.926" rpy="0 0 0"/>
     <geometry>
-      <mesh filename="file://$(find moiro_description)/meshes/pitcharm_1.stl" scale="0.001 0.001 0.001"/>
-    </geometry>
-  </collision>
-</link>
-<link name="rollarm_1">
+      <mesh filename="file://$(find moiro_description)/meshes/link4.stl" scale="0.001 0.001 0.001"/>
+    </geometry>
+  </collision>
+</link>
+<link name="link5">
   <inertial>
     <origin xyz="-3.816391647148976e-15 6.350716433653324e-15 0.042116696506125595" rpy="0 0 0"/>
@@ -113,5 +120,5 @@
     <origin xyz="-0.09 -0.0 -0.971" rpy="0 0 0"/>
     <geometry>
-      <mesh filename="file://$(find moiro_description)/meshes/rollarm_1.stl" scale="0.001 0.001 0.001"/>
+      <mesh filename="file://$(find moiro_description)/meshes/link5.stl" scale="0.001 0.001 0.001"/>
     </geometry>
     <material name="silver"/>
@@ -120,9 +127,9 @@
     <origin xyz="-0.09 -0.0 -0.971" rpy="0 0 0"/>
     <geometry>
-      <mesh filename="file://$(find moiro_description)/meshes/rollarm_1.stl" scale="0.001 0.001 0.001"/>
-    </geometry>
-  </collision>
-</link>
-<link name="gripperarm_1">
+      <mesh filename="file://$(find moiro_description)/meshes/link5.stl" scale="0.001 0.001 0.001"/>
+    </geometry>
+  </collision>
+</link>
+<link name="link6">
   <inertial>
     <origin xyz="0.00999999999999615 6.341038805146582e-15 -9.103828801926284e-15" rpy="0 0 0"/>
@@ -133,5 +140,5 @@
     <origin xyz="-0.13 -0.0 -1.021" rpy="0 0 0"/>
     <geometry>
-      <mesh filename="file://$(find moiro_description)/meshes/gripperarm_1.stl" scale="0.001 0.001 0.001"/>
+      <mesh filename="file://$(find moiro_description)/meshes/link6.stl" scale="0.001 0.001 0.001"/>
     </geometry>
     <material name="silver"/>
@@ -140,9 +147,9 @@
     <origin xyz="-0.13 -0.0 -1.021" rpy="0 0 0"/>
     <geometry>
-      <mesh filename="file://$(find moiro_description)/meshes/gripperarm_1.stl" scale="0.001 0.001 0.001"/>
-    </geometry>
-  </collision>
-</link>
-<link name="cobot_camera_1">
+      <mesh filename="file://$(find moiro_description)/meshes/link6.stl" scale="0.001 0.001 0.001"/>
+    </geometry>
+  </collision>
+</link>
+<link name="cobot_camera">
   <inertial>
     <origin xyz="0.017423960091247193 0.003253426631193808 0.005819385718719872" rpy="0 0 0"/>
@@ -153,5 +160,5 @@
     <origin xyz="-0.15 -0.0 -1.021" rpy="0 0 0"/>
     <geometry>
-      <mesh filename="file://$(find moiro_description)/meshes/cobot_camera_1.stl" scale="0.001 0.001 0.001"/>
+      <mesh filename="file://$(find moiro_description)/meshes/cobot_camera.stl" scale="0.001 0.001 0.001"/>
     </geometry>
     <material name="silver"/>
@@ -160,9 +167,9 @@
     <origin xyz="-0.15 -0.0 -1.021" rpy="0 0 0"/>
     <geometry>
-      <mesh filename="file://$(find moiro_description)/meshes/cobot_camera_1.stl" scale="0.001 0.001 0.001"/>
-    </geometry>
-  </collision>
-</link>
-<link name="cobot_body_1">
+      <mesh filename="file://$(find moiro_description)/meshes/cobot_camera.stl" scale="0.001 0.001 0.001"/>
+    </geometry>
+  </collision>
+</link>
+<link name="link0">
   <inertial>
     <origin xyz="-2.1294138884612695e-08 -0.012465741614899743 0.04360477337725388" rpy="0 0 0"/>
@@ -173,5 +180,5 @@
     <origin xyz="0.0 0.0 -0.516" rpy="0 0 0"/>
     <geometry>
-      <mesh filename="file://$(find moiro_description)/meshes/cobot_body_1.stl" scale="0.001 0.001 0.001"/>
+      <mesh filename="file://$(find moiro_description)/meshes/link0.stl" scale="0.001 0.001 0.001"/>
     </geometry>
     <material name="silver"/>
@@ -180,9 +187,9 @@
     <origin xyz="0.0 0.0 -0.516" rpy="0 0 0"/>
     <geometry>
-      <mesh filename="file://$(find moiro_description)/meshes/cobot_body_1.stl" scale="0.001 0.001 0.001"/>
-    </geometry>
-  </collision>
-</link>
-<link name="wheel_right_1">
+      <mesh filename="file://$(find moiro_description)/meshes/link0.stl" scale="0.001 0.001 0.001"/>
+    </geometry>
+  </collision>
+</link>
+<link name="wheel_right">
   <inertial>
     <origin xyz="7.185686845753172e-07 -0.013441732021015451 6.740004027117052e-08" rpy="0 0 0"/>
@@ -193,5 +200,5 @@
     <origin xyz="-0.000298 0.2233 -0.1025" rpy="0 0 0"/>
     <geometry>
-      <mesh filename="file://$(find moiro_description)/meshes/wheel_right_1.stl" scale="0.001 0.001 0.001"/>
+      <mesh filename="file://$(find moiro_description)/meshes/wheel_right.stl" scale="0.001 0.001 0.001"/>
     </geometry>
     <material name="silver"/>
@@ -200,9 +207,9 @@
     <origin xyz="-0.000298 0.2233 -0.1025" rpy="0 0 0"/>
     <geometry>
-      <mesh filename="file://$(find moiro_description)/meshes/wheel_right_1.stl" scale="0.001 0.001 0.001"/>
-    </geometry>
-  </collision>
-</link>
-<link name="wheel_left_1">
+      <mesh filename="file://$(find moiro_description)/meshes/wheel_right.stl" scale="0.001 0.001 0.001"/>
+    </geometry>
+  </collision>
+</link>
+<link name="wheel_left">
   <inertial>
     <origin xyz="5.370332256415832e-07 0.013441732021011232 2.8938916707410556e-08" rpy="0 0 0"/>
@@ -213,5 +220,5 @@
     <origin xyz="-0.000298 -0.2233 -0.1025" rpy="0 0 0"/>
     <geometry>
-      <mesh filename="file://$(find moiro_description)/meshes/wheel_left_1.stl" scale="0.001 0.001 0.001"/>
+      <mesh filename="file://$(find moiro_description)/meshes/wheel_left.stl" scale="0.001 0.001 0.001"/>
     </geometry>
     <material name="silver"/>
@@ -220,9 +227,9 @@
     <origin xyz="-0.000298 -0.2233 -0.1025" rpy="0 0 0"/>
     <geometry>
-      <mesh filename="file://$(find moiro_description)/meshes/wheel_left_1.stl" scale="0.001 0.001 0.001"/>
-    </geometry>
-  </collision>
-</link>
-<link name="camera_zig_1">
+      <mesh filename="file://$(find moiro_description)/meshes/wheel_left.stl" scale="0.001 0.001 0.001"/>
+    </geometry>
+  </collision>
+</link>
+<link name="camera_zig">
   <inertial>
     <origin xyz="0.014530099919036615 0.044049338752250145 0.028344157098708633" rpy="0 0 0"/>
@@ -233,5 +240,5 @@
     <origin xyz="-0.24875 0.045 -0.52" rpy="0 0 0"/>
     <geometry>
-      <mesh filename="file://$(find moiro_description)/meshes/camera_zig_1.stl" scale="0.001 0.001 0.001"/>
+      <mesh filename="file://$(find moiro_description)/meshes/camera_zig.stl" scale="0.001 0.001 0.001"/>
     </geometry>
     <material name="silver"/>
@@ -240,9 +247,9 @@
     <origin xyz="-0.24875 0.045 -0.52" rpy="0 0 0"/>
     <geometry>
-      <mesh filename="file://$(find moiro_description)/meshes/camera_zig_1.stl" scale="0.001 0.001 0.001"/>
-    </geometry>
-  </collision>
-</link>
-<link name="imu_link_1">
+      <mesh filename="file://$(find moiro_description)/meshes/camera_zig.stl" scale="0.001 0.001 0.001"/>
+    </geometry>
+  </collision>
+</link>
+<link name="imu_link">
   <inertial>
     <origin xyz="-0.04153434985377516 -0.031630029317067154 0.002586806247330431" rpy="0 0 0"/>
@@ -253,5 +260,5 @@
     <origin xyz="-0.048037 -0.045 -0.1" rpy="0 0 0"/>
     <geometry>
-      <mesh filename="file://$(find moiro_description)/meshes/imu_link_1.stl" scale="0.001 0.001 0.001"/>
+      <mesh filename="file://$(find moiro_description)/meshes/imu_link.stl" scale="0.001 0.001 0.001"/>
     </geometry>
     <material name="silver"/>
@@ -260,9 +267,9 @@
     <origin xyz="-0.048037 -0.045 -0.1" rpy="0 0 0"/>
     <geometry>
-      <mesh filename="file://$(find moiro_description)/meshes/imu_link_1.stl" scale="0.001 0.001 0.001"/>
-    </geometry>
-  </collision>
-</link>
-<link name="camera_link_1">
+      <mesh filename="file://$(find moiro_description)/meshes/imu_link.stl" scale="0.001 0.001 0.001"/>
+    </geometry>
+  </collision>
+</link>
+<link name="camera_link">
   <inertial>
     <origin xyz="0.012171550992974123 1.5521819223018093e-06 -4.879803335100519e-05" rpy="0 0 0"/>
@@ -273,5 +280,5 @@
     <origin xyz="-0.26675 -0.00175 -0.558285" rpy="0 0 0"/>
     <geometry>
-      <mesh filename="file://$(find moiro_description)/meshes/camera_link_1.stl" scale="0.001 0.001 0.001"/>
+      <mesh filename="file://$(find moiro_description)/meshes/camera_link.stl" scale="0.001 0.001 0.001"/>
     </geometry>
     <material name="silver"/>
@@ -280,5 +287,5 @@
     <origin xyz="-0.26675 -0.00175 -0.558285" rpy="0 0 0"/>
     <geometry>
-      <mesh filename="file://$(find moiro_description)/meshes/camera_link_1.stl" scale="0.001 0.001 0.001"/>
+      <mesh filename="file://$(find moiro_description)/meshes/camera_link.stl" scale="0.001 0.001 0.001"/>
     </geometry>
   </collision>
@@ -286,10 +293,10 @@
 <link name="caster_6">
   <inertial>
-    <origin xyz="0.020672551156246277 0.009396455766248653 -0.11565460037687647" rpy="0 0 0"/>
+    <origin xyz="0.020672551156246277 0.009396455766248653 -0.02565460037687648" rpy="0 0 0"/>
     <mass value="0.14564908217460187"/>
     <inertia ixx="4.1e-05" iyy="5.4e-05" izz="2.2e-05" ixy="0.0" iyz="0.0" ixz="0.0"/>
   </inertial>
   <visual>
-    <origin xyz="0.238132 -0.037118 -0.145" rpy="0 0 0"/>
+    <origin xyz="0.238132 -0.037118 -0.055" rpy="0 0 0"/>
     <geometry>
       <mesh filename="file://$(find moiro_description)/meshes/caster_6.stl" scale="0.001 0.001 0.001"/>
@@ -298,5 +305,5 @@
   </visual>
   <collision>
-    <origin xyz="0.238132 -0.037118 -0.145" rpy="0 0 0"/>
+    <origin xyz="0.238132 -0.037118 -0.055" rpy="0 0 0"/>
     <geometry>
       <mesh filename="file://$(find moiro_description)/meshes/caster_6.stl" scale="0.001 0.001 0.001"/>
@@ -306,10 +313,10 @@
 <link name="caster_5">
   <inertial>
-    <origin xyz="0.02067255115624614 -0.00939645749397091 -0.1156546003768768" rpy="0 0 0"/>
+    <origin xyz="0.02067255115624614 -0.00939645749397091 -0.025654600376876818" rpy="0 0 0"/>
     <mass value="0.14564908217460187"/>
     <inertia ixx="4.1e-05" iyy="5.4e-05" izz="2.2e-05" ixy="0.0" iyz="0.0" ixz="0.0"/>
   </inertial>
   <visual>
-    <origin xyz="0.238132 0.037118 -0.145" rpy="0 0 0"/>
+    <origin xyz="0.238132 0.037118 -0.055" rpy="0 0 0"/>
     <geometry>
       <mesh filename="file://$(find moiro_description)/meshes/caster_5.stl" scale="0.001 0.001 0.001"/>
@@ -318,5 +325,5 @@
   </visual>
   <collision>
-    <origin xyz="0.238132 0.037118 -0.145" rpy="0 0 0"/>
+    <origin xyz="0.238132 0.037118 -0.055" rpy="0 0 0"/>
     <geometry>
       <mesh filename="file://$(find moiro_description)/meshes/caster_5.stl" scale="0.001 0.001 0.001"/>
@@ -326,10 +333,10 @@
 <link name="caster_4">
   <inertial>
-    <origin xyz="-0.02067270507506061 -0.009396457493972207 -0.11565460037687654" rpy="0 0 0"/>
+    <origin xyz="-0.02067270507506061 -0.009396457493972207 -0.02565460037687655" rpy="0 0 0"/>
     <mass value="0.14564908217460187"/>
     <inertia ixx="4.1e-05" iyy="5.4e-05" izz="2.2e-05" ixy="0.0" iyz="0.0" ixz="0.0"/>
   </inertial>
   <visual>
-    <origin xyz="-0.238132 0.037118 -0.145" rpy="0 0 0"/>
+    <origin xyz="-0.238132 0.037118 -0.055" rpy="0 0 0"/>
     <geometry>
       <mesh filename="file://$(find moiro_description)/meshes/caster_4.stl" scale="0.001 0.001 0.001"/>
@@ -338,5 +345,5 @@
   </visual>
   <collision>
-    <origin xyz="-0.238132 0.037118 -0.145" rpy="0 0 0"/>
+    <origin xyz="-0.238132 0.037118 -0.055" rpy="0 0 0"/>
     <geometry>
       <mesh filename="file://$(find moiro_description)/meshes/caster_4.stl" scale="0.001 0.001 0.001"/>
@@ -364,5 +371,5 @@
   </collision>
 </link>
-<link name="motor_right_1">
+<link name="motor_right">
   <inertial>
     <origin xyz="-0.00788584475935802 -0.006913170455323331 0.014484211131926578" rpy="0 0 0"/>
@@ -373,5 +380,5 @@
     <origin xyz="0.004 0.198 -0.088" rpy="0 0 0"/>
     <geometry>
-      <mesh filename="file://$(find moiro_description)/meshes/motor_right_1.stl" scale="0.001 0.001 0.001"/>
+      <mesh filename="file://$(find moiro_description)/meshes/motor_right.stl" scale="0.001 0.001 0.001"/>
     </geometry>
     <material name="silver"/>
@@ -380,9 +387,9 @@
     <origin xyz="0.004 0.198 -0.088" rpy="0 0 0"/>
     <geometry>
-      <mesh filename="file://$(find moiro_description)/meshes/motor_right_1.stl" scale="0.001 0.001 0.001"/>
-    </geometry>
-  </collision>
-</link>
-<link name="motor_left_1">
+      <mesh filename="file://$(find moiro_description)/meshes/motor_right.stl" scale="0.001 0.001 0.001"/>
+    </geometry>
+  </collision>
+</link>
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